File: KiCAD/AmigaPCI Mainboard-KiCAD/power.kicad_sch (KiCad schematic)
At the start: 64 parts, among them CN600 ATX-24, J600 POWER_SWITCH, J9003 Case Fan, Q600 MMBT3904, U209 74HCT08, U214 74HCT244, U219 74HCT04, U222 74HCT4066, U600 74HCT14, U601 74HCT74

Commit message: Routing June 6 2023
Parts:
- removed U209: 74HCT08, Package_SO:TSSOP-14_4.4x5mm_P0.65mm, symbol 74xx:74LS08
- removed U214: 74HCT244, Package_SO:TSSOP-20_4.4x6.5mm_P0.65mm, symbol 74xx:74LS244_Split
Connections:
- no-connect marks 10 -> 12

Commit message: Routing June 10 2023
Parts:
- added U3: 74HCT08, Package_SO:TSSOP-14_4.4x5mm_P0.65mm, symbol 74xx:74LS08
Connections:
- no-connect marks 12 -> 15
Changed lines of the file:
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@@
   (no_connect (at 283.591 50.546))
   (no_connect (at 268.478 66.548))
+  (no_connect (at 269.494 94.742))
   (no_connect (at 275.971 55.626))
   (no_connect (at 283.718 66.548))
   (no_connect (at 130.175 111.125))
+  (no_connect (at 269.494 89.662))
   (no_connect (at 276.098 76.708))
   (no_connect (at 268.478 69.088))
@@
   (no_connect (at 311.785 44.45))
   (no_connect (at 59.69 39.37))
+  (no_connect (at 284.734 92.202))
   (no_connect (at 268.351 50.546))
   (no_connect (at 276.098 61.468))
@@
         )
       )
+    )
+  )
+  (symbol (lib_id "74xx:74LS08") (at 277.114 92.202 0) (unit 4)
+    (in_bom yes) (on_board yes) (dnp no)
+    (property "Reference" "U3" (at 277.114 83.947 0)
+      (effects (font (size 1.27 1.27)))
+    )
+    (property "Value" "74HCT08" (at 277.114 86.2584 0)
+      (effects (font (size 1.27 1.27)))
+    )
+    (property "Footprint" "Package_SO:TSSOP-14_4.4x5mm_P0.65mm" (at 277.114 92.202 0)
+      (effects (font (size 1.27 1.27)) hide)
+    )
+    (property "Datasheet" "http://www.ti.com/lit/gpn/sn74LS08" (at 277.114 92.202 0)
+      (effects (font (size 1.27 1.27)) hide)
+    )
+    (pin "1")
+    (pin "2")
+    (pin "3")
+    (pin "4")
+    (pin "5")
+    (pin "6")
+    (pin "10")
+    (pin "8")
+    (pin "9")
+    (pin "11")
+    (pin "12")
+    (pin "13")
+    (pin "14")
+    (pin "7")
+    (instances
+      (project "AmigaPCI Mainboard"
+        (path "/72453515-27fe-4336-91f3-e3c8054f7767/34f2eda3-97b6-4f91-ad2d-01637d6f5405"
+          (reference "U3") (unit 4)
+        )
+        (path "/72453515-27fe-4336-91f3-e3c8054f7767/4cb777ef-2899-49f4-b38f-a0c07d84fa7d"
+          (reference "U305") (unit 4)
+        )
+      )
+      (project "2000ATX"
+        (path "/bb595301-1c72-49dc-ac6f-007419f3a7fd/00000000-0000-0000-0000-0000607c1eb7"
+          (reference "U207") (unit 2)
+        )
+      )

Commit message: Routing June 11 2023
Parts:
- added unit 5 of U600
- added unit 6 of U600
Connections:
- no-connect marks 15 -> 19

Commit message: Routing June 12 2023
Parts:
- H1, H10, H2, H3, H4, H5, H6, H7, H8, H9: footprint A2900:MountingHole_Pad -> MountingHole:MountingHole_4mm_Pad_Via
Changed lines of the file:
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@@
       (effects (font (size 1.27 1.27)) (justify left) hide)
     )
-    (property "Footprint" "A2900:MountingHole_Pad" (at 289.56 146.05 0)
+    (property "Footprint" "MountingHole:MountingHole_4mm_Pad_Via" (at 289.56 146.05 0)
       (effects (font (size 1.27 1.27)) hide)
     )
@@
       (effects (font (size 1.27 1.27)) (justify left) hide)
     )
-    (property "Footprint" "A2900:MountingHole_Pad" (at 279.4 151.13 0)
+    (property "Footprint" "MountingHole:MountingHole_4mm_Pad_Via" (at 279.4 151.13 0)
       (effects (font (size 1.27 1.27)) hide)
     )
@@
       (effects (font (size 1.27 1.27)) (justify left) hide)
     )
-    (property "Footprint" "A2900:MountingHole_Pad" (at 289.56 151.13 0)
+    (property "Footprint" "MountingHole:MountingHole_4mm_Pad_Via" (at 289.56 151.13 0)
       (effects (font (size 1.27 1.27)) hide)
     )
@@
       (effects (font (size 1.27 1.27)) (justify left) hide)
     )
-    (property "Footprint" "A2900:MountingHole_Pad" (at 269.24 151.13 0)
+    (property "Footprint" "MountingHole:MountingHole_4mm_Pad_Via" (at 269.24 151.13 0)
       (effects (font (size 1.27 1.27)) hide)
     )
@@
       (effects (font (size 1.27 1.27)) (justify left) hide)
     )
-    (property "Footprint" "A2900:MountingHole_Pad" (at 279.4 146.05 0)
+    (property "Footprint" "MountingHole:MountingHole_4mm_Pad_Via" (at 279.4 146.05 0)
       (effects (font (size 1.27 1.27)) hide)
     )
@@
       (effects (font (size 1.27 1.27)) (justify left) hide)
     )
-    (property "Footprint" "A2900:MountingHole_Pad" (at 279.4 156.21 0)
+    (property "Footprint" "MountingHole:MountingHole_4mm_Pad_Via" (at 279.4 156.21 0)
       (effects (font (size 1.27 1.27)) hide)
     )
@@
       (effects (font (size 1.27 1.27)) (justify left) hide)
     )
-    (property "Footprint" "A2900:MountingHole_Pad" (at 269.24 146.05 0)
+    (property "Footprint" "MountingHole:MountingHole_4mm_Pad_Via" (at 269.24 146.05 0)
       (effects (font (size 1.27 1.27)) hide)
     )
@@
       (effects (font (size 1.27 1.27)) (justify left) hide)
     )
-    (property "Footprint" "A2900:MountingHole_Pad" (at 289.56 156.21 0)
+    (property "Footprint" "MountingHole:MountingHole_4mm_Pad_Via" (at 289.56 156.21 0)
       (effects (font (size 1.27 1.27)) hide)
     )
@@
       (effects (font (size 1.27 1.27)) (justify left) hide)
     )
-    (property "Footprint" "A2900:MountingHole_Pad" (at 289.56 160.655 0)
+    (property "Footprint" "MountingHole:MountingHole_4mm_Pad_Via" (at 289.56 160.655 0)
       (effects (font (size 1.27 1.27)) hide)
     )
@@
       (effects (font (size 1.27 1.27)) (justify left) hide)
     )
-    (property "Footprint" "A2900:MountingHole_Pad" (at 269.24 156.21 0)
-      (effects (font (size 1.27 1.27)) hide)
-    )
+    (property "Footprint" "MountingHole:MountingHole_4mm_Pad_Via" (at 269.24 156.21 0)
+      (effects (font (size 1.27 1.27)) hide)
+    )

Commit message: Routing June 14 2023
Parts:
- added U229: 74CBT16233, Package_SO:SSOP-56_7.5x18.5mm_P0.635mm, symbol AmigaPCI-Symbols:74CBT16233
Connections:
- no-connect marks 19 -> 34
Other:
- moved on the sheet: J9003, U219A, U219D, U219F, U222D, U3D, U600E, U600F, U601A

Commit message: Routing June 16 2023
Parts:
- U229: Part Number (none) -> SN74CBT16233DL
Changed lines of the file:
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@@
+      (effects (font (size 1.27 1.27)) hide)
+    )
+    (property "Part Number" "SN74CBT16233DL" (at 299.593 69.088 0)
       (effects (font (size 1.27 1.27)) hide)
     )
@@
       (effects (font (size 1.27 1.27)) hide)
     )
+    (property "Part Number" "SN74CBT16233DL" (at 299.72 38.481 0)
+      (effects (font (size 1.27 1.27)) hide)
+    )
     (pin "1")
     (pin "55")
@@
       (effects (font (size 1.27 1.27)) hide)
     )
+    (property "Part Number" "SN74CBT16233DL" (at 299.847 54.102 0)
+      (effects (font (size 1.27 1.27)) hide)
+    )

Commit message: Routing June 17 2023
Connections:
- net +3V3 renamed +3.3V
Changed lines of the file:
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@@
-    )
-  )
-  (symbol (lib_id "power:+3V3") (at 381.381 189.611 0) (unit 1)
-    (in_bom yes) (on_board yes) (dnp no) (fields_autoplaced)
-    (property "Reference" "#PWR0105" (at 381.381 193.421 0)
-      (effects (font (size 1.27 1.27)) hide)
-    )
-    (property "Value" "+3V3" (at 381.381 186.1091 0)
-      (effects (font (size 1.27 1.27)))
-    )
-    (property "Footprint" "" (at 381.381 189.611 0)
-      (effects (font (size 1.27 1.27)) hide)
-    )
-    (property "Datasheet" "" (at 381.381 189.611 0)
-      (effects (font (size 1.27 1.27)) hide)
-    )
-    (pin "1")
-    (instances
-      (project "AmigaPCI Mainboard"
-        (path "/72453515-27fe-4336-91f3-e3c8054f7767/4cb777ef-2899-49f4-b38f-a0c07d84fa7d"
-          (reference "#PWR0105") (unit 1)
-        )
-      )
     )
   )
@@
     )
   )
+  (symbol (lib_id "power:+3.3V") (at 381.381 189.611 0) (unit 1)
+    (in_bom yes) (on_board yes) (dnp no) (fields_autoplaced)
+    (property "Reference" "#PWR05" (at 381.381 193.421 0)
+      (effects (font (size 1.27 1.27)) hide)
+    )
+    (property "Value" "+3.3V" (at 381.381 186.1091 0)
+      (effects (font (size 1.27 1.27)))
+    )
+    (property "Footprint" "" (at 381.381 189.611 0)
+      (effects (font (size 1.27 1.27)) hide)
+    )
+    (property "Datasheet" "" (at 381.381 189.611 0)
+      (effects (font (size 1.27 1.27)) hide)
+    )
+    (pin "1")
+    (instances
+      (project "AmigaPCI Mainboard"
+        (path "/72453515-27fe-4336-91f3-e3c8054f7767/60b2ee65-4978-4bd8-934d-67b9c15d34cc"
+          (reference "#PWR05") (unit 1)
+        )
+        (path "/72453515-27fe-4336-91f3-e3c8054f7767/4cb777ef-2899-49f4-b38f-a0c07d84fa7d"
+          (reference "#PWR0105") (unit 1)
+        )
+      )
+    )
+  )
   (symbol (lib_id "2000ATX-rescue:CP_Small-Device") (at 149.352 46.99 180) (unit 1)
     (in_bom yes) (on_board yes) (dnp no)
@@
     )
   )
+  (symbol (lib_id "power:+3.3V") (at 222.123 33.02 0) (unit 1)
+    (in_bom yes) (on_board yes) (dnp no) (fields_autoplaced)
+    (property "Reference" "#PWR05" (at 222.123 36.83 0)
+      (effects (font (size 1.27 1.27)) hide)
+    )
+    (property "Value" "+3.3V" (at 222.123 29.5181 0)
+      (effects (font (size 1.27 1.27)))
+    )
+    (property "Footprint" "" (at 222.123 33.02 0)
+      (effects (font (size 1.27 1.27)) hide)
+    )
+    (property "Datasheet" "" (at 222.123 33.02 0)
+      (effects (font (size 1.27 1.27)) hide)
+    )
+    (pin "1")
+    (instances
+      (project "AmigaPCI Mainboard"
+        (path "/72453515-27fe-4336-91f3-e3c8054f7767/60b2ee65-4978-4bd8-934d-67b9c15d34cc"
+          (reference "#PWR05") (unit 1)
+        )
+        (path "/72453515-27fe-4336-91f3-e3c8054f7767/4cb777ef-2899-49f4-b38f-a0c07d84fa7d"
+          (reference "#PWR0108") (unit 1)
+        )
+      )
+    )
+  )
   (symbol (lib_id "2000ATX-rescue:CP_Small-Device") (at 103.632 46.99 180) (unit 1)
     (in_bom yes) (on_board yes) (dnp no)
@@
         )
       )
-    )
-  )
-  (symbol (lib_id "power:+3V3") (at 222.123 33.02 0) (unit 1)
-    (in_bom yes) (on_board yes) (dnp no)
-    (property "Reference" "#PWR0223" (at 222.123 36.83 0)
-      (effects (font (size 1.27 1.27)) hide)
-    )
-    (property "Value" "+3V3" (at 221.996 29.464 0)
-      (effects (font (size 1.27 1.27)))
-    )
-    (property "Footprint" "" (at 222.123 33.02 0)
-      (effects (font (size 1.27 1.27)) hide)
-    )
-    (property "Datasheet" "" (at 222.123 33.02 0)
-      (effects (font (size 1.27 1.27)) hide)
-    )
-    (pin "1")
-    (instances
-      (project "AmigaPCI Mainboard"
-        (path "/72453515-27fe-4336-91f3-e3c8054f7767/4cb777ef-2899-49f4-b38f-a0c07d84fa7d"
-          (reference "#PWR0223") (unit 1)
-        )
-      )

Commit message: Routing June 24 2023
Parts:
- added FID1, FID2, FID3: Fiducial, Fiducial:Fiducial_1mm_Mask2mm, symbol Mechanical:Fiducial
- added U216: 74HCT08, Package_SO:SOIC-14_3.9x8.7mm_P1.27mm, symbol 74xx:74LS08
Connections:
- no-connect marks 34 -> 37
Changed lines of the file:
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@@
   (no_connect (at 307.34 35.941))
   (no_connect (at 292.227 54.102))
+  (no_connect (at 316.738 42.418))
   (no_connect (at 307.213 84.582))
   (no_connect (at 307.467 56.642))
@@
   (no_connect (at 282.194 79.756))
   (no_connect (at 291.973 84.582))
+  (no_connect (at 316.738 37.338))
   (no_connect (at 307.34 94.996))
   (no_connect (at 307.213 109.347))
   (no_connect (at 282.067 96.647))
+  (no_connect (at 331.978 39.878))
   (no_connect (at 265.811 38.1))
   (no_connect (at 273.558 49.022))
@@
     )
   )
+  (symbol (lib_id "Mechanical:Fiducial") (at 308.102 151.511 0) (unit 1)
+    (in_bom yes) (on_board yes) (dnp no) (fields_autoplaced)
+    (property "Reference" "FID3" (at 310.261 150.8673 0)
+      (effects (font (size 1.27 1.27)) (justify left))
+    )
+    (property "Value" "Fiducial" (at 310.261 152.7883 0)
+      (effects (font (size 1.27 1.27)) (justify left))
+    )
+    (property "Footprint" "Fiducial:Fiducial_1mm_Mask2mm" (at 308.102 151.511 0)
+      (effects (font (size 1.27 1.27)) hide)
+    )
+    (property "Datasheet" "~" (at 308.102 151.511 0)
+      (effects (font (size 1.27 1.27)) hide)
+    )
+    (instances
+      (project "AmigaPCI Mainboard"
+        (path "/72453515-27fe-4336-91f3-e3c8054f7767/4cb777ef-2899-49f4-b38f-a0c07d84fa7d"
+          (reference "FID3") (unit 1)
+        )
+      )
+    )
+  )
   (symbol (lib_id "2000ATX-rescue:CP_Small-Device") (at 111.887 58.42 0) (mirror y) (unit 1)
     (in_bom yes) (on_board yes) (dnp no)
@@
     )
   )
+  (symbol (lib_id "74xx:74LS08") (at 324.358 39.878 0) (mirror x) (unit 4)
+    (in_bom yes) (on_board yes) (dnp no)
+    (property "Reference" "U216" (at 324.358 31.8262 0)
+      (effects (font (size 1.27 1.27)))
+    )
+    (property "Value" "74HCT08" (at 324.358 34.1376 0)
+      (effects (font (size 1.27 1.27)))
+    )
+    (property "Footprint" "Package_SO:SOIC-14_3.9x8.7mm_P1.27mm" (at 324.358 39.878 0)
+      (effects (font (size 1.27 1.27)) hide)
+    )
+    (property "Datasheet" "http://www.ti.com/lit/gpn/sn74LS08" (at 324.358 39.878 0)
+      (effects (font (size 1.27 1.27)) hide)
+    )
+    (pin "1")
+    (pin "2")
+    (pin "3")
+    (pin "4")
+    (pin "5")
+    (pin "6")
+    (pin "10")
+    (pin "8")
+    (pin "9")
+    (pin "11")
+    (pin "12")
+    (pin "13")
+    (pin "14")
+    (pin "7")
+    (instances
+      (project "AmigaPCI Mainboard"
+        (path "/72453515-27fe-4336-91f3-e3c8054f7767/64185471-b9ae-4a50-a046-7157e86a04d0"
+          (reference "U216") (unit 4)
+        )
+        (path "/72453515-27fe-4336-91f3-e3c8054f7767/4cb777ef-2899-49f4-b38f-a0c07d84fa7d"
+          (reference "U216") (unit 4)
+        )
+      )
+      (project "2000ATX"
+        (path "/bb595301-1c72-49dc-ac6f-007419f3a7fd/00000000-0000-0000-0000-000060df4324"
+          (reference "U607") (unit 4)
+        )
+      )
+    )
+  )
   (symbol (lib_id "2000ATX-rescue:CP_Small-Device") (at 121.031 58.42 0) (mirror y) (unit 1)
     (in_bom yes) (on_board yes) (dnp no)
@@
     )
   )
+  (symbol (lib_id "Mechanical:Fiducial") (at 307.975 146.177 0) (unit 1)
+    (in_bom yes) (on_board yes) (dnp no) (fields_autoplaced)
+    (property "Reference" "FID2" (at 310.134 145.5333 0)
+      (effects (font (size 1.27 1.27)) (justify left))
+    )
+    (property "Value" "Fiducial" (at 310.134 147.4543 0)
+      (effects (font (size 1.27 1.27)) (justify left))
+    )
+    (property "Footprint" "Fiducial:Fiducial_1mm_Mask2mm" (at 307.975 146.177 0)
+      (effects (font (size 1.27 1.27)) hide)
+    )
+    (property "Datasheet" "~" (at 307.975 146.177 0)
+      (effects (font (size 1.27 1.27)) hide)
+    )
+    (instances
+      (project "AmigaPCI Mainboard"
+        (path "/72453515-27fe-4336-91f3-e3c8054f7767/4cb777ef-2899-49f4-b38f-a0c07d84fa7d"
+          (reference "FID2") (unit 1)
+        )
+      )
+    )
+  )
   (symbol (lib_id "Device:C_Polarized") (at 288.544 199.771 0) (unit 1)
     (in_bom yes) (on_board yes) (dnp no) (fields_autoplaced)
@@
         )
       )
+    )
+  )
+  (symbol (lib_id "Mechanical:Fiducial") (at 307.848 140.843 0) (unit 1)
+    (in_bom yes) (on_board yes) (dnp no) (fields_autoplaced)
+    (property "Reference" "FID1" (at 310.007 140.1993 0)
+      (effects (font (size 1.27 1.27)) (justify left))
+    )
+    (property "Value" "Fiducial" (at 310.007 142.1203 0)
+      (effects (font (size 1.27 1.27)) (justify left))
+    )
+    (property "Footprint" "Fiducial:Fiducial_1mm_Mask2mm" (at 307.848 140.843 0)
+      (effects (font (size 1.27 1.27)) hide)
+    )
+    (property "Datasheet" "~" (at 307.848 140.843 0)
+      (effects (font (size 1.27 1.27)) hide)
+    )
+    (instances
+      (project "AmigaPCI Mainboard"
+        (path "/72453515-27fe-4336-91f3-e3c8054f7767/4cb777ef-2899-49f4-b38f-a0c07d84fa7d"
+          (reference "FID1") (unit 1)
+        )
+      )
