File: KiCAD/AmigaPCI Mainboard-KiCAD/video.kicad_sch (KiCad schematic)
At the start: 51 parts, among them CN300 DB15_Female_HighDensity, CN301 Video-Slot, CN302 Video-Slot, CN303 Raspberry_Pi_Zero, J301 PI_BUTTON, J303 HSYNC/COMPSYNC, U201 74LVC1G74, U300 DENISE, U301 74AHCT244, U302 74AHCT244, U303 74LVC574, U304 74LVC574, U305 74HCT08, U307 74LVC86

Commit message: Routing June 9 2023
Connections:
- net M0V: now also RN300.5 (R4); no longer RN300.6 (R5)
- net M1H: now also RN300.6 (R5); no longer RN300.3 (R2)
- net M1V: now also RN300.3 (R2); no longer RN300.5 (R4)

Commit message: Routing-1 June 9 2023
Parts:
- CN303: footprint Module:Raspberry_Pi_Zero_Socketed_THT_FaceDown_MountingHoles -> Connector_PinSocket_2.54mm:PinSocket_2x20_P2.54mm_Vertical
- U301, U302: footprint Package_SO:SOIC-20W_7.5x12.8mm_P1.27mm -> Package_SO:TSSOP-20_4.4x5mm_P0.5mm
Changed lines of the file:
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@@
       (effects (font (size 1.27 1.27)))
     )
-    (property "Footprint" "Module:Raspberry_Pi_Zero_Socketed_THT_FaceDown_MountingHoles" (at 209.804 200.025 0)
+    (property "Footprint" "Connector_PinSocket_2.54mm:PinSocket_2x20_P2.54mm_Vertical" (at 209.804 200.025 0)
       (effects (font (size 1.27 1.27)) hide)
     )
@@
       (effects (font (size 1.27 1.27)))
     )
-    (property "Footprint" "Package_SO:SOIC-20W_7.5x12.8mm_P1.27mm" (at 135.255 137.414 0)
+    (property "Footprint" "Package_SO:TSSOP-20_4.4x5mm_P0.5mm" (at 135.255 137.414 0)
       (effects (font (size 1.27 1.27)) hide)
     )
@@
       (effects (font (size 1.27 1.27)))
     )
-    (property "Footprint" "Package_SO:SOIC-20W_7.5x12.8mm_P1.27mm" (at 135.255 61.214 0)
-      (effects (font (size 1.27 1.27)) hide)
-    )
+    (property "Footprint" "Package_SO:TSSOP-20_4.4x5mm_P0.5mm" (at 135.255 61.214 0)
+      (effects (font (size 1.27 1.27)) hide)
+    )

Commit message: Routing June 10 2023
Parts:
- CN300: symbol 2000ATX-rescue:DB15_Female_HighDensity-Connector -> AmigaPCI-Symbols:DB15_Female_HighDensity
- renumbered R203A1 to R226
Connections:
- net BURST: no longer U300.18 (BURST), U301.4 (1A1)
- net GND: now also CN300.16 (SHIELD)
- net PIXELSW: no longer U300.33 (PIXELSW), U301.6 (1A2)
- new net BUR: U300.18 (BURST), U301.4 (1A1)
- new net PSW: U300.33 (PIXELSW), U301.6 (1A2)
Changed lines of the file:
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@@
     (effects (font (size 1.27 1.27)) (justify left bottom))
   )
-  (label "PIXELSW" (at 74.422 87.884 0) (fields_autoplaced)
+  (label "PSW" (at 74.422 87.884 0) (fields_autoplaced)
     (effects (font (size 1.27 1.27)) (justify left bottom))
   )
@@
     (effects (font (size 1.2954 1.2954)) (justify right bottom))
   )
-  (label "BURST" (at 74.422 82.804 0) (fields_autoplaced)
+  (label "BUR" (at 74.422 82.804 0) (fields_autoplaced)
     (effects (font (size 1.27 1.27)) (justify left bottom))
   )
@@
   (symbol (lib_id "Device:R_Small") (at 341.503 204.089 270) (unit 1)
     (in_bom yes) (on_board yes) (dnp no)
-    (property "Reference" "R203A1" (at 337.82 202.311 90)
+    (property "Reference" "R226" (at 338.963 202.184 90)
       (effects (font (size 1.27 1.27)) (justify left))
     )
@@
       (project "AmigaPCI Mainboard"
         (path "/72453515-27fe-4336-91f3-e3c8054f7767/34f2eda3-97b6-4f91-ad2d-01637d6f5405"
-          (reference "R203A1") (unit 1)
+          (reference "R226") (unit 1)
         )
       )
@@
     )
   )
-  (symbol (lib_id "2000ATX-rescue:DB15_Female_HighDensity-Connector") (at 346.583 179.959 0) (unit 1)
+  (symbol (lib_id "AmigaPCI-Symbols:DB15_Female_HighDensity") (at 346.583 179.959 0) (unit 1)
     (in_bom yes) (on_board yes) (dnp no)
     (property "Reference" "CN300" (at 346.583 157.9372 0)
@@
       (effects (font (size 1.27 1.27)) hide)
     )
+    (pin "16")
     (pin "1")
     (pin "10")
@@
   (symbol (lib_id "Device:R_Small") (at 370.713 160.909 180) (unit 1)
     (in_bom yes) (on_board yes) (dnp no)
-    (property "Reference" "R304" (at 379.349 160.02 0)
+    (property "Reference" "R304" (at 376.936 160.02 0)
       (effects (font (size 1.27 1.27)) (justify left))
     )
@@
         )
       )
+    )
+  )
+  (symbol (lib_id "power:GND") (at 350.393 197.739 0) (unit 1)
+    (in_bom yes) (on_board yes) (dnp no)
+    (property "Reference" "#PWR0196" (at 350.393 204.089 0)
+      (effects (font (size 1.27 1.27)) hide)
+    )
+    (property "Value" "GND" (at 350.52 202.1332 0)
+      (effects (font (size 1.27 1.27)))
+    )
+    (property "Footprint" "" (at 350.393 197.739 0)
+      (effects (font (size 1.27 1.27)) hide)
+    )
+    (property "Datasheet" "" (at 350.393 197.739 0)
+      (effects (font (size 1.27 1.27)) hide)
+    )
+    (pin "1")
+    (instances
+      (project "AmigaPCI Mainboard"
+        (path "/72453515-27fe-4336-91f3-e3c8054f7767/34f2eda3-97b6-4f91-ad2d-01637d6f5405"
+          (reference "#PWR0196") (unit 1)
+        )
+      )
+      (project "2000ATX"
+        (path "/bb595301-1c72-49dc-ac6f-007419f3a7fd/00000000-0000-0000-0000-0000607c1eb7"
+          (reference "#PWR0175") (unit 1)
+        )
+      )

Commit message: Routing June 10 2023a
Parts:
- C313, C314: footprint Capacitor_SMD:CP_Elec_8x10 -> Capacitor_THT:CP_Radial_D10.0mm_P5.00mm
Connections:
- net B0: now also RN3.5 (R4.2); no longer RN3.4 (R4.1)
- net B3: now also RN3.6 (R3.2); no longer RN3.3 (R3.1)
- net G3: now also RN3.7 (R2.2); no longer RN3.2 (R2.1)
- net R3: now also RN3.8 (R1.2); no longer RN3.1 (R1.1)
- net at CN301.23: now also RN3.4 (R4.1); no longer RN3.5 (R4.2)
- net at CN301.25: now also RN3.3 (R3.1); no longer RN3.6 (R3.2)
- net at CN301.27: now also RN3.2 (R2.1); no longer RN3.7 (R2.2)
- net at CN301.29: now also RN3.1 (R1.1); no longer RN3.8 (R1.2)
Other:
- moved on the sheet: RN3
Changed lines of the file:
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@@
       (effects (font (size 1.27 1.27)))
     )
-    (property "Footprint" "Capacitor_SMD:CP_Elec_8x10" (at 386.588 104.14 0)
+    (property "Footprint" "Capacitor_THT:CP_Radial_D10.0mm_P5.00mm" (at 386.588 104.14 0)
       (effects (font (size 1.27 1.27)) hide)
     )
@@
     )
   )
-  (symbol (lib_id "Device:R_Pack04") (at 272.669 81.915 180) (unit 1)
+  (symbol (lib_id "Device:R_Pack04") (at 272.669 81.915 0) (mirror y) (unit 1)
     (in_bom yes) (on_board yes) (dnp no)
     (property "Reference" "RN3" (at 265.938 81.915 90)
@@
       (effects (font (size 1.27 1.27)))
     )
-    (property "Footprint" "Capacitor_SMD:CP_Elec_8x10" (at 376.428 104.14 0)
-      (effects (font (size 1.27 1.27)) hide)
-    )
+    (property "Footprint" "Capacitor_THT:CP_Radial_D10.0mm_P5.00mm" (at 376.428 104.14 0)
+      (effects (font (size 1.27 1.27)) hide)
+    )

Commit message: Routing June 10 2023b
Parts:
- removed C306, C307, C308, C309: 0.1uF, Capacitor_SMD:C_0603_1608Metric, symbol Device:C_Small
- removed CN303: Raspberry_Pi_Zero, Connector_PinSocket_2.54mm:PinSocket_2x20_P2.54mm_Vertical, symbol Connector:Raspberry_Pi_2_3
- removed J301: PI_BUTTON, Connector_PinHeader_2.54mm:PinHeader_1x02_P2.54mm_Vertical, symbol Connector:Conn_01x02_Pin
- removed JP302: DENISE(1)/S.DENISE(3), Connector_PinHeader_2.54mm:PinHeader_1x03_P2.54mm_Vertical, symbol Jumper:Jumper_3_Bridged12
- removed R303: 3.3k, Resistor_SMD:R_0603_1608Metric, symbol Device:R_Small
- removed RN302: 4.7K, Resistor_THT:R_Array_SIP5, symbol Device:R_Network04
- removed U303, U304: 74LVC574, Package_SO:TSSOP-20_4.4x6.5mm_P0.65mm, symbol 74xx:74LS574
- removed U307: 74LVC86, Package_SO:TSSOP-14_4.4x5mm_P0.65mm, symbol 74xx:74LS86
- RN301: footprint Resistor_THT:R_Array_SIP5 -> Resistor_THT:R_Array_SIP9; symbol Device:R_Network04 -> Device:R_Network08
- renumbered RN303 to RN302
Connections:
- net BLU0: now also RN301.9 (R8); no longer RN301.2 (R1)
- net BLU1: now also RN301.2 (R1); no longer RN301.3 (R2)
- net BLU2: now also RN301.3 (R2); no longer RN301.4 (R3)
- net BLU3: now also RN301.4 (R3); no longer RN301.5 (R4)
- net GRN0: now also RN301.8 (R7)
- net GRN1: now also RN301.7 (R6)
- net GRN2: now also RN301.6 (R5)
- net GRN3: now also RN301.5 (R4)
- net RED0: now also RN302.4 (R3); no longer RN302.5 (R4)
- net RED1: now also RN302.5 (R4); no longer RN302.4 (R3)
- net RED2: now also RN302.2 (R1); no longer RN302.3 (R2)
- net RED3: now also RN302.3 (R2); no longer RN302.2 (R1)
- no-connect marks 27 -> 11
Other:
- note removed: "RGB2HDMI"

Commit message: Routing June 24 2023
Parts:
- removed C317: 0.1uF, Capacitor_SMD:C_0603_1608Metric, symbol Device:C_Small
- removed U201: 74LVC1G74, Package_SO:TSSOP-8_3x3mm_P0.65mm, symbol 74xGxx:74AUC1G74
Connections:
- net _C4 renamed C4
- no-connect marks 11 -> 10
Changed lines of the file:
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@@
   (junction (at 75.565 49.784) (diameter 0) (color 0 0 0 0)
   )
-  (junction (at 338.963 50.8) (diameter 0) (color 0 0 0 0)
-  )
   (junction (at 193.675 136.017) (diameter 0) (color 0 0 0 0)
   )
@@
   (junction (at 231.648 42.926) (diameter 0) (color 0 0 0 0)
   )
-  (junction (at 333.883 80.772) (diameter 0) (color 0 0 0 0)
-  )
   (junction (at 225.044 136.017) (diameter 0) (color 0 0 0 0)
   )
@@
   (junction (at 381.508 109.22) (diameter 0) (color 0 0 0 0)
   )
-  (junction (at 333.883 50.8) (diameter 0) (color 0 0 0 0)
-  )
   (junction (at 80.01 141.224) (diameter 0) (color 0 0 0 0)
   )
@@
   (junction (at 135.255 117.094) (diameter 0) (color 0 0 0 0)
   )
-  (junction (at 338.963 80.772) (diameter 0) (color 0 0 0 0)
-  )
   (junction (at 221.488 42.926) (diameter 0) (color 0 0 0 0)
   )
@@
   )
   (no_connect (at 212.979 104.394))
-  (no_connect (at 323.723 71.12))
   (no_connect (at 210.439 106.934))
   (no_connect (at 354.203 169.799))
@@
     (stroke (width 0) (type default))
   )
-  (wire (pts (xy 356.362 82.55) (xy 338.963 82.55))
-    (stroke (width 0) (type default))
-  )
   (wire (pts (xy 297.688 54.356) (xy 297.688 31.496))
     (stroke (width 0) (type default))
@@
     (stroke (width 0) (type default))
   )
-  (wire (pts (xy 338.963 50.8) (xy 356.362 50.8))
-    (stroke (width 0) (type default))
-  )
   (wire (pts (xy 370.713 153.67) (xy 370.713 158.369))
     (stroke (width 0) (type default))
   )
-  (wire (pts (xy 256.159 60.96) (xy 256.159 106.934))
+  (wire (pts (xy 256.159 82.931) (xy 256.159 106.934))
     (stroke (width 0) (type default))
   )
@@
     (stroke (width 0) (type default))
   )
-  (wire (pts (xy 323.723 60.96) (xy 256.159 60.96))
-    (stroke (width 0) (type default))
-  )
   (wire (pts (xy 102.87 105.664) (xy 107.315 105.664))
     (stroke (width 0) (type default))
@@
     (stroke (width 0) (type default))
   )
-  (wire (pts (xy 338.963 80.772) (xy 338.963 78.74))
-    (stroke (width 0) (type default))
-  )
   (wire (pts (xy 377.063 149.86) (xy 391.668 149.86))
     (stroke (width 0) (type default))
@@
     (stroke (width 0) (type default))
   )
-  (wire (pts (xy 338.963 82.55) (xy 338.963 80.772))
-    (stroke (width 0) (type default))
-  )
   (wire (pts (xy 284.988 51.816) (xy 284.988 31.496))
     (stroke (width 0) (type default))
@@
     (stroke (width 0) (type default))
   )
-  (wire (pts (xy 333.883 48.387) (xy 333.883 50.8))
-    (stroke (width 0) (type default))
-  )
   (wire (pts (xy 233.299 104.394) (xy 233.299 94.234))
     (stroke (width 0) (type default))
@@
     (stroke (width 0) (type default))
   )
-  (wire (pts (xy 349.123 71.12) (xy 355.219 71.12))
-    (stroke (width 0) (type default))
-  )
   (wire (pts (xy 277.368 54.356) (xy 277.368 31.496))
     (stroke (width 0) (type default))
@@
     (stroke (width 0) (type default))
   )
-  (wire (pts (xy 356.362 50.8) (xy 356.362 82.55))
-    (stroke (width 0) (type default))
-  )
   (bus (pts (xy 34.925 54.864) (xy 37.465 54.864))
     (stroke (width 0) (type default))
@@
     (stroke (width 0) (type default))
   )
-  (wire (pts (xy 333.883 80.772) (xy 333.883 78.74))
-    (stroke (width 0) (type default))
-  )
   (wire (pts (xy 259.588 51.816) (xy 259.588 31.496))
     (stroke (width 0) (type default))
@@
     (stroke (width 0) (type default))
   )
-  (wire (pts (xy 338.963 53.34) (xy 338.963 50.8))
-    (stroke (width 0) (type default))
-  )
-  (wire (pts (xy 333.883 82.55) (xy 333.883 80.772))
-    (stroke (width 0) (type default))
-  )
   (wire (pts (xy 214.122 136.017) (xy 214.122 140.335))
     (stroke (width 0) (type default))
@@
     (stroke (width 0) (type default))
   )
-  (wire (pts (xy 338.963 50.8) (xy 333.883 50.8))
-    (stroke (width 0) (type default))
-  )
   (wire (pts (xy 85.09 118.364) (xy 85.09 150.495))
     (stroke (width 0) (type default))
@@
     (stroke (width 0) (type default))
   )
-  (wire (pts (xy 333.883 50.8) (xy 333.883 53.34))
-    (stroke (width 0) (type default))
-  )
   (wire (pts (xy 376.428 109.22) (xy 376.428 106.68))
     (stroke (width 0) (type default))
@@
     (stroke (width 0) (type default))
   )
-  (wire (pts (xy 349.123 60.96) (xy 355.219 60.96))
-    (stroke (width 0) (type default))
-  )
   (wire (pts (xy 77.47 143.764) (xy 77.47 150.495))
     (stroke (width 0) (type default))
@@
     (effects (font (size 1.2954 1.2954)) (justify left bottom))
   )
-  (label "VCDAC" (at 355.219 71.12 180) (fields_autoplaced)
-    (effects (font (size 1.27 1.27)) (justify right bottom))
-  )
   (label "B3" (at 272.669 70.866 270) (fields_autoplaced)
     (effects (font (size 1.27 1.27)) (justify right bottom))
@@
     (effects (font (size 1.27 1.27)) (justify left bottom))
   )
-  (label "_C4" (at 323.723 60.96 180) (fields_autoplaced)
-    (effects (font (size 1.27 1.27)) (justify right bottom))
-  )
   (label "G0" (at 153.035 132.334 180) (fields_autoplaced)
     (effects (font (size 1.27 1.27)) (justify right bottom))
@@
     (effects (font (size 1.27 1.27)) (justify left bottom))
   )
-  (label "_VC3" (at 355.219 60.96 180) (fields_autoplaced)
-    (effects (font (size 1.27 1.27)) (justify right bottom))
-  )
   (label "G1" (at 384.048 67.31 180) (fields_autoplaced)
     (effects (font (size 1.1938 1.1938)) (justify right bottom))
@@
     )
   )
+  (global_label "C4" (shape input) (at 256.159 82.931 90) (fields_autoplaced)
+    (effects (font (size 1.27 1.27)) (justify left))
+    (property "Intersheetrefs" "${INTERSHEET_REFS}" (at 256.159 77.5457 90)
+      (effects (font (size 1.27 1.27)) (justify left))
+    )
+  )
   (global_label "M0H" (shape output) (at 89.535 59.944 0) (fields_autoplaced)
     (effects (font (size 1.27 1.27)) (justify left))
@@
     )
   )
-  (symbol (lib_id "74xGxx:74AUC1G74") (at 336.423 66.04 0) (mirror y) (unit 1)
-    (in_bom yes) (on_board yes) (dnp no)
-    (property "Reference" "U201" (at 336.296 64.881 0)
-      (effects (font (size 1.27 1.27)))
-    )
-    (property "Value" "74LVC1G74" (at 336.296 66.802 0)
-      (effects (font (size 1.27 1.27)))
-    )
-    (property "Footprint" "Package_SO:TSSOP-8_3x3mm_P0.65mm" (at 336.423 66.04 0)
-      (effects (font (size 1.27 1.27)) hide)
-    )
-    (property "Datasheet" "https://assets.nexperia.com/documents/data-sheet/74LVC1G74.pdf" (at 336.423 66.04 0)
-      (effects (font (size 1.27 1.27)) hide)
-    )
-    (pin "1")
-    (pin "2")
-    (pin "3")
-    (pin "4")
-    (pin "5")
-    (pin "6")
-    (pin "7")
-    (pin "8")
-    (instances
-      (project "AmigaPCI Mainboard"
-        (path "/72453515-27fe-4336-91f3-e3c8054f7767/d671396a-959f-409b-8612-87cb620c51cb"
-          (reference "U201") (unit 1)
-        )
-        (path "/72453515-27fe-4336-91f3-e3c8054f7767/34f2eda3-97b6-4f91-ad2d-01637d6f5405"
-          (reference "U306") (unit 1)
-        )
-      )
-    )
-  )
-  (symbol (lib_id "power:GND") (at 333.883 82.55 0) (unit 1)
-    (in_bom yes) (on_board yes) (dnp no) (fields_autoplaced)
-    (property "Reference" "#PWR0242" (at 333.883 88.9 0)
-      (effects (font (size 1.27 1.27)) hide)
-    )
-    (property "Value" "GND" (at 333.883 86.6855 0)
-      (effects (font (size 1.27 1.27)))
-    )
-    (property "Footprint" "" (at 333.883 82.55 0)
-      (effects (font (size 1.27 1.27)) hide)
-    )
-    (property "Datasheet" "" (at 333.883 82.55 0)
-      (effects (font (size 1.27 1.27)) hide)
-    )
-    (pin "1")
-    (instances
-      (project "AmigaPCI Mainboard"
-        (path "/72453515-27fe-4336-91f3-e3c8054f7767/34f2eda3-97b6-4f91-ad2d-01637d6f5405"
-          (reference "#PWR0242") (unit 1)
-        )
-      )
-    )
-  )
   (symbol (lib_id "power:-5V") (at 286.639 84.074 0) (unit 1)
     (in_bom yes) (on_board yes) (dnp no)
@@
     )
   )
-  (symbol (lib_id "power:+5V") (at 333.883 48.387 0) (unit 1)
-    (in_bom yes) (on_board yes) (dnp no) (fields_autoplaced)
-    (property "Reference" "#PWR054" (at 333.883 52.197 0)
-      (effects (font (size 1.27 1.27)) hide)
-    )
-    (property "Value" "+5V" (at 333.883 44.8851 0)
-      (effects (font (size 1.27 1.27)))
-    )
-    (property "Footprint" "" (at 333.883 48.387 0)
-      (effects (font (size 1.27 1.27)) hide)
-    )
-    (property "Datasheet" "" (at 333.883 48.387 0)
-      (effects (font (size 1.27 1.27)) hide)
-    )
-    (pin "1")
-    (instances
-      (project "AmigaPCI Mainboard"
-        (path "/72453515-27fe-4336-91f3-e3c8054f7767/34f2eda3-97b6-4f91-ad2d-01637d6f5405"
-          (reference "#PWR054") (unit 1)
-        )
-      )
-    )
-  )
   (symbol (lib_id "Amiga-Library:+VID") (at 367.538 95.25 0) (unit 1)
     (in_bom yes) (on_board yes) (dnp no)
@@
         )
       )
-    )
-  )
-  (symbol (lib_id "Device:C_Small") (at 336.423 80.772 90) (unit 1)
-    (in_bom yes) (on_board yes) (dnp no)
-    (property "Reference" "C317" (at 343.027 77.581 90)
-      (effects (font (size 1.27 1.27)))
-    )
-    (property "Value" "0.1uF" (at 343.027 79.502 90)
-      (effects (font (size 1.27 1.27)))
-    )
-    (property "Footprint" "Capacitor_SMD:C_0603_1608Metric" (at 336.423 80.772 0)
-      (effects (font (size 1.27 1.27)) hide)
-    )
-    (property "Datasheet" "~" (at 336.423 80.772 0)
-      (effects (font (size 1.27 1.27)) hide)
-    )
-    (pin "1")
-    (pin "2")
-    (instances
-      (project "AmigaPCI Mainboard"
-        (path "/72453515-27fe-4336-91f3-e3c8054f7767/34f2eda3-97b6-4f91-ad2d-01637d6f5405"
-          (reference "C317") (unit 1)
-        )
-      )

Commit message: Updated Schematic 12-DEC-2023
Connections:
- net _LPEN renamed _FIR1
Other:
- note removed: "VIDIOT"
Changed lines of the file:
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@@
     (effects (font (size 6 6) (thickness 1.2) bold) (justify left bottom))
-  )
-  (text "VIDIOT" (at 366.268 35.306 0)
-    (effects (font (size 2.9972 2.9972)) (justify left bottom))
   )
   (label "DRD4" (at 47.625 85.344 180) (fields_autoplaced)
@@
     )
   )
-  (global_label "_LPEN" (shape input) (at 257.048 31.496 90) (fields_autoplaced)
-    (effects (font (size 1.27 1.27)) (justify left))
-    (property "Intersheetrefs" "${INTERSHEET_REFS}" (at 257.048 22.845 90)
-      (effects (font (size 1.27 1.27)) (justify left))
-    )
+  (global_label "_FIR1" (shape input) (at 257.048 31.496 90) (fields_autoplaced)
+    (effects (font (size 1.27 1.27)) (justify left))
+    (property "Intersheetrefs" "${INTERSHEET_REFS}" (at 257.048 23.3703 90)
+      (effects (font (size 1.27 1.27)) (justify left))
+    )

Commit message: Schematic and PCB Updates 13-DEC-2023
Parts:
- removed RN300: 1k, Resistor_THT:R_Array_SIP6, symbol Device:R_Network05
- added R303, R309, R311, R312: 1k, Resistor_SMD:R_0603_1608Metric, symbol Device:R_Small
Connections:
- net GND: now also R303.1, R309.1, R311.1, R312.1
- net M0H: now also R311.2
- net M0V: now also R309.2
- net M1H: now also R303.2
- net M1V: now also R312.2
- net 7M renamed CLK7
- no-connect marks 10 -> 9
