File: KiCAD/AmigaPCI Mainboard-KiCAD/IDE.kicad_sch (KiCad schematic)
At the start: 43 parts, among them CN20 SECONDARY IDE, CN227 JTAG/SWD, CN5 PRIMARY IDE, CN6 IDE_LED, J202 SYSTEM CLK, J905 CABLE SELECT, U2 XC9572XL-VQ64, U220 74AHCT08, U900 74HCT245, U901 74HCT245, U902 74HCT245, U904 74HCT245, U905 74FCT646, U906 74FCT646

Commit message: Schematic and PCB Updates 13-DEC-2023
Connections:
- net 28M renamed CLK28
Changed lines of the file:
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@@
     (effects (font (size 1.27 1.27)) (justify left bottom))
   )
-  (label "28M" (at 220.218 198.628 0) (fields_autoplaced)
+  (label "CLK28" (at 220.218 198.628 0) (fields_autoplaced)
     (effects (font (size 1.27 1.27)) (justify left bottom))
   )

Commit message: Schematic and Routing 14-DEC-2023
Connections:
- net _IDEROMEN is gone; now on net _LDS: U2.12 (P12)
- net _LDS: no longer U2.13 (P13)
- net _UDS: now also U2.13 (P13); no longer U2.15 (I/O/GCK1)
- new net CLK40: U2.15 (I/O/GCK1)
Changed lines of the file:
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@@
-    )
-  )
-  (global_label "_IDEROMEN" (shape output) (at 234.696 168.148 180) (fields_autoplaced)
-    (effects (font (size 1.27 1.27)) (justify right))
-    (property "Intersheetrefs" "${INTERSHEET_REFS}" (at 221.2674 168.148 0)
-      (effects (font (size 1.27 1.27)) (justify right))
     )
   )
@@
     (property "Intersheetrefs" "${INTERSHEET_REFS}" (at 297.449 188.468 0)
       (effects (font (size 1.27 1.27)) (justify left))
+    )
+  )
+  (global_label "CLK40" (shape input) (at 234.696 173.228 180) (fields_autoplaced)
+    (effects (font (size 1.27 1.27)) (justify right))
+    (property "Intersheetrefs" "${INTERSHEET_REFS}" (at 225.7237 173.228 0)
+      (effects (font (size 1.27 1.27)) (justify right))
     )
   )
@@
     )
   )
-  (global_label "_LDS" (shape output) (at 234.696 170.688 180) (fields_autoplaced)
+  (global_label "_LDS" (shape output) (at 234.696 168.148 180) (fields_autoplaced)
     (effects (font (size 1.27 1.27)) (justify right))
-    (property "Intersheetrefs" "${INTERSHEET_REFS}" (at 227.315 170.688 0)
+    (property "Intersheetrefs" "${INTERSHEET_REFS}" (at 227.315 168.148 0)
       (effects (font (size 1.27 1.27)) (justify right))
     )
@@
     )
   )
-  (global_label "_UDS" (shape output) (at 234.696 173.228 180) (fields_autoplaced)
+  (global_label "_UDS" (shape output) (at 234.696 170.688 180) (fields_autoplaced)
     (effects (font (size 1.27 1.27)) (justify right))
-    (property "Intersheetrefs" "${INTERSHEET_REFS}" (at 227.0126 173.228 0)
+    (property "Intersheetrefs" "${INTERSHEET_REFS}" (at 227.0126 170.688 0)
       (effects (font (size 1.27 1.27)) (justify right))
     )

Commit message: Schematic Cleanup 15-DEC-2023
Parts:
- CN20, CN5: symbol Connector_Generic:Conn_02x20_Odd_Even -> AmigaPCI-Symbols:Conn_02x20_IDE
- U900, U901, U902, U904: symbol N2630:74HCT245 -> AmigaPCI-Symbols:74LVC245

Commit message: Routing 17-DEC-2023
Connections:
- net _IDEEN: now reaches U2.63 (P63)
Changed lines of the file:
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@@
+    (stroke (width 0) (type default))
+  )
+  (wire (pts (xy 234.442 221.488) (xy 241.3 221.488))
     (stroke (width 0) (type default))
   )
@@
       (effects (font (size 1.27 1.27)) (justify right))
     )
+  )
+  (global_label "_IDEEN" (shape input) (at 234.442 221.488 180) (fields_autoplaced)
+    (effects (font (size 1.27 1.27)) (justify right))
+    (property "Intersheetrefs" "${INTERSHEET_REFS}" (at 224.9859 221.488 0)
+      (effects (font (size 1.27 1.27)) (justify right))
+    )

Commit message: Routing 19-DEC-2023
Connections:
- net VCDAC: now also U2.1 (P1); no longer U2.17 (I/O/GCK3)
- new net CLK80: U2.17 (I/O/GCK3)
Changed lines of the file:
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@@
+    (stroke (width 0) (type default))
+  )
+  (wire (pts (xy 234.696 193.548) (xy 241.3 193.548))
     (stroke (width 0) (type default))
   )
@@
     )
   )
-  (global_label "VCDAC" (shape input) (at 234.696 178.308 180) (fields_autoplaced)
+  (global_label "CLK80" (shape input) (at 234.696 178.308 180) (fields_autoplaced)
     (effects (font (size 1.27 1.27)) (justify right))
-    (property "Intersheetrefs" "${INTERSHEET_REFS}" (at 225.803 178.308 0)
+    (property "Intersheetrefs" "${INTERSHEET_REFS}" (at 225.7237 178.308 0)
       (effects (font (size 1.27 1.27)) (justify right))
     )
@@
     )
   )
+  (global_label "VCDAC" (shape input) (at 234.696 193.548 180) (fields_autoplaced)
+    (effects (font (size 1.27 1.27)) (justify right))
+    (property "Intersheetrefs" "${INTERSHEET_REFS}" (at 225.803 193.548 0)
+      (effects (font (size 1.27 1.27)) (justify right))
+    )
+  )

Commit message: Routing 21-DEC-2023
Connections:
- net _IDELATCH: now also U2.51 (P51); no longer U2.58 (P58)
Changed lines of the file:
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@@
     (stroke (width 0) (type default))
   )
-  (wire (pts (xy 234.696 208.788) (xy 241.3 208.788))
+  (wire (pts (xy 288.544 213.868) (xy 281.94 213.868))
     (stroke (width 0) (type default))
   )
@@
     )
   )
-  (global_label "_IDELATCH" (shape output) (at 234.696 208.788 180) (fields_autoplaced)
-    (effects (font (size 1.27 1.27)) (justify right))
-    (property "Intersheetrefs" "${INTERSHEET_REFS}" (at 222.114 208.788 0)
-      (effects (font (size 1.27 1.27)) (justify right))
-    )
-  )
+  (global_label "_IDELATCH" (shape output) (at 288.544 213.868 0) (fields_autoplaced)
+    (effects (font (size 1.27 1.27)) (justify left))
+    (property "Intersheetrefs" "${INTERSHEET_REFS}" (at 301.2054 213.868 0)
+      (effects (font (size 1.27 1.27)) (justify left))
+    )
+  )

Commit message: Routing 23-DEC-2023
Parts:
- removed J905 (x2): CABLE SELECT, Connector_PinHeader_2.54mm:PinHeader_1x02_P2.54mm_Vertical, symbol Jumper:Jumper_2_Open
- added J901: ULTRA MODE, Connector_PinHeader_2.54mm:PinHeader_2x02_P2.54mm_Vertical, symbol Connector_Generic:Conn_02x02_Odd_Even
- added R950 (x2): 1k, Resistor_SMD:R_0603_1608Metric, symbol Device:R
- CN6: value IDE_LED -> IDE LED
Connections:
- net CSELP is gone; now on net GND: CN5.28 (Pin_28)
- net CSELS is gone; now on net GND: CN20.28 (Pin_28)
- net +3.3V: now also R950.2, R950.2
- net GND: now also J901.2 (Pin_2), J901.4 (Pin_4)
- net _IDELATCH: now also U2.50 (P50); no longer U2.51 (P51)
- net ULTRA_S: now reaches U2.52 (P52)
- net ULTRA_S: now also J901.3 (Pin_3), R950.1
- net PIO_P0: now reaches U2.57 (P57)
- net PIO_P1: now reaches U2.58 (P58)
- net PIO_P2: now reaches U2.59 (P59)
- net PIO_S0: now reaches U2.60 (P60)
- net PIO_S1: now reaches U2.61 (P61)
- net PIO_S2: now reaches U2.62 (P62)
- new net ULTRA_P: J901.1 (Pin_1), R950.1, U2.51 (P51)
- no-connect marks 24 -> 28
Other:
- note added: "DURING WRITE CYCLES, ALL DATA IS REAL-TIME. FOR THE FIRST WRITE COMMAND, D16..31 IS ENABLED. FOR THE SECOND WRITE COMMAND, D0..15 IS ENABLED. DURING READ CYCLES, D16..31 IS LATCHED AFTER THE FIRST READ COMMAND FROM THE IDE DEVICE. THE SECOND READ FROM THE IDE DEVICE DRIVES D0..15 LIVE. THE DATA IS THEN LATCHED BY THE MC68040."
- note removed: "DURING WRITE CYCLES, ALL DATA IS REAL-TIME. FOR THE FIRST WRITE COMMAND, D16..31 IS ENABLED. FOR THE SECOND WRITE COMMAND, D0..15 IS ENABLED. DURING READ CYCLES, D16..31 IS LATCHED AFTER THE FIRST READ COMMAND FROM THE IDE DEVICE. THE SECOND READ FROM THE IDE DEVICE DRIVES D0..15 LIVE. THE DATA IS THEN LATCH BY THE MC68040."

Commit message: Silkscreen Cleanup 24-DEC-2023
Parts:
- R903: value 2.7K -> 2k7
- R924, R950: value 82 -> 82R
Changed lines of the file:
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@@
       (effects (font (size 1.27 1.27)) (justify left))
     )
-    (property "Value" "2.7K" (at 77.343 242.062 90)
+    (property "Value" "2k7" (at 77.343 242.062 90)
       (effects (font (size 1.27 1.27)) (justify left))
     )
@@
       (effects (font (size 1.27 1.27)) (justify left))
     )
-    (property "Value" "82" (at 146.05 221.996 90)
+    (property "Value" "82R" (at 146.05 221.996 90)
       (effects (font (size 1.27 1.27)) (justify left))
     )
@@
       (effects (font (size 1.27 1.27)) (justify left))
     )
-    (property "Value" "82" (at 66.294 221.996 90)
-      (effects (font (size 1.27 1.27)) (justify left))
-    )
+    (property "Value" "82R" (at 66.294 221.996 90)
+      (effects (font (size 1.27 1.27)) (justify left))
+    )
