File: KiCAD/AmigaPCI Mainboard-KiCAD/clocks.kicad_sch (KiCad schematic)
At the start: 30 parts, among them CN201 I2C, U108 74AHCT04, U201 Si5351A-B-GM, U210 AT27C4096, U211 AT27C4096, U219 74HCT04, U906 AT27C1024, U907 AT27C1024, Y3 25MHz

Commit message: Schematic and Routing 14-DEC-2023
Parts:
- removed C903, C907: 0.1uF, Capacitor_SMD:C_0603_1608Metric, symbol Device:C_Small
- removed U210, U211 (x3): AT27C4096, Package_LCC:PLCC-44_SMD-Socket, symbol AmigaPCI-Symbols:AT27C4096-PLCC
- removed U906, U907: AT27C1024, Package_LCC:PLCC-44_SMD-Socket, symbol AmigaPCI-Symbols:AT27C4096-PLCC
- added U210, U211: AT27C4096, Package_DIP:DIP-40_W16.51mm_SMDSocket_LongPads, symbol AmigaPCI-Symbols:AT27C4096
Connections:
- net +5V: now also U210.40 (Vcc), U211.40 (Vcc)
- net A10: now also U210.29 (A8), U211.29 (A8)
- net A11: now also U210.31 (A9), U211.31 (A9)
- net A12: now also U210.32 (A10), U211.32 (A10)
- net A13: now also U210.33 (A11), U211.33 (A11)
- net A14: now also U210.34 (A12), U211.34 (A12)
- net A15: now also U210.35 (A13), U211.35 (A13)
- net A16: now also U210.36 (A14), U211.36 (A14)
- net A17: now also U210.37 (A15), U211.37 (A15)
- net A18: now also U210.38 (A16), U211.38 (A16)
- net A19: now also U210.39 (A17), U211.39 (A17)
- net A2: now also U210.21 (A0), U211.21 (A0)
- net A3: now also U210.22 (A1), U211.22 (A1)
- net A4: now also U210.23 (A2), U211.23 (A2)
- net A5: now also U210.24 (A3), U211.24 (A3)
- net A6: now also U210.25 (A4), U211.25 (A4)
- net A7: now also U210.26 (A5), U211.26 (A5)
- net A8: now also U210.27 (A6), U211.27 (A6)
- net A9: now also U210.28 (A7), U211.28 (A7)
- net D0: now also U210.19 (O0)
- net D1: now also U210.18 (O1)
- net D10: now also U210.8 (O10)
- net D11: now also U210.7 (O11)
- net D12: now also U210.6 (O12)
- net D13: now also U210.5 (O13)
- net D14: now also U210.4 (O14)
- net D15: now also U210.3 (O15)
- net D16: now also U211.19 (O0)
- net D17: now also U211.18 (O1)
- net D18: now also U211.17 (O2)
- net D19: now also U211.16 (O3)
- net D2: now also U210.17 (O2)
- net D20: now also U211.15 (O4)
- net D21: now also U211.14 (O5)
- net D22: now also U211.13 (O6)
- net D23: now also U211.12 (O7)
- net D24: now also U211.10 (O8)
- net D25: now also U211.9 (O9)
- net D26: now also U211.8 (O10)
- net D27: now also U211.7 (O11)
- net D28: now also U211.6 (O12)
- net D29: now also U211.5 (O13)
- net D3: now also U210.16 (O3)
- net D30: now also U211.4 (O14)
- net D31: now also U211.3 (O15)
- net D4: now also U210.15 (O4)
- net D5: now also U210.14 (O5)
- net D6: now also U210.13 (O6)
- net D7: now also U210.12 (O7)
- net D8: now also U210.10 (O8)
- net D9: now also U210.9 (O9)
- net GND: now also U210.11 (GND), U210.2 (_CE), U210.30 (GND), U211.11 (GND), U211.2 (_CE), U211.30 (GND)
- net _ROMEN: now also U210.20 (_OE), U211.20 (_OE)
Other:
- note added: "ROM Address Mapping: $000000 - $01FFFF Kickstart $03E000 - $03FFFF IDE Autoboot (CAN WE HAVE LONG WORD WIDE AUTOBOOT ROMS?)"
- note removed: "IDE AUTOBOOT"
- note removed: "KICKSTART"
- note removed: "SWITCH TO THE Si5351A CLOCK GENERATOR! PART SI5351A-B-GTR"

Commit message: Schematic Cleanup 15-DEC-2023
Parts:
- added J400: RAM CLK, Connector_PinHeader_2.54mm:PinHeader_1x03_P2.54mm_Vertical, symbol Connector:Conn_01x03_Pin
- added J4011: INV RAM CLK, Connector_PinHeader_2.54mm:PinHeader_1x03_P2.54mm_Vertical, symbol Connector:Conn_01x03_Pin
- added unit 1 of U219
Connections:
- net CLK40: now also J400.1 (Pin_1)
- net CLK80: now also J400.3 (Pin_3)
- new net: J4011.3 (Pin_3), U219.2
- new net CLK_RAM: J4011.2 (Pin_2)
- new net RAM_SPD: J400.2 (Pin_2), J4011.1 (Pin_1), U219.1
Other:
- moved on the sheet: C719, C720, C721, C722, CN201, RN215, U201, Y3

Commit message: Routing Work 15-DEC-2023
Parts:
- renumbered J4011 to J401
Changed lines of the file:
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@@
   (symbol (lib_id "Connector:Conn_01x03_Pin") (at 127.254 122.428 90) (mirror x) (unit 1)
     (in_bom yes) (on_board yes) (dnp no)
-    (property "Reference" "J4011" (at 125.73 115.316 0)
+    (property "Reference" "J401" (at 125.73 115.316 0)
       (effects (font (size 1.27 1.27)))
     )
@@
       (project "AmigaPCI Mainboard"
         (path "/72453515-27fe-4336-91f3-e3c8054f7767/d671396a-959f-409b-8612-87cb620c51cb"
-          (reference "J4011") (unit 1)
+          (reference "J401") (unit 1)
         )
         (path "/72453515-27fe-4336-91f3-e3c8054f7767/64185471-b9ae-4a50-a046-7157e86a04d0"

Commit message: Routing 18-DEC-2023
Parts:
- U219: value 74HCT04 -> 74AHCT04
Changed lines of the file:
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@@
       (effects (font (size 1.27 1.27)) (justify left))
     )
-    (property "Value" "74HCT04" (at 367.411 158.623 90)
+    (property "Value" "74AHCT04" (at 367.411 158.623 90)
       (effects (font (size 1.27 1.27)) (justify left))
     )
@@
       (effects (font (size 1.27 1.27)))
     )
-    (property "Value" "74HCT04" (at 64.262 68.453 0)
+    (property "Value" "74AHCT04" (at 64.262 68.453 0)
       (effects (font (size 1.27 1.27)))
     )
@@
       (effects (font (size 1.27 1.27)))
     )
-    (property "Value" "74HCT04" (at 133.858 137.414 0)
+    (property "Value" "74AHCT04" (at 133.858 137.414 0)
       (effects (font (size 1.27 1.27)))
     )
@@
       (effects (font (size 1.27 1.27)))
     )
-    (property "Value" "74HCT04" (at 60.452 55.753 0)
+    (property "Value" "74AHCT04" (at 60.452 55.753 0)
       (effects (font (size 1.27 1.27)))
     )
@@
       (effects (font (size 1.27 1.27)))
     )
-    (property "Value" "74HCT04" (at 61.087 42.164 0)
-      (effects (font (size 1.27 1.27)))
-    )
+    (property "Value" "74AHCT04" (at 61.087 42.164 0)
+      (effects (font (size 1.27 1.27)))
+    )

Commit message: Routing 22-DEC-2023
Parts:
- U201: footprint Package_DFN_QFN:QFN-20-1EP_4x4mm_P0.5mm_EP2.7x2.7mm_ThermalVias -> Package_DFN_QFN:QFN-20-1EP_4x4mm_P0.5mm_EP2.7x2.7mm
Changed lines of the file:
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@@
       (effects (font (size 1.27 1.27)) (justify left))
     )
-    (property "Footprint" "Package_DFN_QFN:QFN-20-1EP_4x4mm_P0.5mm_EP2.7x2.7mm_ThermalVias" (at 64.516 200.152 0)
+    (property "Footprint" "Package_DFN_QFN:QFN-20-1EP_4x4mm_P0.5mm_EP2.7x2.7mm" (at 64.516 200.152 0)
       (effects (font (size 1.27 1.27)) hide)
     )

Commit message: Routing 23-DEC-2023
Other:
- note added: "ROM Address Mapping: $000000 - $01FFFF Kickstart $03E000 - $03FFFF IDE Autoboot"
- note added: "VIDEO CLOCK FANOUT"
- note removed: "CLOCK FANOUT"
- note removed: "ROM Address Mapping: $000000 - $01FFFF Kickstart $03E000 - $03FFFF IDE Autoboot (CAN WE HAVE LONG WORD WIDE AUTOBOOT ROMS?)"
- moved on the sheet: C135, C238, C239, C262, C719, C720, C721, C722, CN201, J400, J401, R200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

Commit message: PCB Prototype Candidate 1 21-DEC-2023
Parts:
- U210, U211: footprint Package_DIP:DIP-40_W16.51mm_SMDSocket_LongPads -> Package_DIP:DIP-40_W15.24mm_Socket
Changed lines of the file:
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@@
       (effects (font (size 1.27 1.27)))
     )
-    (property "Footprint" "Package_DIP:DIP-40_W16.51mm_SMDSocket_LongPads" (at 190.246 53.594 0)
+    (property "Footprint" "Package_DIP:DIP-40_W15.24mm_Socket" (at 190.246 53.594 0)
       (effects (font (size 1.27 1.27)) hide)
     )
@@
       (effects (font (size 1.27 1.27)) (justify left))
     )
-    (property "Footprint" "Package_DIP:DIP-40_W16.51mm_SMDSocket_LongPads" (at 41.783 214.757 0)
+    (property "Footprint" "Package_DIP:DIP-40_W15.24mm_Socket" (at 41.783 214.757 0)
       (effects (font (size 1.27 1.27)) hide)
     )
@@
       (effects (font (size 1.27 1.27)))
     )
-    (property "Footprint" "Package_DIP:DIP-40_W16.51mm_SMDSocket_LongPads" (at 232.156 53.594 0)
+    (property "Footprint" "Package_DIP:DIP-40_W15.24mm_Socket" (at 232.156 53.594 0)
       (effects (font (size 1.27 1.27)) hide)
     )
@@
       (effects (font (size 1.27 1.27)) (justify left))
     )
-    (property "Footprint" "Package_DIP:DIP-40_W16.51mm_SMDSocket_LongPads" (at 18.669 214.757 0)
-      (effects (font (size 1.27 1.27)) hide)
-    )
+    (property "Footprint" "Package_DIP:DIP-40_W15.24mm_Socket" (at 18.669 214.757 0)
+      (effects (font (size 1.27 1.27)) hide)
+    )

Commit message: Silkscreen Cleanup 24-DEC-2023
Parts:
- R200: value 22 -> 22R
Changed lines of the file:
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@@
       (effects (font (size 1.27 1.27)))
     )
-    (property "Value" "22" (at 72.644 165.1 90)
+    (property "Value" "22R" (at 72.644 165.1 90)
       (effects (font (size 1.27 1.27)))
     )
@@
       (effects (font (size 1.27 1.27)))
     )
-    (property "Value" "22" (at 72.771 178.308 90)
+    (property "Value" "22R" (at 72.771 178.308 90)
       (effects (font (size 1.27 1.27)))
     )
@@
       (effects (font (size 1.27 1.27)))
     )
-    (property "Value" "22" (at 72.517 139.065 90)
+    (property "Value" "22R" (at 72.517 139.065 90)
       (effects (font (size 1.27 1.27)))
     )
@@
       (effects (font (size 1.27 1.27)))
     )
-    (property "Value" "22" (at 72.898 190.881 90)
+    (property "Value" "22R" (at 72.898 190.881 90)
       (effects (font (size 1.27 1.27)))
     )
@@
       (effects (font (size 1.27 1.27)))
     )
-    (property "Value" "22" (at 72.517 151.638 90)
-      (effects (font (size 1.27 1.27)))
-    )
+    (property "Value" "22R" (at 72.517 151.638 90)
+      (effects (font (size 1.27 1.27)))
+    )
