File: KiCAD/AmigaPCI Mainboard-KiCAD/bcontroller.kicad_sch (KiCad schematic)
At the start: 20 parts, among them CN227 JTAG/SWD, J200 DISABLE AUTOBOOT, U6 XC95144XL-TQ144, U711 XC9572XL-VQ64

Commit message: Routing 17-DEC-2023
Connections:
- net _OVL is gone; now on net _TIP: U6.106 (P106)
- net CLKCIA: now also U6.104 (P104); no longer U6.91 (P91)
- net CONFIGED: now also U6.97 (P97); no longer U6.113 (P113)
- net CPUSPACE: now also U6.98 (P98); no longer U6.115 (P115)
- net D29: now also U6.45 (P45); no longer U6.43 (P43)
- net D31: now also U6.43 (P43); no longer U6.45 (P45)
- net OVL: now also U6.64 (P64)
- net PCISOFTMODE: now also U6.101 (P101)
- net TM0: now also U6.113 (P113)
- net TM1: now also U6.115 (P115)
- net TM2: now also U6.116 (P116)
- net TT0: now also U6.117 (P117)
- net TT1: now also U6.118 (P118)
- net _AS: now also U6.51 (P51); no longer U6.46 (P46)
- net _AVEC: now also U6.54 (P54); no longer U6.53 (P53)
- net _BEN: now also U6.100 (P100)
- net _BTNRST: now also U6.107 (P107); no longer U6.93 (P93)
- net _CIA0: now also U6.58 (P58)
- net _CIA1: now also U6.59 (P59); no longer U6.111 (P111)
- net _DBR: now also U6.49 (P49); no longer U6.48 (P48)
- net _IDEEN: now also U6.103 (P103)
- net _KBRST: now also U6.46 (P46); no longer U6.94 (P94)
- net _RAMEN: now also U6.57 (P57); no longer U6.112 (P112)
- net _REGEN: now also U6.50 (P50)
- net _RESET: now also U6.105 (P105)
- net _ROMEN: now also U6.110 (P110)
- net _RTCRD: now also U6.60 (P60)
- net _RTCWR: now also U6.61 (P61)
- net _SYSTEMRST: now also U6.112 (P112); no longer U6.92 (P92)
- net _TA: now also U6.56 (P56)
- net _TBI: now also U6.53 (P53); no longer U6.110 (P110)
- net _TCI: now also U6.102 (P102)
- net _TIP: no longer U6.52 (P52)
- net _VBEN: now also U6.111 (P111)
- net AUTOBOOT: now reaches J200.1 (Pin_1), R28.2
- new net _BLS: U6.48 (P48)
Other:
- moved on the sheet: J200, R28

Commit message: Routing 18-DEC-2023
Connections:
- net AR_W: now also U6.100 (P100); no longer U6.70 (P70)
- net AUTOBOOT: now also U6.95 (P95)
- net CONFIGED: now also U6.58 (P58); no longer U6.97 (P97)
- net CPUSPACE: now also U6.96 (P96); no longer U6.98 (P98)
- net OVL: now also U6.66 (P66); no longer U6.64 (P64)
- net PCISOFTMODE: now also U6.98 (P98); no longer U6.101 (P101)
- net _BEN: now also U6.97 (P97); no longer U6.100 (P100)
- net _BTNRST: now also U6.102 (P102); no longer U6.107 (P107)
- net _CIA0: now also U6.59 (P59); no longer U6.58 (P58)
- net _CIA1: now also U6.60 (P60); no longer U6.59 (P59)
- net _EMEN: now also U6.101 (P101); no longer U6.69 (P69)
- net _RTCRD: now also U6.61 (P61); no longer U6.60 (P60)
- net _RTCWR: now also U6.64 (P64); no longer U6.61 (P61)
- net _TCI: now also U6.52 (P52); no longer U6.102 (P102)
- net _TS: now also U6.107 (P107); no longer U6.68 (P68)
Other:
- moved on the sheet: J200, R28

Commit message: Routing 19-DEC-2023
Connections:
- net C1: now also U711.48 (P48); no longer U711.16 (I/O/GCK2)
- net C3: now also U6.74 (P74); no longer U6.30 (I/O/GCK1)
- new net CLK80: U6.30 (I/O/GCK1), U711.16 (I/O/GCK2)
- no-connect marks 1 -> 0
Other:
- note added: "U409 PROVIDES RAM AND IDE AUTOCONFIG, ADDRESS DECODE, REPLACEMENT GARY FUNCTIONS, STARTUP AND KEYBOARD RESET, AND FAST RAM CONTROLLER."
Changed lines of the file:
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@@
   (junction (at 192.024 59.69) (diameter 0) (color 0 0 0 0)
   )
-  (no_connect (at 337.566 148.082))
   (bus_entry (at 85.852 134.112) (size -2.54 -2.54)
     (stroke (width 0) (type default))
@@
     (stroke (width 0) (type default))
   )
-  (wire (pts (xy 109.982 101.092) (xy 112.776 101.092))
+  (wire (pts (xy 181.61 146.812) (xy 178.816 146.812))
     (stroke (width 0) (type default))
   )
@@
     (stroke (width 0) (type default))
   )
+  (wire (pts (xy 110.236 101.092) (xy 112.776 101.092))
+    (stroke (width 0) (type default))
+  )
   (bus (pts (xy 83.312 136.906) (xy 83.312 139.192))
     (stroke (width 0) (type default))
@@
     (stroke (width 0) (type default))
   )
+  (wire (pts (xy 288.036 117.602) (xy 296.926 117.602))
+    (stroke (width 0) (type default))
+  )
   (wire (pts (xy 110.236 159.512) (xy 112.776 159.512))
     (stroke (width 0) (type default))
@@
     (stroke (width 0) (type default))
   )
-  (wire (pts (xy 288.036 117.602) (xy 296.926 117.602))
+  (wire (pts (xy 346.202 148.082) (xy 337.566 148.082))
     (stroke (width 0) (type default))
   )
@@
   )
   (text "CHIP RAM CONTROLLER" (at 291.973 65.913 0)
+    (effects (font (size 3 3) (thickness 0.6) bold) (justify left bottom))
+  )
+  (text "U409 PROVIDES RAM AND IDE AUTOCONFIG, ADDRESS DECODE,\nREPLACEMENT GARY FUNCTIONS, STARTUP AND KEYBOARD RESET, \nAND FAST RAM CONTROLLER."
+    (at 248.412 40.894 0)
     (effects (font (size 3 3) (thickness 0.6) bold) (justify left bottom))
   )
@@
     )
   )
-  (global_label "C3" (shape input) (at 109.982 101.092 180) (fields_autoplaced)
-    (effects (font (size 1.27 1.27)) (justify right))
-    (property "Intersheetrefs" "${INTERSHEET_REFS}" (at 104.5967 101.092 0)
-      (effects (font (size 1.27 1.27)) (justify right))
+  (global_label "C3" (shape input) (at 181.61 146.812 0) (fields_autoplaced)
+    (effects (font (size 1.27 1.27)) (justify left))
+    (property "Intersheetrefs" "${INTERSHEET_REFS}" (at 186.9953 146.812 0)
+      (effects (font (size 1.27 1.27)) (justify left))
     )
   )
@@
     )
   )
-  (global_label "C1" (shape input) (at 288.036 117.602 180) (fields_autoplaced)
+  (global_label "C1" (shape input) (at 346.202 148.082 0) (fields_autoplaced)
+    (effects (font (size 1.27 1.27)) (justify left))
+    (property "Intersheetrefs" "${INTERSHEET_REFS}" (at 351.6667 148.082 0)
+      (effects (font (size 1.27 1.27)) (justify left))
+    )
+  )
+  (global_label "_CUMBE" (shape output) (at 346.202 127.762 0) (fields_autoplaced)
+    (effects (font (size 1.27 1.27)) (justify left))
+    (property "Intersheetrefs" "${INTERSHEET_REFS}" (at 356.5463 127.762 0)
+      (effects (font (size 1.27 1.27)) (justify left))
+    )
+  )
+  (global_label "CLK80" (shape input) (at 288.036 117.602 180) (fields_autoplaced)
     (effects (font (size 1.27 1.27)) (justify right))
-    (property "Intersheetrefs" "${INTERSHEET_REFS}" (at 282.6507 117.602 0)
-      (effects (font (size 1.27 1.27)) (justify right))
-    )
-  )
-  (global_label "_CUMBE" (shape output) (at 346.202 127.762 0) (fields_autoplaced)
-    (effects (font (size 1.27 1.27)) (justify left))
-    (property "Intersheetrefs" "${INTERSHEET_REFS}" (at 356.5463 127.762 0)
-      (effects (font (size 1.27 1.27)) (justify left))
+    (property "Intersheetrefs" "${INTERSHEET_REFS}" (at 279.0637 117.602 0)
+      (effects (font (size 1.27 1.27)) (justify right))
     )
   )
@@
     )
   )
+  (global_label "CLK80" (shape input) (at 110.236 101.092 180) (fields_autoplaced)
+    (effects (font (size 1.27 1.27)) (justify right))
+    (property "Intersheetrefs" "${INTERSHEET_REFS}" (at 101.2637 101.092 0)
+      (effects (font (size 1.27 1.27)) (justify right))
+    )
+  )
   (global_label "_AS" (shape output) (at 104.14 187.452 180) (fields_autoplaced)
     (effects (font (size 1.27 1.27)) (justify right))
@@
     )
   )
-  (global_label "_BLS" (shape input) (at 104.14 179.832 180) (fields_autoplaced)
+  (global_label "_BLS" (shape output) (at 104.14 179.832 180) (fields_autoplaced)
     (effects (font (size 1.27 1.27)) (justify right))
     (property "Intersheetrefs" "${INTERSHEET_REFS}" (at 96.6796 179.832 0)

Commit message: Routing 20-DEC-2023
Connections:
- net _REGEN: now also U711.49 (P49); no longer U711.64 (I/O/GSR)
- net _RESET: now also U711.64 (I/O/GSR); no longer U711.49 (P49)
- net PCISOFTMODE: no longer names the net of U6.98 (P98)
Changed lines of the file:
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@@
     )
   )
-  (global_label "_REGEN" (shape input) (at 288.036 165.862 180) (fields_autoplaced)
-    (effects (font (size 1.2954 1.2954)) (justify right))
-    (property "Intersheetrefs" "${INTERSHEET_REFS}" (at 277.7937 165.862 0)
-      (effects (font (size 1.27 1.27)) (justify right))
+  (global_label "_REGEN" (shape input) (at 346.202 150.622 0) (fields_autoplaced)
+    (effects (font (size 1.2954 1.2954)) (justify left))
+    (property "Intersheetrefs" "${INTERSHEET_REFS}" (at 356.5253 150.622 0)
+      (effects (font (size 1.27 1.27)) (justify left))
     )
   )
@@
     )
   )
-  (global_label "_RESET" (shape input) (at 346.202 150.622 0) (fields_autoplaced)
-    (effects (font (size 1.27 1.27)) (justify left))
-    (property "Intersheetrefs" "${INTERSHEET_REFS}" (at 355.8205 150.622 0)
-      (effects (font (size 1.27 1.27)) (justify left))
+  (global_label "_RESET" (shape input) (at 288.036 165.862 180) (fields_autoplaced)
+    (effects (font (size 1.27 1.27)) (justify right))
+    (property "Intersheetrefs" "${INTERSHEET_REFS}" (at 278.3381 165.862 0)
+      (effects (font (size 1.27 1.27)) (justify right))
     )
   )
@@
     )
   )
-  (global_label "PCISOFTMODE" (shape input) (at 187.452 202.692 0) (fields_autoplaced)
-    (effects (font (size 1.27 1.27)) (justify left))
-    (property "Intersheetrefs" "${INTERSHEET_REFS}" (at 203.2997 202.692 0)
-      (effects (font (size 1.27 1.27)) (justify left))
-    )
-  )

Commit message: Routing 21-DEC-2023
Connections:
- net AUTOBOOT: now also U6.96 (P96); no longer U6.95 (P95)
- net CPUSPACE: now also U6.94 (P94); no longer U6.96 (P96)
- net _BEN: now also U6.68 (P68); no longer U6.97 (P97)
Other:
- moved on the sheet: J200, R28
Changed lines of the file:
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@@
   (junction (at 168.402 46.736) (diameter 0) (color 0 0 0 0)
   )
-  (junction (at 210.566 195.072) (diameter 0) (color 0 0 0 0)
+  (junction (at 210.566 197.612) (diameter 0) (color 0 0 0 0)
   )
   (junction (at 332.232 75.946) (diameter 0) (color 0 0 0 0)
@@
     (stroke (width 0) (type default))
   )
-  (wire (pts (xy 215.9 195.072) (xy 210.566 195.072))
+  (wire (pts (xy 215.9 197.612) (xy 210.566 197.612))
     (stroke (width 0) (type default))
   )
@@
     (stroke (width 0) (type default))
   )
-  (wire (pts (xy 210.566 183.642) (xy 210.566 184.658))
+  (wire (pts (xy 210.566 186.182) (xy 210.566 187.198))
     (stroke (width 0) (type default))
   )
@@
     (stroke (width 0) (type default))
   )
-  (wire (pts (xy 187.452 197.612) (xy 178.816 197.612))
-    (stroke (width 0) (type default))
-  )
   (wire (pts (xy 153.416 46.736) (xy 150.876 46.736))
     (stroke (width 0) (type default))
@@
     (stroke (width 0) (type default))
   )
-  (wire (pts (xy 210.566 195.072) (xy 178.816 195.072))
+  (wire (pts (xy 210.566 197.612) (xy 178.816 197.612))
     (stroke (width 0) (type default))
   )
@@
     (stroke (width 0) (type default))
   )
-  (wire (pts (xy 210.566 192.278) (xy 210.566 195.072))
+  (wire (pts (xy 210.566 194.818) (xy 210.566 197.612))
     (stroke (width 0) (type default))
   )
@@
     (effects (font (size 1.27 1.27)) (justify left bottom))
   )
-  (label "AUTOBOOT" (at 210.566 195.072 180) (fields_autoplaced)
+  (label "AUTOBOOT" (at 210.566 197.612 180) (fields_autoplaced)
     (effects (font (size 1.27 1.27)) (justify right bottom))
   )
@@
     )
   )
-  (global_label "_BEN" (shape output) (at 187.452 200.152 0) (fields_autoplaced)
-    (effects (font (size 1.27 1.27)) (justify left))
-    (property "Intersheetrefs" "${INTERSHEET_REFS}" (at 195.0749 200.152 0)
+  (global_label "_BEN" (shape output) (at 187.452 98.552 0) (fields_autoplaced)
+    (effects (font (size 1.27 1.27)) (justify left))
+    (property "Intersheetrefs" "${INTERSHEET_REFS}" (at 195.0749 98.552 0)
       (effects (font (size 1.27 1.27)) (justify left))
     )
@@
     )
   )
-  (global_label "CPUSPACE" (shape output) (at 187.452 197.612 0) (fields_autoplaced)
-    (effects (font (size 1.27 1.27)) (justify left))
-    (property "Intersheetrefs" "${INTERSHEET_REFS}" (at 200.2154 197.612 0)
+  (global_label "CPUSPACE" (shape output) (at 187.452 192.532 0) (fields_autoplaced)
+    (effects (font (size 1.27 1.27)) (justify left))
+    (property "Intersheetrefs" "${INTERSHEET_REFS}" (at 200.2154 192.532 0)
       (effects (font (size 1.27 1.27)) (justify left))
     )
@@
     )
   )
-  (symbol (lib_id "power:+3.3V") (at 210.566 183.642 0) (mirror y) (unit 1)
+  (symbol (lib_id "power:+3.3V") (at 210.566 186.182 0) (mirror y) (unit 1)
     (in_bom yes) (on_board yes) (dnp no) (fields_autoplaced)
-    (property "Reference" "#PWR05" (at 210.566 187.452 0)
-      (effects (font (size 1.27 1.27)) hide)
-    )
-    (property "Value" "+3.3V" (at 210.566 180.1401 0)
+    (property "Reference" "#PWR05" (at 210.566 189.992 0)
+      (effects (font (size 1.27 1.27)) hide)
+    )
+    (property "Value" "+3.3V" (at 210.566 182.6801 0)
       (effects (font (size 1.27 1.27)))
     )
-    (property "Footprint" "" (at 210.566 183.642 0)
-      (effects (font (size 1.27 1.27)) hide)
-    )
-    (property "Datasheet" "" (at 210.566 183.642 0)
+    (property "Footprint" "" (at 210.566 186.182 0)
+      (effects (font (size 1.27 1.27)) hide)
+    )
+    (property "Datasheet" "" (at 210.566 186.182 0)
       (effects (font (size 1.27 1.27)) hide)
     )
@@
     )
   )
-  (symbol (lib_id "Device:R") (at 210.566 188.468 0) (mirror y) (unit 1)
+  (symbol (lib_id "Device:R") (at 210.566 191.008 0) (mirror y) (unit 1)
     (in_bom yes) (on_board yes) (dnp no)
-    (property "Reference" "R28" (at 208.788 187.2996 0)
-      (effects (font (size 1.27 1.27)) (justify left))
-    )
-    (property "Value" "1K" (at 208.788 189.611 0)
-      (effects (font (size 1.27 1.27)) (justify left))
-    )
-    (property "Footprint" "Resistor_SMD:R_0603_1608Metric" (at 212.344 188.468 90)
-      (effects (font (size 1.27 1.27)) hide)
-    )
-    (property "Datasheet" "~" (at 210.566 188.468 0)
+    (property "Reference" "R28" (at 208.788 189.8396 0)
+      (effects (font (size 1.27 1.27)) (justify left))
+    )
+    (property "Value" "1K" (at 208.788 192.151 0)
+      (effects (font (size 1.27 1.27)) (justify left))
+    )
+    (property "Footprint" "Resistor_SMD:R_0603_1608Metric" (at 212.344 191.008 90)
+      (effects (font (size 1.27 1.27)) hide)
+    )
+    (property "Datasheet" "~" (at 210.566 191.008 0)
       (effects (font (size 1.27 1.27)) hide)
     )
@@
     )
   )
-  (symbol (lib_id "power:GND") (at 218.44 195.072 0) (mirror y) (unit 1)
+  (symbol (lib_id "power:GND") (at 218.44 197.612 0) (mirror y) (unit 1)
     (in_bom yes) (on_board yes) (dnp no) (fields_autoplaced)
-    (property "Reference" "#PWR0243" (at 218.44 201.422 0)
-      (effects (font (size 1.27 1.27)) hide)
-    )
-    (property "Value" "GND" (at 218.44 199.2075 0)
+    (property "Reference" "#PWR0243" (at 218.44 203.962 0)
+      (effects (font (size 1.27 1.27)) hide)
+    )
+    (property "Value" "GND" (at 218.44 201.7475 0)
       (effects (font (size 1.27 1.27)))
     )
-    (property "Footprint" "" (at 218.44 195.072 0)
-      (effects (font (size 1.27 1.27)) hide)
-    )
-    (property "Datasheet" "" (at 218.44 195.072 0)
+    (property "Footprint" "" (at 218.44 197.612 0)
+      (effects (font (size 1.27 1.27)) hide)
+    )
+    (property "Datasheet" "" (at 218.44 197.612 0)
       (effects (font (size 1.27 1.27)) hide)
     )
@@
     )
   )
-  (symbol (lib_id "Connector:Conn_01x02_Pin") (at 215.9 189.992 90) (mirror x) (unit 1)
+  (symbol (lib_id "Connector:Conn_01x02_Pin") (at 215.9 192.532 90) (mirror x) (unit 1)
     (in_bom yes) (on_board yes) (dnp no)
-    (property "Reference" "J200" (at 214.884 188.849 90)
-      (effects (font (size 1.27 1.27)) (justify right))
-    )
-    (property "Value" "DISABLE AUTOBOOT" (at 215.011 187.071 90)
-      (effects (font (size 1.27 1.27)) (justify right))
-    )
-    (property "Footprint" "Connector_PinHeader_2.54mm:PinHeader_1x02_P2.54mm_Vertical" (at 215.9 189.992 0)
-      (effects (font (size 1.27 1.27)) hide)
-    )
-    (property "Datasheet" "~" (at 215.9 189.992 0)
-      (effects (font (size 1.27 1.27)) hide)
-    )
+    (property "Reference" "J200" (at 214.884 191.389 90)
+      (effects (font (size 1.27 1.27)) (justify right))
+    )
+    (property "Value" "DISABLE AUTOBOOT" (at 215.011 189.611 90)
+      (effects (font (size 1.27 1.27)) (justify right))
+    )
+    (property "Footprint" "Connector_PinHeader_2.54mm:PinHeader_1x02_P2.54mm_Vertical" (at 215.9 192.532 0)
+      (effects (font (size 1.27 1.27)) hide)
+    )
+    (property "Datasheet" "~" (at 215.9 192.532 0)
+      (effects (font (size 1.27 1.27)) hide)
+    )

Commit message: Routing 22-DEC-2023
Parts:
- removed C730, C731, C732: 0.1uF, Capacitor_SMD:C_0603_1608Metric, symbol Device:C_Small
Changed lines of the file:
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@@
-    )
-  )
-  (symbol (lib_id "Device:C_Small") (at 195.834 53.34 0) (unit 1)
-    (in_bom yes) (on_board yes) (dnp no)
-    (property "Reference" "C731" (at 197.104 59.309 90)
-      (effects (font (size 1.27 1.27)) (justify left))
-    )
-    (property "Value" "0.1uF" (at 197.104 52.578 90)
-      (effects (font (size 1.27 1.27)) (justify left))
-    )
-    (property "Footprint" "Capacitor_SMD:C_0603_1608Metric" (at 195.834 53.34 0)
-      (effects (font (size 1.27 1.27)) hide)
-    )
-    (property "Datasheet" "~" (at 195.834 53.34 0)
-      (effects (font (size 1.27 1.27)) hide)
-    )
-    (pin "1")
-    (pin "2")
-    (instances
-      (project "AmigaPCI Mainboard"
-        (path "/72453515-27fe-4336-91f3-e3c8054f7767/62a07d55-3759-49a3-8a3f-631cb4902a24"
-          (reference "C731") (unit 1)
-        )
-      )
     )
   )
@@
         (path "/72453515-27fe-4336-91f3-e3c8054f7767/62a07d55-3759-49a3-8a3f-631cb4902a24"
           (reference "C728") (unit 1)
-        )
-      )
-    )
-  )
-  (symbol (lib_id "Device:C_Small") (at 199.898 53.34 0) (unit 1)
-    (in_bom yes) (on_board yes) (dnp no)
-    (property "Reference" "C732" (at 201.168 59.309 90)
-      (effects (font (size 1.27 1.27)) (justify left))
-    )
-    (property "Value" "0.1uF" (at 201.168 52.578 90)
-      (effects (font (size 1.27 1.27)) (justify left))
-    )
-    (property "Footprint" "Capacitor_SMD:C_0603_1608Metric" (at 199.898 53.34 0)
-      (effects (font (size 1.27 1.27)) hide)
-    )
-    (property "Datasheet" "~" (at 199.898 53.34 0)
-      (effects (font (size 1.27 1.27)) hide)
-    )
-    (pin "1")
-    (pin "2")
-    (instances
-      (project "AmigaPCI Mainboard"
-        (path "/72453515-27fe-4336-91f3-e3c8054f7767/62a07d55-3759-49a3-8a3f-631cb4902a24"
-          (reference "C732") (unit 1)
         )
       )
@@
         )
       )
-    )
-  )
-  (symbol (lib_id "Device:C_Small") (at 192.024 53.34 0) (unit 1)
-    (in_bom yes) (on_board yes) (dnp no)
-    (property "Reference" "C730" (at 193.294 59.309 90)
-      (effects (font (size 1.27 1.27)) (justify left))
-    )
-    (property "Value" "0.1uF" (at 193.294 52.578 90)
-      (effects (font (size 1.27 1.27)) (justify left))
-    )
-    (property "Footprint" "Capacitor_SMD:C_0603_1608Metric" (at 192.024 53.34 0)
-      (effects (font (size 1.27 1.27)) hide)
-    )
-    (property "Datasheet" "~" (at 192.024 53.34 0)
-      (effects (font (size 1.27 1.27)) hide)
-    )
-    (pin "1")
-    (pin "2")
-    (instances
-      (project "AmigaPCI Mainboard"
-        (path "/72453515-27fe-4336-91f3-e3c8054f7767/62a07d55-3759-49a3-8a3f-631cb4902a24"
-          (reference "C730") (unit 1)
-        )
-      )

Commit message: Routing 23-DEC-2023
Connections:
- net CPUSPACE: now also U6.79 (P79); no longer U6.94 (P94)
- net PIO_P0: now reaches U6.80 (P80)
- net PIO_P1: now reaches U6.81 (P81)
- net PIO_P2: now reaches U6.82 (P82)
- net PIO_S0: now reaches U6.83 (P83)
- net PIO_S1: now reaches U6.85 (P85)
- net PIO_S2: now reaches U6.86 (P86)
Changed lines of the file:
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@@
+    )
+  )
+  (global_label "PIO_S2" (shape output) (at 191.008 174.752 0) (fields_autoplaced)
+    (effects (font (size 1.27 1.27)) (justify left))
+    (property "Intersheetrefs" "${INTERSHEET_REFS}" (at 200.5851 174.752 0)
+      (effects (font (size 1.27 1.27)) (justify left))
     )
   )
@@
     )
   )
+  (global_label "PIO_S0" (shape output) (at 191.008 169.672 0) (fields_autoplaced)
+    (effects (font (size 1.27 1.27)) (justify left))
+    (property "Intersheetrefs" "${INTERSHEET_REFS}" (at 200.5851 169.672 0)
+      (effects (font (size 1.27 1.27)) (justify left))
+    )
+  )
   (global_label "C3" (shape input) (at 181.61 146.812 0) (fields_autoplaced)
     (effects (font (size 1.27 1.27)) (justify left))
@@
     (property "Intersheetrefs" "${INTERSHEET_REFS}" (at 98.0895 192.532 0)
       (effects (font (size 1.27 1.27)) (justify right))
+    )
+  )
+  (global_label "PIO_P0" (shape output) (at 191.008 162.052 0) (fields_autoplaced)
+    (effects (font (size 1.27 1.27)) (justify left))
+    (property "Intersheetrefs" "${INTERSHEET_REFS}" (at 200.6456 162.052 0)
+      (effects (font (size 1.27 1.27)) (justify left))
     )
   )
@@
     )
   )
+  (global_label "PIO_S1" (shape output) (at 191.008 172.212 0) (fields_autoplaced)
+    (effects (font (size 1.27 1.27)) (justify left))
+    (property "Intersheetrefs" "${INTERSHEET_REFS}" (at 200.5851 172.212 0)
+      (effects (font (size 1.27 1.27)) (justify left))
+    )
+  )
   (global_label "_BEN" (shape output) (at 187.452 98.552 0) (fields_autoplaced)
     (effects (font (size 1.27 1.27)) (justify left))
@@
     )
   )
-  (global_label "CPUSPACE" (shape output) (at 187.452 192.532 0) (fields_autoplaced)
-    (effects (font (size 1.27 1.27)) (justify left))
-    (property "Intersheetrefs" "${INTERSHEET_REFS}" (at 200.2154 192.532 0)
+  (global_label "CPUSPACE" (shape output) (at 191.008 159.512 0) (fields_autoplaced)
+    (effects (font (size 1.27 1.27)) (justify left))
+    (property "Intersheetrefs" "${INTERSHEET_REFS}" (at 203.7714 159.512 0)
       (effects (font (size 1.27 1.27)) (justify left))
     )
@@
     )
   )
+  (global_label "PIO_P1" (shape output) (at 191.008 164.592 0) (fields_autoplaced)
+    (effects (font (size 1.27 1.27)) (justify left))
+    (property "Intersheetrefs" "${INTERSHEET_REFS}" (at 200.6456 164.592 0)
+      (effects (font (size 1.27 1.27)) (justify left))
+    )
+  )
   (global_label "_RTCWR" (shape output) (at 187.452 93.472 0) (fields_autoplaced)
     (effects (font (size 1.27 1.27)) (justify left))
@@
     )
   )
+  (global_label "PIO_P2" (shape output) (at 191.008 167.132 0) (fields_autoplaced)
+    (effects (font (size 1.27 1.27)) (justify left))
+    (property "Intersheetrefs" "${INTERSHEET_REFS}" (at 200.6456 167.132 0)
+      (effects (font (size 1.27 1.27)) (justify left))
+    )
+  )

Commit message: PCB Prototype Candidate 2 24-DEC-2023
Parts:
- R28: value 1K -> 1k
Changed lines of the file:
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@@
       (effects (font (size 1.27 1.27)) (justify left))
     )
-    (property "Value" "1K" (at 208.788 192.151 0)
+    (property "Value" "1k" (at 208.788 192.151 0)
       (effects (font (size 1.27 1.27)) (justify left))
     )
