File: KiCAD/AmigaPCI Mainboard-KiCAD/AmigaPCI Mainboard.kicad_sch (KiCad schematic)
At the start: 0 parts

Commit message: KiCAD Schematic Update
Other:
- sheet Clocks and PCI Buffers: file gary.kicad_sch -> clocks.kicad_sch
Changed lines of the file:
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@@
       (effects (font (size 1.27 1.27)) (justify left bottom))
     )
-    (property "Sheetfile" "gary.kicad_sch" (at 172.847 40.9706 0)
+    (property "Sheetfile" "clocks.kicad_sch" (at 172.847 40.9706 0)
       (effects (font (size 1.27 1.27)) (justify left top))
     )

Commit message: IDE Timing and Schematic
Other:
- added sheet IDE Interface (IDE.kicad_sch)

Commit message: Schematic Cleanup
Other:
- note added: "100 = PCI BUS 200 = CPU AND CHIPSET 300 = VIDEO 400 = FAST RAM 500 = AUDIO 600 = POWER 700 = CHIPSET RAM 900 = IDE"
- note removed: "100 = PCI BUS 200 = CPU AND CHIPSET 300 = VIDEO 400 = FAST RAM 500 = AUDIO 700 = CHIPSET RAM 900 = IDE"
Changed lines of the file:
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@@
     )
   )
-  (text "100 = PCI BUS\n200 = CPU AND CHIPSET\n300 = VIDEO\n400 = FAST RAM\n500 = AUDIO\n700 = CHIPSET RAM\n900 = IDE"
+  (text "100 = PCI BUS\n200 = CPU AND CHIPSET\n300 = VIDEO\n400 = FAST RAM\n500 = AUDIO\n600 = POWER\n700 = CHIPSET RAM\n900 = IDE"
     (at 162.052 152.908 0)
     (effects (font (size 3 3) bold) (justify left bottom))

Commit message: Schematic Cleanup 15-DEC-2023
Other:
- note added: "DESIGNED WITH KiCAD REV 7"
Changed lines of the file:
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@@
     (effects (font (size 3 3) bold) (justify left bottom))
+  )
+  (text "DESIGNED WITH KiCAD REV 7" (at 21.336 260.858 0)
+    (effects (font (size 2 2)) (justify left bottom))
   )
   (sheet (at 45.466 121.412) (size 32.258 17.272) (fields_autoplaced)
