File: KiCAD/AmigaPCI Mainboard-KiCAD/pci_level_shift.kicad_sch (KiCad schematic)
At the start: 11 parts, among them U111 74AHCT157, U112 74AHCT157, U2 74LVC245, U812 SN74LVC16T245DLR, U813 SN74LVC16T245DLR

Commit message: PCB Routing 31-JAN-2024
Parts:
- removed U2: 74LVC245, Package_SO:TSSOP-20_4.4x6.5mm_P0.65mm, symbol AmigaPCI-Symbols:74LVC245
Changed lines of the file:
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@@
   (title_block
     (title "AMIGA PCI")
-    (date "2024-01-30")
+    (date "2024-01-31")
     (rev "2.0")
   )
@@
   )
   (junction (at 244.602 156.718) (diameter 0) (color 0 0 0 0)
-  )
-  (junction (at 126.365 65.405) (diameter 0) (color 0 0 0 0)
   )
   (junction (at 77.851 171.958) (diameter 0) (color 0 0 0 0)
@@
     (stroke (width 0) (type default))
   )
-  (wire (pts (xy 131.572 62.865) (xy 126.365 62.865))
-    (stroke (width 0) (type default))
-  )
   (bus (pts (xy 41.148 144.272) (xy 41.148 139.192))
     (stroke (width 0) (type default))
@@
     (stroke (width 0) (type default))
   )
-  (wire (pts (xy 126.365 65.405) (xy 126.365 71.374))
-    (stroke (width 0) (type default))
-  )
   (wire (pts (xy 220.472 131.318) (xy 231.902 131.318))
     (stroke (width 0) (type default))
@@
     (stroke (width 0) (type default))
   )
-  (wire (pts (xy 126.365 62.865) (xy 126.365 65.405))
-    (stroke (width 0) (type default))
-  )
   (bus (pts (xy 96.012 131.572) (xy 96.012 129.032))
     (stroke (width 0) (type default))
@@
   )
   (bus (pts (xy 41.148 32.258) (xy 41.148 27.178))
-    (stroke (width 0) (type default))
-  )
-  (wire (pts (xy 126.365 65.405) (xy 131.572 65.405))
     (stroke (width 0) (type default))
   )
@@
     (effects (font (size 1.27 1.27)) (justify left bottom))
   )
-  (label "_INTD" (at 131.572 47.625 180) (fields_autoplaced)
-    (effects (font (size 1.27 1.27)) (justify right bottom))
-  )
   (label "LVR_W" (at 43.688 159.512 0) (fields_autoplaced)
     (effects (font (size 1.27 1.27)) (justify left bottom))
@@
     (effects (font (size 1.27 1.27)) (justify right bottom))
   )
-  (label "_INTB" (at 131.572 42.545 180) (fields_autoplaced)
-    (effects (font (size 1.27 1.27)) (justify right bottom))
-  )
   (label "LVAD7" (at 43.815 70.358 0) (fields_autoplaced)
     (effects (font (size 1.27 1.27)) (justify left bottom))
@@
     (effects (font (size 1.27 1.27)) (justify left bottom))
   )
-  (label "_INTA" (at 131.572 40.005 180) (fields_autoplaced)
-    (effects (font (size 1.27 1.27)) (justify right bottom))
-  )
   (label "LVAD23" (at 43.815 141.732 0) (fields_autoplaced)
     (effects (font (size 1.27 1.27)) (justify left bottom))
@@
     (effects (font (size 1.27 1.27)) (justify right bottom))
   )
-  (label "_REQ3" (at 131.572 57.785 180) (fields_autoplaced)
-    (effects (font (size 1.27 1.27)) (justify right bottom))
-  )
   (label "LVAD16" (at 43.815 118.872 0) (fields_autoplaced)
     (effects (font (size 1.27 1.27)) (justify left bottom))
@@
     (effects (font (size 1.27 1.27)) (justify right bottom))
   )
-  (label "_REQ0" (at 131.572 50.165 180) (fields_autoplaced)
-    (effects (font (size 1.27 1.27)) (justify right bottom))
-  )
   (label "+5V" (at 93.472 101.092 180) (fields_autoplaced)
     (effects (font (size 1.27 1.27)) (justify right bottom))
@@
     (effects (font (size 1.27 1.27)) (justify left bottom))
   )
-  (label "_INTC" (at 131.572 45.085 180) (fields_autoplaced)
-    (effects (font (size 1.27 1.27)) (justify right bottom))
-  )
   (label "AD16" (at 93.345 118.872 180) (fields_autoplaced)
     (effects (font (size 1.27 1.27)) (justify right bottom))
@@
     (effects (font (size 1.27 1.27)) (justify right bottom))
   )
-  (label "_REQ2" (at 131.572 55.245 180) (fields_autoplaced)
-    (effects (font (size 1.27 1.27)) (justify right bottom))
-  )
-  (label "_REQ1" (at 131.572 52.705 180) (fields_autoplaced)
-    (effects (font (size 1.27 1.27)) (justify right bottom))
-  )
   (label "LVR_W" (at 43.688 101.092 0) (fields_autoplaced)
     (effects (font (size 1.27 1.27)) (justify left bottom))
   )
-  (label "_REQ4" (at 135.763 75.946 0) (fields_autoplaced)
-    (effects (font (size 1.27 1.27)) (justify left bottom))
-  )
   (label "AD5" (at 93.472 65.278 180) (fields_autoplaced)
     (effects (font (size 1.27 1.27)) (justify right bottom))
@@
   (label "LVAD22" (at 43.815 139.192 0) (fields_autoplaced)
     (effects (font (size 1.27 1.27)) (justify left bottom))
-  )
-  (global_label "_BUSREQ0" (shape output) (at 156.972 50.165 0) (fields_autoplaced)
-    (effects (font (size 1.27 1.27)) (justify left))
-    (property "Intersheetrefs" "${INTERSHEET_REFS}" (at 169.1218 50.0856 0)
-      (effects (font (size 1.27 1.27)) (justify left))
-    )
   )
   (global_label "LVAD[31..0]" (shape bidirectional) (at 33.02 20.066 180) (fields_autoplaced)
@@
     )
   )
-  (global_label "_INTC" (shape output) (at 156.972 45.085 0) (fields_autoplaced)
-    (effects (font (size 1.27 1.27)) (justify left))
-    (property "Intersheetrefs" "${INTERSHEET_REFS}" (at 164.5256 45.0056 0)
-      (effects (font (size 1.27 1.27)) (justify left))
-    )
-  )
   (global_label "CONFIG_CYCLE" (shape input) (at 230.251 85.725 180) (fields_autoplaced)
     (effects (font (size 1.27 1.27)) (justify right))
@@
     )
   )
-  (global_label "_INTA" (shape output) (at 156.972 40.005 0) (fields_autoplaced)
-    (effects (font (size 1.27 1.27)) (justify left))
-    (property "Intersheetrefs" "${INTERSHEET_REFS}" (at 164.3441 39.9256 0)
-      (effects (font (size 1.27 1.27)) (justify left))
-    )
-  )
-  (global_label "_BUSREQ1" (shape output) (at 156.972 52.705 0) (fields_autoplaced)
-    (effects (font (size 1.27 1.27)) (justify left))
-    (property "Intersheetrefs" "${INTERSHEET_REFS}" (at 169.1218 52.6256 0)
-      (effects (font (size 1.27 1.27)) (justify left))
-    )
-  )
-  (global_label "_INTB" (shape output) (at 156.972 42.545 0) (fields_autoplaced)
-    (effects (font (size 1.27 1.27)) (justify left))
-    (property "Intersheetrefs" "${INTERSHEET_REFS}" (at 164.5256 42.4656 0)
-      (effects (font (size 1.27 1.27)) (justify left))
-    )
-  )
   (global_label "IDSEL1" (shape output) (at 257.683 62.865 0) (fields_autoplaced)
     (effects (font (size 1.27 1.27)) (justify left))
@@
     )
   )
-  (global_label "_BUSREQ3" (shape output) (at 156.972 57.785 0) (fields_autoplaced)
-    (effects (font (size 1.27 1.27)) (justify left))
-    (property "Intersheetrefs" "${INTERSHEET_REFS}" (at 169.1218 57.7056 0)
-      (effects (font (size 1.27 1.27)) (justify left))
-    )
-  )
   (global_label "ACSEL1" (shape input) (at 230.251 65.405 180) (fields_autoplaced)
     (effects (font (size 1.27 1.27)) (justify right))
@@
     )
   )
-  (global_label "_INTD" (shape output) (at 156.972 47.625 0) (fields_autoplaced)
-    (effects (font (size 1.27 1.27)) (justify left))
-    (property "Intersheetrefs" "${INTERSHEET_REFS}" (at 164.5256 47.5456 0)
-      (effects (font (size 1.27 1.27)) (justify left))
-    )
-  )
   (global_label "ACSEL0" (shape input) (at 230.251 73.025 180) (fields_autoplaced)
     (effects (font (size 1.27 1.27)) (justify right))
@@
     )
   )
-  (global_label "_BUSREQ4" (shape output) (at 151.511 75.946 0) (fields_autoplaced)
-    (effects (font (size 1.27 1.27)) (justify left))
-    (property "Intersheetrefs" "${INTERSHEET_REFS}" (at 164.1534 75.946 0)
-      (effects (font (size 1.27 1.27)) (justify left))
-    )
-  )
   (global_label "IDSEL4" (shape output) (at 257.302 131.318 0) (fields_autoplaced)
     (effects (font (size 1.27 1.27)) (justify left))
     (property "Intersheetrefs" "${INTERSHEET_REFS}" (at 266.7581 131.318 0)
       (effects (font (size 1.27 1.27)) (justify left))
-    )
-  )
-  (global_label "_BUSREQ2" (shape output) (at 156.972 55.245 0) (fields_autoplaced)
-    (effects (font (size 1.27 1.27)) (justify left))
-    (property "Intersheetrefs" "${INTERSHEET_REFS}" (at 169.1218 55.1656 0)
-      (effects (font (size 1.27 1.27)) (justify left))
-    )
-  )
-  (symbol (lib_id "power:GND") (at 126.365 71.374 0) (unit 1)
-    (in_bom yes) (on_board yes) (dnp no) (fields_autoplaced)
-    (property "Reference" "#PWR0202" (at 126.365 77.724 0)
-      (effects (font (size 1.27 1.27)) hide)
-    )
-    (property "Value" "GND" (at 126.365 76.2 0)
-      (effects (font (size 1.27 1.27)))
-    )
-    (property "Footprint" "" (at 126.365 71.374 0)
-      (effects (font (size 1.27 1.27)) hide)
-    )
-    (property "Datasheet" "" (at 126.365 71.374 0)
-      (effects (font (size 1.27 1.27)) hide)
-    )
-    (pin "1")
-    (instances
-      (project "AmigaPCI Mainboard"
-        (path "/72453515-27fe-4336-91f3-e3c8054f7767/ef92c99c-ab64-412b-bb4d-da92b597d4b5"
-          (reference "#PWR0202") (unit 1)
-        )
-      )
     )
   )
@@
   )
   (symbol (lib_id "power:GND") (at 221.234 116.078 0) (unit 1)
-    (in_bom yes) (on_board yes) (dnp no) (fields_autoplaced)
+    (in_bom yes) (on_board yes) (dnp no)
     (property "Reference" "#PWR0238" (at 221.234 122.428 0)
       (effects (font (size 1.27 1.27)) hide)
@@
         )
       )
-    )
-  )
-  (symbol (lib_id "AmigaPCI-Symbols:74LVC245") (at 144.272 52.705 0) (unit 1)
-    (in_bom yes) (on_board yes) (dnp no) (fields_autoplaced)
-    (property "Reference" "U2" (at 144.272 33.02 0)
-      (effects (font (size 1.27 1.27)))
-    )
-    (property "Value" "74LVC245" (at 144.272 35.56 0)
-      (effects (font (size 1.27 1.27)))
-    )
-    (property "Footprint" "Package_SO:TSSOP-20_4.4x6.5mm_P0.65mm" (at 144.272 52.705 0)
-      (effects (font (size 1.27 1.27)) hide)
-    )
-    (property "Datasheet" "http://www.ti.com/lit/gpn/sn74LS245" (at 144.272 52.705 0)
-      (effects (font (size 1.27 1.27)) hide)
-    )
-    (pin "2")
-    (pin "12")
-    (pin "14")
-    (pin "6")
-    (pin "5")
-    (pin "9")
-    (pin "4")
-    (pin "19")
-    (pin "3")
-    (pin "1")
-    (pin "10")
-    (pin "20")
-    (pin "8")
-    (pin "15")
-    (pin "16")
-    (pin "11")
-    (pin "18")
-    (pin "7")
-    (pin "17")
-    (pin "13")
-    (instances
-      (project "AmigaPCI Mainboard"
-        (path "/72453515-27fe-4336-91f3-e3c8054f7767/ef92c99c-ab64-412b-bb4d-da92b597d4b5"
-          (reference "U2") (unit 1)
-        )
-      )

Commit message: PCB Routing 01-FEB-2024
Parts:
- removed U112: 74AHCT157, Package_SO:TSSOP-16_4.4x5mm_P0.65mm, symbol 74xx:74LS157
- added U112: 74LVC1G157, Package_TO_SOT_SMD:SOT-363_SC-70-6, symbol AmigaPCI-Symbols:74LVC1G157
Connections:
- net +5V: now also U112.5 (VCC)
- net ACSEL4: now also U112.1 (I1)
- net CONFIG_CYCLE: now also U112.6 (S)
- net GND: now also U112.2 (GND)
- net IDSEL4: now also U112.4 (Y)
- net LVAD20: now also U112.3 (I0)
- no-connect marks 3 -> 0
Other:
- moved on the sheet: C155
