File: KiCAD/AmigaPCI Mainboard-KiCAD REV 30/cpu.kicad_sch (KiCad schematic)
At the start: 47 parts, among them CN712 SPI, U200 MC68040, U712 ICE40HX4K-TQ144, U712F1 W25X20CLSN

Commit message: Rev 3.0 PCB Updates 29-APR-2024
Connections:
- net U712_SDI: now also U712.67 (IOB_105_SDO); no longer U712.68 (IOB_106_SDI)
- net U712_SDO: now also U712.68 (IOB_106_SDI); no longer U712.67 (IOB_105_SDO)
Other:
- moved on the sheet: C202, C203, C204, C205, C212, C247, C719, C720, C721, C722, C723, C724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

Commit message: Rev 3.0 Updates 30-APR-2024
Parts:
- added R218, R219: 22R, Resistor_SMD:R_0603_1608Metric, symbol Device:R
- RN200, RN201, RN202, RN203, RN204, RN205, RN206, RN207, RN208, RN209: value 1k -> 4k7; Part 746X101102JP -> YC358TJK-074K7L
- RN210: value 1k -> 4k7; Part (none) -> YC358TJK-074K7L
Connections:
- net CLK40: now also R218.2; no longer U712.21 (IO3_14A_GBIN6)
- net CLK80: now also R219.2; no longer U712.38 (IO2_57)
- new net: R218.1, U712.21 (IO3_14A_GBIN6)
- new net: R219.1, U712.38 (IO2_57)

Commit message: Rev 3.0 PCB Routing 12-MAY-2024
Parts:
- removed C200, C201, C202, C203, C204, C205, C206, C207, C208, C209, C210, C211, C212, C247: 0.1uF, Capacitor_SMD:C_0603_1608Metric, symbol Device:C_Small
- removed RN200, RN201, RN202, RN203, RN204, RN205, RN206, RN207: 4k7, Resistor_SMD:R_Array_Convex_5x1206, symbol AmigaPCI-Symbols:R_SM_Network08
- removed U200: MC68040, AmigaPCI:PGA179, symbol AmigaPCI-Symbols:MC68040RC33
- added CN1: DIN41612_03x40, AmigaPCI:DIN41612_C_3x40_Female_Vertical_THT, symbol AmigaPCI-Symbols:DIN41612_03x40
- added RN1, RN2, RN3, RN4, RN5, RN6: R_Network08, Resistor_THT:R_Array_SIP9, symbol Device:R_Network08
- RN208, RN209, RN210: value 4k7 -> 3k3; footprint Resistor_SMD:R_Array_Convex_5x1206 -> Resistor_SMD:R_Array_Convex_5x0603; Part YC358TJK-074K7L -> YC158TJR-073K3L
Connections:
- net +1V2: now also CN1.a6 (Pin_a6)
- net +3V3: now also CN1.a21 (Pin_a21), CN1.a34 (Pin_a34), CN1.b5 (Pin_b5), CN1.b6 (Pin_b6), CN1.c13 (Pin_c13), CN1.c14 (Pin_c14)
- net +5V: now also CN1.a22 (Pin_a22), CN1.a25 (Pin_a25), CN1.a26 (Pin_a26), CN1.a33 (Pin_a33), CN1.a7 (Pin_a7), CN1.c5 (Pin_c5), RN1.1 (common), RN2.1 (common), RN3.1 (common), RN4.1 (common), RN5.1 (common), RN6.1 (common)
- net A0: now also CN1.b3 (Pin_b3)
- net A1: now also CN1.a4 (Pin_a4)
- net A10: now also CN1.b10 (Pin_b10)
- net A11: now also CN1.a10 (Pin_a10)
- net A12: now also CN1.a2 (Pin_a2)
- net A13: now also CN1.b2 (Pin_b2)
- net A14: now also CN1.a3 (Pin_a3)
- net A15: now also CN1.c3 (Pin_c3)
- net A16: now also CN1.c40 (Pin_c40), RN1.2 (R1)
- net A17: now also CN1.b40 (Pin_b40), RN2.2 (R1)
- net A18: now also CN1.a40 (Pin_a40), RN2.3 (R2)
- net A19: now also CN1.c39 (Pin_c39), RN1.3 (R2)
- net A2: now also CN1.b4 (Pin_b4)
- net A20: now also CN1.b39 (Pin_b39), RN1.4 (R3)
- net A21: now also CN1.c38 (Pin_c38), RN1.5 (R4)
- net A22: now also CN1.a35 (Pin_a35), RN2.9 (R8)
- net A23: now also CN1.a39 (Pin_a39), RN2.4 (R3)
- net A24: now also CN1.a36 (Pin_a36), RN2.7 (R6)
- net A25: now also CN1.b38 (Pin_b38), RN2.5 (R4)
- net A26: now also CN1.b35 (Pin_b35), RN1.9 (R8)
- net A27: now also CN1.c37 (Pin_c37), RN1.6 (R5)
- net A28: now also CN1.c35 (Pin_c35), RN2.8 (R7)
- net A29: now also CN1.c36 (Pin_c36), RN1.7 (R6)
- net A3: now also CN1.c4 (Pin_c4)
- net A30: now also CN1.b36 (Pin_b36), RN1.8 (R7)
- net A31: now also CN1.b37 (Pin_b37), RN2.6 (R5)
- net A4: now also CN1.a5 (Pin_a5)
- net A5: now also CN1.b8 (Pin_b8)
- net A6: now also CN1.a8 (Pin_a8)
- net A7: now also CN1.b9 (Pin_b9)
- net A8: now also CN1.a9 (Pin_a9)
- net A9: now also CN1.c8 (Pin_c8)
- net CLK40: now also CN1.a28 (Pin_a28)
- net CLK80: now also CN1.a24 (Pin_a24)
- net D0: now also CN1.a32 (Pin_a32), RN3.2 (R1)
- net D1: now also CN1.c31 (Pin_c31), RN3.3 (R2)
- net D10: now also CN1.c26 (Pin_c26), RN4.4 (R3)
- net D11: now also CN1.b26 (Pin_b26), RN4.5 (R4)
- net D12: now also CN1.c25 (Pin_c25), RN4.6 (R5)
- net D13: now also CN1.c24 (Pin_c24), RN4.7 (R6)
- net D14: now also CN1.c20 (Pin_c20), RN4.8 (R7)
- net D15: now also CN1.b20 (Pin_b20), RN4.9 (R8)
- net D16: now also CN1.b25 (Pin_b25), RN5.2 (R1)
- net D17: now also CN1.a20 (Pin_a20), RN5.3 (R2)
- net D18: now also CN1.b24 (Pin_b24), RN5.4 (R3)
- net D19: now also CN1.b19 (Pin_b19), RN5.5 (R4)
- net D2: now also CN1.a31 (Pin_a31), RN3.4 (R3)
- net D20: now also CN1.a18 (Pin_a18), RN5.6 (R5)
- net D21: now also CN1.c15 (Pin_c15), RN5.7 (R6)
- net D22: now also CN1.b18 (Pin_b18), RN5.8 (R7)
- net D23: now also CN1.c19 (Pin_c19), RN5.9 (R8)
- net D24: now also CN1.b14 (Pin_b14), RN6.2 (R1)
- net D25: now also CN1.a19 (Pin_a19), RN6.3 (R2)
- net D26: now also CN1.a14 (Pin_a14), RN6.4 (R3)
- net D27: now also CN1.b16 (Pin_b16), RN6.5 (R4)
- net D28: now also CN1.b13 (Pin_b13), RN6.6 (R5)
- net D29: now also CN1.a16 (Pin_a16), RN6.7 (R6)
- net D3: now also CN1.b32 (Pin_b32), RN3.5 (R4)
- net D30: now also CN1.b15 (Pin_b15), RN6.8 (R7)
- net D31: now also CN1.a15 (Pin_a15), RN6.9 (R8)
- net D4: now also CN1.b31 (Pin_b31), RN3.6 (R5)
- net D5: now also CN1.c30 (Pin_c30), RN3.7 (R6)
- net D6: now also CN1.b30 (Pin_b30), RN3.8 (R7)
- net D7: now also CN1.c29 (Pin_c29), RN3.9 (R8)
- net D8: now also CN1.a27 (Pin_a27), RN4.2 (R1)
- net D9: now also CN1.b27 (Pin_b27), RN4.3 (R2)
- net GND: now also CN1.a29 (Pin_a29), CN1.a30 (Pin_a30), CN1.a37 (Pin_a37), CN1.a38 (Pin_a38), CN1.b7 (Pin_b7), CN1.c1 (Pin_c1), CN1.c10 (Pin_c10), CN1.c17 (Pin_c17), CN1.c18 (Pin_c18), CN1.c2 (Pin_c2), CN1.c9 (Pin_c9)
- net R_W: now also CN1.b12 (Pin_b12)
- net SIZ0: now also CN1.c16 (Pin_c16)
- net SIZ1: now also CN1.a17 (Pin_a17)
- net TDO: now also RN208.4 (R4); no longer RN208.3 (R3)
- net TM0: now also CN1.a12 (Pin_a12)
- net TM1: now also CN1.c12 (Pin_c12)
- net TM2: now also CN1.a13 (Pin_a13)
- net TT0: now also RN208.2 (R2), CN1.c32 (Pin_c32); no longer RN208.1 (R1)
- net TT1: now also RN208.3 (R3), CN1.b33 (Pin_b33); no longer RN208.2 (R2)
- net UPA0: now also RN208.8 (R7), CN1.c33 (Pin_c33); no longer RN208.7 (R6)
- net UPA1: now also RN208.9 (R8), CN1.b34 (Pin_b34); no longer RN208.8 (R7)
- net _BB: now also CN1.b1 (Pin_b1)
- net _BG: now also CN1.c22 (Pin_c22)
- net _BR: now also CN1.a11 (Pin_a11)
- net _CDIS: now also RN208.1 (R1); no longer RN208.4 (R4)
- net _IPL0: now also CN1.c27 (Pin_c27)
- net _IPL1: now also CN1.c28 (Pin_c28)
- net _IPL2: now also CN1.b29 (Pin_b29)
- net _LOCK: now also CN1.b11 (Pin_b11)
- net _LOCKE: now also CN1.c11 (Pin_c11)
- net _MDIS: now also RN208.7 (R6); no longer RN208.9 (R8)
- net _RESET: now also CN1.b28 (Pin_b28)
- net _RSTOUT: now also CN1.c34 (Pin_c34)
- net _TA: now also CN1.b21 (Pin_b21)
- net _TBI: now also CN1.a23 (Pin_a23)
- net _TCI: now also CN1.c23 (Pin_c23)
- net _TEA: now also CN1.c21 (Pin_c21)
- net _TIP: now also CN1.a1 (Pin_a1)
- net _TS: now also CN1.b17 (Pin_b17)
- new net BUFDIS: CN1.b22 (Pin_b22)
- new net _CPUCONF: CN1.c7 (Pin_c7)
- new net _INT2: CN1.c6 (Pin_c6)
- new net _INT6: CN1.b23 (Pin_b23)
- no-connect marks 35 -> 13
Other:
- note added: "CPU LOCAL BUS CONNECTOR"
- note removed: "MC68040"
- note removed: "MC68040 POWER"
- note removed: "MC68040 PREFERED HEATSINK: ATS-CPX060060025-132-C1-R0 x 1 ATS-HK127-R0 x 4 ALTERNATE HEATSINK: BDN18-6CB/A01"
- moved on the sheet: RN208, RN209, RN210

Commit message: Main board routing 14-MAY-2024
Parts:
- added R200, R221: 10k, Resistor_SMD:R_0603_1608Metric, symbol Device:R
- renumbered CN1 to CN200
Connections:
- net A10: now also RN2.2 (R1)
- net A11: now also RN2.3 (R2)
- net A12: now also RN2.4 (R3)
- net A13: now also RN2.5 (R4)
- net A14: now also RN2.6 (R5)
- net A15: now also RN2.7 (R6)
- net A16: now also RN2.8 (R7); no longer RN1.2 (R1)
- net A17: now also RN2.9 (R8); no longer RN2.2 (R1)
- net A18: no longer RN2.3 (R2)
- net A19: no longer RN1.3 (R2)
- net A2: now also RN1.2 (R1)
- net A20: no longer RN1.4 (R3)
- net A21: no longer RN1.5 (R4)
- net A22: no longer RN2.9 (R8)
- net A23: no longer RN2.4 (R3)
- net A24: no longer RN2.7 (R6)
- net A25: no longer RN2.5 (R4)
- net A26: no longer RN1.9 (R8)
- net A27: no longer RN1.6 (R5)
- net A28: no longer RN2.8 (R7)
- net A29: no longer RN1.7 (R6)
- net A3: now also RN1.3 (R2)
- net A30: no longer RN1.8 (R7)
- net A31: no longer RN2.6 (R5)
- net A4: now also RN1.4 (R3)
- net A5: now also RN1.5 (R4)
- net A6: now also RN1.6 (R5)
- net A7: now also RN1.7 (R6)
- net A8: now also RN1.8 (R7)
- net A9: now also RN1.9 (R8)
- net BUFDIS: now also R221.2
- net GND: now also R200.2, R221.1
- net _CPUCONF: now also R200.1

Commit message: Main Board Routing 18-MAY-2024
Connections:
- net DRDDIR: now also U712.107 (IO1_167); no longer U712.87 (IO1_136)
- net LVDRA0-G: now also U712.102 (IO1_161); no longer U712.104 (IO1_164)
- net LVDRA1-0: now also U712.101 (IO1_160); no longer U712.102 (IO1_161)
- net LVDRA2-1: now also U712.99 (IO1_152); no longer U712.101 (IO1_160)
- net LVDRA3-2: now also U712.98 (IO1_148); no longer U712.99 (IO1_152)
- net LVDRA4-3: now also U712.97 (IO1_147); no longer U712.98 (IO1_148)
- net LVDRA5-4: now also U712.96 (IO1_146); no longer U712.97 (IO1_147)
- net LVDRA6-5: now also U712.95 (IO1_144); no longer U712.96 (IO1_146)
- net LVDRA7-6: now also U712.91 (IO1_139); no longer U712.95 (IO1_144)
- net LVDRA8-7: now also U712.90 (IO1_138); no longer U712.91 (IO1_139)
- net LVDRA9-8: now also U712.106 (IO1_166); no longer U712.107 (IO1_167)
- net _LVCASL: now also U712.104 (IO1_164); no longer U712.105 (IO1_165)
- net _LVCASU: now also U712.105 (IO1_165); no longer U712.106 (IO1_166)
- net _LVRAS0: now also U712.88 (IO1_137); no longer U712.90 (IO1_138)
- net _LVRAS1: now also U712.87 (IO1_136); no longer U712.88 (IO1_137)
Changed lines of the file:
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@@
 	(title_block
 		(title "AMIGA PCI")
-		(date "2024-05-14")
+		(date "2024-05-18")
 		(rev "3.0")
 	)
@@
 	(global_label "LVDRA1-0"
 		(shape input)
-		(at 134.62 147.32 0)
+		(at 134.62 144.78 0)
 		(fields_autoplaced yes)
 		(effects
@@
 		)
 		(property "Intersheetrefs" "${INTERSHEET_REFS}"
-			(at 147.5957 147.32 0)
+			(at 147.5957 144.78 0)
 			(effects
 				(font
@@
 	(global_label "DRDDIR"
 		(shape output)
-		(at 134.62 121.92 0)
+		(at 134.62 157.48 0)
 		(fields_autoplaced yes)
 		(effects
@@
 		)
 		(property "Intersheetrefs" "${INTERSHEET_REFS}"
-			(at 144.56 121.92 0)
+			(at 144.56 157.48 0)
 			(effects
 				(font
@@
 	(global_label "LVDRA9-8"
 		(shape input)
-		(at 134.62 157.48 0)
+		(at 134.62 154.94 0)
 		(fields_autoplaced yes)
 		(effects
@@
 		)
 		(property "Intersheetrefs" "${INTERSHEET_REFS}"
-			(at 147.5957 157.48 0)
+			(at 147.5957 154.94 0)
 			(effects
 				(font
@@
 	(global_label "_LVCASL"
 		(shape input)
-		(at 134.62 152.4 0)
+		(at 134.62 149.86 0)
 		(fields_autoplaced yes)
 		(effects
@@
 		)
 		(property "Intersheetrefs" "${INTERSHEET_REFS}"
-			(at 145.4985 152.4 0)
+			(at 145.4985 149.86 0)
 			(effects
 				(font
@@
 	(global_label "LVDRA7-6"
 		(shape input)
-		(at 134.62 132.08 0)
+		(at 134.62 129.54 0)
 		(fields_autoplaced yes)
 		(effects
@@
 		)
 		(property "Intersheetrefs" "${INTERSHEET_REFS}"
-			(at 147.5957 132.08 0)
+			(at 147.5957 129.54 0)
 			(effects
 				(font
@@
 	(global_label "_LVCASU"
 		(shape input)
-		(at 134.62 154.94 0)
+		(at 134.62 152.4 0)
 		(fields_autoplaced yes)
 		(effects
@@
 		)
 		(property "Intersheetrefs" "${INTERSHEET_REFS}"
-			(at 145.8069 154.94 0)
+			(at 145.8069 152.4 0)
 			(effects
 				(font
@@
 	(global_label "LVDRA3-2"
 		(shape input)
-		(at 134.62 142.24 0)
+		(at 134.62 139.7 0)
 		(fields_autoplaced yes)
 		(effects
@@
 		)
 		(property "Intersheetrefs" "${INTERSHEET_REFS}"
-			(at 147.5957 142.24 0)
+			(at 147.5957 139.7 0)
 			(effects
 				(font
@@
 	(global_label "LVDRA5-4"
 		(shape input)
-		(at 134.62 137.16 0)
+		(at 134.62 134.62 0)
 		(fields_autoplaced yes)
 		(effects
@@
 		)
 		(property "Intersheetrefs" "${INTERSHEET_REFS}"
-			(at 147.5957 137.16 0)
+			(at 147.5957 134.62 0)
 			(effects
 				(font
@@
 	(global_label "LVDRA8-7"
 		(shape input)
-		(at 134.62 129.54 0)
+		(at 134.62 127 0)
 		(fields_autoplaced yes)
 		(effects
@@
 		)
 		(property "Intersheetrefs" "${INTERSHEET_REFS}"
-			(at 147.5957 129.54 0)
+			(at 147.5957 127 0)
 			(effects
 				(font
@@
 	(global_label "LVDRA2-1"
 		(shape input)
-		(at 134.62 144.78 0)
+		(at 134.62 142.24 0)
 		(fields_autoplaced yes)
 		(effects
@@
 		)
 		(property "Intersheetrefs" "${INTERSHEET_REFS}"
-			(at 147.5957 144.78 0)
+			(at 147.5957 142.24 0)
 			(effects
 				(font
@@
 	(global_label "LVDRA6-5"
 		(shape input)
-		(at 134.62 134.62 0)
+		(at 134.62 132.08 0)
 		(fields_autoplaced yes)
 		(effects
@@
 		)
 		(property "Intersheetrefs" "${INTERSHEET_REFS}"
-			(at 147.5957 134.62 0)
+			(at 147.5957 132.08 0)
 			(effects
 				(font
@@
 	(global_label "LVDRA4-3"
 		(shape input)
-		(at 134.62 139.7 0)
+		(at 134.62 137.16 0)
 		(fields_autoplaced yes)
 		(effects
@@
 		)
 		(property "Intersheetrefs" "${INTERSHEET_REFS}"
-			(at 147.5957 139.7 0)
+			(at 147.5957 137.16 0)
 			(effects
 				(font
@@
 	(global_label "_LVRAS1"
 		(shape input)
-		(at 134.62 124.46 0)
+		(at 134.62 121.92 0)
 		(fields_autoplaced yes)
 		(effects
@@
 		)
 		(property "Intersheetrefs" "${INTERSHEET_REFS}"
-			(at 145.6835 124.46 0)
+			(at 145.6835 121.92 0)
 			(effects
 				(font
@@
 	(global_label "LVDRA0-G"
 		(shape input)
-		(at 134.62 149.86 0)
+		(at 134.62 147.32 0)
 		(fields_autoplaced yes)
 		(effects
@@
 		)
 		(property "Intersheetrefs" "${INTERSHEET_REFS}"
-			(at 147.6574 149.86 0)
+			(at 147.6574 147.32 0)
 			(effects
 				(font
@@
 	(global_label "_LVRAS0"
 		(shape input)
-		(at 134.62 127 0)
+		(at 134.62 124.46 0)
 		(fields_autoplaced yes)
 		(effects
@@
 		)
 		(property "Intersheetrefs" "${INTERSHEET_REFS}"
-			(at 145.6835 127 0)
+			(at 145.6835 124.46 0)
 			(effects
 				(font

Commit message: Main Board Routing 19-MAY-2024
Connections:
- net LVA0: now also U712.12 (IO3_8B); no longer U712.34 (IO3_25B)
- net LVA1: now also U712.10 (IO3_5B); no longer U712.28 (IO3_23A)
- net LVA10: now also U712.23 (IO3_17A); no longer U712.32 (IO3_24B)
- net LVA11: now also U712.24 (IO3_17B); no longer U712.31 (IO3_24A)
- net LVA12: now also U712.25 (IO3_18A); no longer U712.33 (IO3_25A)
- net LVA13: now also U712.26 (IO3_18B); no longer U712.29 (IO3_23B)
- net LVA14: now also U712.28 (IO3_23A); no longer U712.25 (IO3_18A)
- net LVA15: now also U712.29 (IO3_23B); no longer U712.22 (IO3_14B)
- net LVA16: now also U712.31 (IO3_24A); no longer U712.23 (IO3_17A)
- net LVA17: now also U712.32 (IO3_24B); no longer U712.17 (IO3_12A)
- net LVA18: now also U712.33 (IO3_25A); no longer U712.12 (IO3_8B)
- net LVA19: now also U712.34 (IO3_25B); no longer U712.18 (IO3_12B)
- net LVA2: now also U712.8 (IO3_4B); no longer U712.26 (IO3_18B)
- net LVA20: now also U712.11 (IO3_8A); no longer U712.9 (IO3_5A)
- net LVA3: now also U712.9 (IO3_5A); no longer U712.24 (IO3_17B)
- net LVA4: now also U712.15 (IO3_10A); no longer U712.19 (IO3_13A)
- net LVA6: now also U712.17 (IO3_12A); no longer U712.15 (IO3_10A)
- net LVA7: now also U712.18 (IO3_12B); no longer U712.10 (IO3_5B)
- net LVA8: now also U712.19 (IO3_13A); no longer U712.8 (IO3_4B)
- net LVA9: now also U712.22 (IO3_14B); no longer U712.11 (IO3_8A)
- net TICK60: now reaches U712.114 (IO0_171)
- net TICK50: now reaches U712.115 (IO0_172)
- net _BTNRST renamed _FRST
- no-connect marks 13 -> 11
Other:
- note added: "CPU LOCAL BUS PORT"
- note removed: "CPU LOCAL BUS CONNECTOR"
Changed lines of the file:
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@@
 	)
 	(no_connect
-		(at 134.62 170.18)
-	)
-	(no_connect
 		(at 134.62 210.82)
 	)
@@
 	)
 	(no_connect
-		(at 134.62 177.8)
+		(at 134.62 170.18)
 	)
 	(no_connect
@@
 	)
 	(no_connect
-		(at 134.62 175.26)
+		(at 134.62 172.72)
 	)
 	(no_connect
@@
 	)
 	(no_connect
-		(at 134.62 172.72)
-	)
-	(no_connect
 		(at 125.73 83.82)
 	)
@@
 		)
 	)
-	(text "CPU LOCAL BUS CONNECTOR"
+	(text "CPU LOCAL BUS PORT"
 		(exclude_from_sim no)
 		(at 211.582 28.194 0)
@@
 	)
 	(label "LVA9"
-		(at 66.04 157.48 0)
+		(at 66.04 175.26 0)
 		(fields_autoplaced yes)
 		(effects
@@
 	)
 	(label "LVA18"
-		(at 66.04 160.02 0)
+		(at 66.04 198.12 0)
 		(fields_autoplaced yes)
 		(effects
@@
 	)
 	(label "LVA20"
-		(at 66.04 152.4 0)
+		(at 66.04 157.48 0)
 		(fields_autoplaced yes)
 		(effects
@@
 	)
 	(label "LVA8"
-		(at 66.04 149.86 0)
+		(at 66.04 172.72 0)
 		(fields_autoplaced yes)
 		(effects
@@
 	)
 	(label "LVA3"
-		(at 66.04 180.34 0)
+		(at 66.04 152.4 0)
 		(fields_autoplaced yes)
 		(effects
@@
 	)
 	(label "LVA12"
-		(at 66.04 198.12 0)
+		(at 66.04 182.88 0)
 		(fields_autoplaced yes)
 		(effects
@@
 	)
 	(label "LVA13"
-		(at 66.04 190.5 0)
+		(at 66.04 185.42 0)
 		(fields_autoplaced yes)
 		(effects
@@
 	)
 	(label "LVA4"
-		(at 66.04 172.72 0)
+		(at 66.04 162.56 0)
 		(fields_autoplaced yes)
 		(effects
@@
 	)
 	(label "LVA17"
-		(at 66.04 167.64 0)
+		(at 66.04 195.58 0)
 		(fields_autoplaced yes)
 		(effects
@@
 	)
 	(label "LVA14"
-		(at 66.04 182.88 0)
+		(at 66.04 187.96 0)
 		(fields_autoplaced yes)
 		(effects
@@
 	)
 	(label "LVA0"
-		(at 66.04 200.66 0)
+		(at 66.04 160.02 0)
 		(fields_autoplaced yes)
 		(effects
@@
 	)
 	(label "LVA1"
-		(at 66.04 187.96 0)
+		(at 66.04 154.94 0)
 		(fields_autoplaced yes)
 		(effects
@@
 	)
 	(label "LVA15"
-		(at 66.04 175.26 0)
+		(at 66.04 190.5 0)
 		(fields_autoplaced yes)
 		(effects
@@
 	)
 	(label "LVA19"
-		(at 66.04 170.18 0)
+		(at 66.04 200.66 0)
 		(fields_autoplaced yes)
 		(effects
@@
 	)
 	(label "LVA2"
-		(at 66.04 185.42 0)
+		(at 66.04 149.86 0)
 		(fields_autoplaced yes)
 		(effects
@@
 	)
 	(label "LVA11"
-		(at 66.04 193.04 0)
+		(at 66.04 180.34 0)
 		(fields_autoplaced yes)
 		(effects
@@
 	)
 	(label "LVA6"
-		(at 66.04 162.56 0)
+		(at 66.04 167.64 0)
 		(fields_autoplaced yes)
 		(effects
@@
 	)
 	(label "LVA16"
-		(at 66.04 177.8 0)
+		(at 66.04 193.04 0)
 		(fields_autoplaced yes)
 		(effects
@@
 	)
 	(label "LVA7"
-		(at 66.04 154.94 0)
+		(at 66.04 170.18 0)
 		(fields_autoplaced yes)
 		(effects
@@
 	)
 	(label "LVA10"
-		(at 66.04 195.58 0)
+		(at 66.04 177.8 0)
 		(fields_autoplaced yes)
 		(effects
@@
 		)
 	)
+	(global_label "TICK50"
+		(shape output)
+		(at 134.62 177.8 0)
+		(effects
+			(font
+				(size 1.27 1.27)
+			)
+			(justify left)
+		)
+		(property "Intersheetrefs" "${INTERSHEET_REFS}"
+			(at 143.383 177.8 0)
+			(effects
+				(font
+					(size 1.27 1.27)
+				)
+				(justify left)
+			)
+		)
+	)
 	(global_label "_LVCASU"
 		(shape input)
@@
 		)
 	)
+	(global_label "TICK60"
+		(shape output)
+		(at 134.62 175.26 0)
+		(effects
+			(font
+				(size 1.27 1.27)
+			)
+			(justify left)
+		)
+		(property "Intersheetrefs" "${INTERSHEET_REFS}"
+			(at 143.383 175.387 0)
+			(effects
+				(font
+					(size 1.27 1.27)
+				)
+				(justify left)
+			)
+		)
+	)
 	(global_label "TT0"
 		(shape bidirectional)
@@
 		)
 	)
-	(global_label "_BTNRST"
+	(global_label "_FRST"
 		(shape output)
 		(at 73.66 43.18 180)

Commit message: Main Board Routing 22-MAY-2024
Connections:
- net TICK50: no longer names the net of U712.115 (IO0_172)
- net TICK60: no longer names the net of U712.114 (IO0_171)
- net _FRST renamed _BTNRST
- no-connect marks 11 -> 13
Changed lines of the file:
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@@
 	(title_block
 		(title "AMIGA PCI")
-		(date "2024-05-18")
+		(date "2024-05-22")
 		(rev "3.0")
 	)
@@
 	)
 	(no_connect
+		(at 134.62 175.26)
+	)
+	(no_connect
 		(at 74.93 53.34)
 	)
 	(no_connect
+		(at 134.62 177.8)
+	)
+	(no_connect
 		(at 134.62 172.72)
 	)
@@
 		)
 	)
-	(global_label "TICK50"
-		(shape output)
-		(at 134.62 177.8 0)
-		(effects
-			(font
-				(size 1.27 1.27)
-			)
-			(justify left)
-		)
-		(property "Intersheetrefs" "${INTERSHEET_REFS}"
-			(at 143.383 177.8 0)
-			(effects
-				(font
-					(size 1.27 1.27)
-				)
-				(justify left)
-			)
-		)
-	)
 	(global_label "_LVCASU"
 		(shape input)
@@
 		)
 	)
-	(global_label "TICK60"
-		(shape output)
-		(at 134.62 175.26 0)
-		(effects
-			(font
-				(size 1.27 1.27)
-			)
-			(justify left)
-		)
-		(property "Intersheetrefs" "${INTERSHEET_REFS}"
-			(at 143.383 175.387 0)
-			(effects
-				(font
-					(size 1.27 1.27)
-				)
-				(justify left)
-			)
-		)
-	)
 	(global_label "TT0"
 		(shape bidirectional)
@@
 		)
 	)
-	(global_label "_FRST"
+	(global_label "_BTNRST"
 		(shape output)
 		(at 73.66 43.18 180)

Commit message: Main Board Routing 22-May-2024a
Parts:
- added RN7, RN8: R_Network08, Resistor_THT:R_Array_SIP9, symbol Device:R_Network08
Connections:
- net +5V: now also RN7.1 (common), RN8.1 (common)
- net A0: now also RN7.3 (R2)
- net A1: now also RN7.2 (R1)
- net A18: now also RN7.4 (R3)
- net A19: now also RN7.5 (R4)
- net A20: now also RN7.6 (R5)
- net A21: now also RN7.7 (R6)
- net A22: now also RN7.8 (R7)
- net A23: now also RN7.9 (R8)
- net A24: now also RN8.2 (R1)
- net A25: now also RN8.3 (R2)
- net A26: now also RN8.4 (R3)
- net A27: now also RN8.5 (R4)
- net A28: now also RN8.6 (R5)
- net A29: now also RN8.7 (R6)
- net A30: now also RN8.8 (R7)
- net A31: now also RN8.9 (R8)
