File: KiCAD/AmigaPCI Mainboard-KiCAD REV 30/pci-bridge.kicad_sch (KiCad schematic)
At the start: 46 parts, among them CN109 SPI, CN110 SPI, U109 ICE40HX4K-TQ144, U109F1 W25X20CLSN, U110 ICE40HX4K-TQ144, U110F1 W25X20CLSN

Commit message: Rev 3.0 PCB Updates 29-APR-2024
Connections:
- net U109_SDI: now also U109.67 (IOB_105_SDO); no longer U109.68 (IOB_106_SDI)
- net U109_SDO: now also U109.68 (IOB_106_SDI); no longer U109.67 (IOB_105_SDO)
- net U409_SDI: now also U110.67 (IOB_105_SDO); no longer U110.68 (IOB_106_SDI)
- net U409_SDO: now also U110.68 (IOB_106_SDI); no longer U110.67 (IOB_105_SDO)
Other:
- moved on the sheet: C123, C125, C126, C127, C129, C130, C131, C132, C136, C138, C140, C141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

Commit message: Main Board Routing 18-MAY-2024
Connections:
- net LVA24: now also U109.33 (IO3_25A); no longer U109.64 (IO2_104_CBSEL1)
- net LVA30: now also U109.34 (IO3_25B); no longer U109.63 (IO2_103_CBSEL0)
- net LVA8: now also U109.32 (IO3_24B); no longer U109.62 (IO2_102)
- net LVD0: now also U109.62 (IO2_102); no longer U109.33 (IO3_25A)
- net LVD1: now also U109.63 (IO2_103_CBSEL0); no longer U109.73 (IO1_109)
- net LVD12: now also U109.83 (IO1_119); no longer U109.107 (IO1_167)
- net LVD13: now also U109.84 (IO1_120); no longer U109.105 (IO1_165)
- net LVD14: now also U109.85 (IO1_128); no longer U109.104 (IO1_164)
- net LVD15: now also U109.87 (IO1_136); no longer U109.101 (IO1_160)
- net LVD16: now also U109.88 (IO1_137); no longer U109.106 (IO1_166)
- net LVD17: now also U109.90 (IO1_138); no longer U109.99 (IO1_152)
- net LVD18: now also U109.91 (IO1_139); no longer U109.102 (IO1_161)
- net LVD19: now also U109.93 (IO1_140_GBIN3); no longer U109.97 (IO1_147)
- net LVD2: now also U109.64 (IO2_104_CBSEL1); no longer U109.34 (IO3_25B)
- net LVD21: now also U109.95 (IO1_144); no longer U109.90 (IO1_138)
- net LVD22: now also U109.96 (IO1_146); no longer U109.95 (IO1_144)
- net LVD23: now also U109.97 (IO1_147); no longer U109.98 (IO1_148)
- net LVD24: now also U109.98 (IO1_148); no longer U109.85 (IO1_128)
- net LVD25: now also U109.99 (IO1_152); no longer U109.96 (IO1_146)
- net LVD26: now also U109.101 (IO1_160); no longer U109.84 (IO1_120)
- net LVD27: now also U109.102 (IO1_161); no longer U109.93 (IO1_140_GBIN3)
- net LVD28: now also U109.104 (IO1_164); no longer U109.83 (IO1_119)
- net LVD29: now also U109.105 (IO1_165); no longer U109.91 (IO1_139)
- net LVD3: now also U109.73 (IO1_109); no longer U109.75 (IO1_111)
- net LVD30: now also U109.106 (IO1_166); no longer U109.88 (IO1_137)
- net LVD31: now also U109.107 (IO1_167); no longer U109.87 (IO1_136)
- net LVD5: now also U109.75 (IO1_111); no longer U109.76 (IO1_112)
- net LVD6: now also U109.76 (IO1_112); no longer U109.78 (IO1_114)
- net LVD7: now also U109.78 (IO1_114); no longer U109.79 (IO1_115)
- net LVD8: now also U109.79 (IO1_115); no longer U109.32 (IO3_24B)
Changed lines of the file:
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@@
 	(title_block
 		(title "AMIGA PCI")
-		(date "2024-05-14")
+		(date "2024-05-18")
 		(rev "3.0")
 	)
@@
 	)
 	(label "LVD29"
-		(at 54.61 146.05 0)
+		(at 54.61 168.91 0)
 		(fields_autoplaced yes)
 		(effects
@@
 	)
 	(label "LVD22"
-		(at 54.61 148.59 0)
+		(at 54.61 151.13 0)
 		(fields_autoplaced yes)
 		(effects
@@
 	)
 	(label "LVD17"
-		(at 54.61 158.75 0)
+		(at 54.61 143.51 0)
 		(fields_autoplaced yes)
 		(effects
@@
 	)
 	(label "LVD18"
-		(at 54.61 163.83 0)
+		(at 54.61 146.05 0)
 		(fields_autoplaced yes)
 		(effects
@@
 	)
 	(label "LVD13"
-		(at 54.61 168.91 0)
+		(at 54.61 133.35 0)
 		(fields_autoplaced yes)
 		(effects
@@
 	)
 	(label "LVD14"
-		(at 54.61 166.37 0)
+		(at 54.61 135.89 0)
 		(fields_autoplaced yes)
 		(effects
@@
 	)
 	(label "LVD23"
-		(at 54.61 156.21 0)
+		(at 54.61 153.67 0)
 		(fields_autoplaced yes)
 		(effects
@@
 	)
 	(label "LVD31"
-		(at 54.61 138.43 0)
+		(at 54.61 173.99 0)
 		(fields_autoplaced yes)
 		(effects
@@
 	)
 	(label "LVD2"
-		(at 121.92 217.17 180)
+		(at 121.92 69.85 180)
 		(fields_autoplaced yes)
 		(effects
@@
 	)
 	(label "LVD7"
-		(at 54.61 120.65 0)
+		(at 54.61 118.11 0)
 		(fields_autoplaced yes)
 		(effects
@@
 	)
 	(label "LVD12"
-		(at 54.61 173.99 0)
+		(at 54.61 130.81 0)
 		(fields_autoplaced yes)
 		(effects
@@
 	)
 	(label "LVD26"
-		(at 54.61 133.35 0)
+		(at 54.61 161.29 0)
 		(fields_autoplaced yes)
 		(effects
@@
 	)
 	(label "LVD28"
-		(at 54.61 130.81 0)
+		(at 54.61 166.37 0)
 		(fields_autoplaced yes)
 		(effects
@@
 	)
 	(label "LVD1"
-		(at 54.61 107.95 0)
+		(at 121.92 67.31 180)
 		(fields_autoplaced yes)
 		(effects
@@
 				(size 1.27 1.27)
 			)
-			(justify left bottom)
+			(justify right bottom)
 		)
 	)
@@
 	)
 	(label "LVD0"
-		(at 121.92 214.63 180)
+		(at 54.61 105.41 0)
 		(fields_autoplaced yes)
 		(effects
@@
 				(size 1.27 1.27)
 			)
-			(justify right bottom)
+			(justify left bottom)
 		)
 	)
 	(label "LVA24"
-		(at 121.92 69.85 180)
+		(at 121.92 214.63 180)
 		(fields_autoplaced yes)
 		(effects
@@
 	)
 	(label "LVD8"
-		(at 121.92 212.09 180)
+		(at 54.61 120.65 0)
 		(fields_autoplaced yes)
 		(effects
@@
 				(size 1.27 1.27)
 			)
-			(justify right bottom)
+			(justify left bottom)
 		)
 	)
@@
 	)
 	(label "LVA8"
-		(at 54.61 105.41 0)
+		(at 121.92 212.09 180)
 		(fields_autoplaced yes)
 		(effects
@@
 				(size 1.27 1.27)
 			)
-			(justify left bottom)
+			(justify right bottom)
 		)
 	)
@@
 	)
 	(label "LVD19"
-		(at 54.61 153.67 0)
+		(at 121.92 100.33 180)
 		(fields_autoplaced yes)
 		(effects
@@
 				(size 1.27 1.27)
 			)
-			(justify left bottom)
+			(justify right bottom)
 		)
 	)
@@
 	)
 	(label "LVD5"
-		(at 54.61 115.57 0)
+		(at 54.61 113.03 0)
 		(fields_autoplaced yes)
 		(effects
@@
 	)
 	(label "LVD15"
-		(at 54.61 161.29 0)
+		(at 54.61 138.43 0)
 		(fields_autoplaced yes)
 		(effects
@@
 	)
 	(label "LVD27"
-		(at 121.92 100.33 180)
+		(at 54.61 163.83 0)
 		(fields_autoplaced yes)
 		(effects
@@
 				(size 1.27 1.27)
 			)
-			(justify right bottom)
+			(justify left bottom)
 		)
 	)
@@
 	)
 	(label "LVD21"
-		(at 54.61 143.51 0)
+		(at 54.61 148.59 0)
 		(fields_autoplaced yes)
 		(effects
@@
 	)
 	(label "LVD30"
-		(at 54.61 140.97 0)
+		(at 54.61 171.45 0)
 		(fields_autoplaced yes)
 		(effects
@@
 	)
 	(label "LVD24"
-		(at 54.61 135.89 0)
+		(at 54.61 156.21 0)
 		(fields_autoplaced yes)
 		(effects
@@
 	)
 	(label "LVD16"
-		(at 54.61 171.45 0)
+		(at 54.61 140.97 0)
 		(fields_autoplaced yes)
 		(effects
@@
 	)
 	(label "LVA30"
-		(at 121.92 67.31 180)
+		(at 121.92 217.17 180)
 		(fields_autoplaced yes)
 		(effects
@@
 	)
 	(label "LVD3"
-		(at 54.61 113.03 0)
+		(at 54.61 107.95 0)
 		(fields_autoplaced yes)
 		(effects
@@
 	)
 	(label "LVD25"
-		(at 54.61 151.13 0)
+		(at 54.61 158.75 0)
 		(fields_autoplaced yes)
 		(effects
@@
 	)
 	(label "LVD6"
-		(at 54.61 118.11 0)
+		(at 54.61 115.57 0)
 		(fields_autoplaced yes)
 		(effects

Commit message: Main Board Routing 19-MAY-2024
Connections:
- net LVA10: now also U109.43 (IO2_71); no longer U109.18 (IO3_12B)
- net LVA11: now also U109.44 (IO2_72); no longer U109.19 (IO3_13A)
- net LVA12: now also U109.45 (IO2_73); no longer U109.17 (IO3_12A)
- net LVA13: now also U109.47 (IO2_79); no longer U109.20 (IO3_13B_GBIN7)
- net LVA14: now also U109.48 (IO2_80); no longer U109.23 (IO3_17A)
- net LVA15: now also U109.49 (IO2_81_GBIN5); no longer U109.26 (IO3_18B)
- net LVA16: now also U109.55 (IO2_91); no longer U109.25 (IO3_18A)
- net LVA17: now also U109.56 (IO2_94); no longer U109.37 (IO2_56)
- net LVA18: now also U109.60 (IO2_95); no longer U109.41 (IO2_63)
- net LVA19: now also U109.61 (IO2_96); no longer U109.31 (IO3_24A)
- net LVA2: now also U109.17 (IO3_12A); no longer U109.22 (IO3_14B)
- net LVA20: now also U109.33 (IO3_25A); no longer U109.44 (IO2_72)
- net LVA21: now also U109.31 (IO3_24A); no longer U109.48 (IO2_80)
- net LVA22: now also U109.20 (IO3_13B_GBIN7); no longer U109.56 (IO2_94)
- net LVA23: now also U109.32 (IO3_24B); no longer U109.45 (IO2_73)
- net LVA24: now also U109.24 (IO3_17B); no longer U109.33 (IO3_25A)
- net LVA25: now also U109.29 (IO3_23B); no longer U109.47 (IO2_79)
- net LVA26: now also U109.22 (IO3_14B); no longer U109.55 (IO2_91)
- net LVA27: now also U109.28 (IO3_23A); no longer U109.61 (IO2_96)
- net LVA28: now also U109.19 (IO3_13A); no longer U109.49 (IO2_81_GBIN5)
- net LVA29: now also U109.23 (IO3_17A); no longer U109.60 (IO2_95)
- net LVA3: now also U109.18 (IO3_12B); no longer U109.24 (IO3_17B)
- net LVA30: now also U109.25 (IO3_18A); no longer U109.34 (IO3_25B)
- net LVA31: now also U109.26 (IO3_18B); no longer U109.29 (IO3_23B)
- net LVA4: now also U109.34 (IO3_25B); no longer U109.28 (IO3_23A)
- net LVA5: now also U109.37 (IO2_56); no longer U109.38 (IO2_57)
- net LVA6: now also U109.38 (IO2_57); no longer U109.39 (IO2_61)
- net LVA7: now also U109.39 (IO2_61); no longer U109.43 (IO2_71)
- net LVA8: now also U109.41 (IO2_63); no longer U109.32 (IO3_24B)
- net _LVLOCKE: now reaches U110.7 (IO3_4A)
- net TICK50: no longer names the net of U110.74 (IO1_110)
- net TICK60: no longer names the net of U110.75 (IO1_111)
- net _BTNRST renamed _FRST
- no-connect marks 16 -> 15
Changed lines of the file:
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@@
 	)
 	(no_connect
-		(at 281.94 162.56)
-	)
-	(no_connect
 		(at 281.94 208.28)
 	)
@@
 	)
 	(label "LVA5"
-		(at 123.19 118.11 180)
+		(at 123.19 115.57 180)
 		(fields_autoplaced yes)
 		(effects
@@
 	)
 	(label "LVA28"
-		(at 121.92 92.71 180)
+		(at 121.92 189.23 180)
 		(fields_autoplaced yes)
 		(effects
@@
 	)
 	(label "LVA18"
-		(at 123.19 123.19 180)
+		(at 123.19 146.05 180)
 		(fields_autoplaced yes)
 		(effects
@@
 	)
 	(label "LVA10"
-		(at 121.92 186.69 180)
+		(at 123.19 128.27 180)
 		(fields_autoplaced yes)
 		(effects
@@
 	)
 	(label "LVA3"
-		(at 121.92 196.85 180)
+		(at 121.92 186.69 180)
 		(fields_autoplaced yes)
 		(effects
@@
 	)
 	(label "LVA16"
-		(at 121.92 199.39 180)
+		(at 123.19 140.97 180)
 		(fields_autoplaced yes)
 		(effects
@@
 	)
 	(label "LVA19"
-		(at 121.92 209.55 180)
+		(at 123.19 148.59 180)
 		(fields_autoplaced yes)
 		(effects
@@
 	)
 	(label "LVA23"
-		(at 123.19 133.35 180)
+		(at 121.92 212.09 180)
 		(fields_autoplaced yes)
 		(effects
@@
 	)
 	(label "LVA7"
-		(at 123.19 128.27 180)
+		(at 123.19 120.65 180)
 		(fields_autoplaced yes)
 		(effects
@@
 	)
 	(label "LVA14"
-		(at 121.92 194.31 180)
+		(at 123.19 138.43 180)
 		(fields_autoplaced yes)
 		(effects
@@
 	)
 	(label "LVA26"
-		(at 123.19 140.97 180)
+		(at 121.92 191.77 180)
 		(fields_autoplaced yes)
 		(effects
@@
 	)
 	(label "LVA13"
-		(at 121.92 85.09 180)
+		(at 123.19 135.89 180)
 		(fields_autoplaced yes)
 		(effects
@@
 	)
 	(label "LVA24"
-		(at 121.92 214.63 180)
+		(at 121.92 196.85 180)
 		(fields_autoplaced yes)
 		(effects
@@
 	)
 	(label "LVA4"
-		(at 121.92 204.47 180)
+		(at 121.92 217.17 180)
 		(fields_autoplaced yes)
 		(effects
@@
 	)
 	(label "LVA17"
-		(at 123.19 115.57 180)
+		(at 123.19 143.51 180)
 		(fields_autoplaced yes)
 		(effects
@@
 	)
 	(label "LVA20"
-		(at 123.19 130.81 180)
+		(at 121.92 214.63 180)
 		(fields_autoplaced yes)
 		(effects
@@
 	)
 	(label "LVA8"
-		(at 121.92 212.09 180)
+		(at 123.19 123.19 180)
 		(fields_autoplaced yes)
 		(effects
@@
 	)
 	(label "LVA25"
-		(at 123.19 135.89 180)
+		(at 121.92 207.01 180)
 		(fields_autoplaced yes)
 		(effects
@@
 	)
 	(label "LVA11"
-		(at 121.92 189.23 180)
+		(at 123.19 130.81 180)
 		(fields_autoplaced yes)
 		(effects
@@
 	)
 	(label "LVA27"
-		(at 123.19 148.59 180)
+		(at 121.92 204.47 180)
 		(fields_autoplaced yes)
 		(effects
@@
 	)
 	(label "LVA21"
-		(at 123.19 138.43 180)
+		(at 121.92 209.55 180)
 		(fields_autoplaced yes)
 		(effects
@@
 	)
 	(label "LVA12"
-		(at 121.92 184.15 180)
+		(at 123.19 133.35 180)
 		(fields_autoplaced yes)
 		(effects
@@
 	)
 	(label "LVA6"
-		(at 123.19 120.65 180)
+		(at 123.19 118.11 180)
 		(fields_autoplaced yes)
 		(effects
@@
 	)
 	(label "LVA22"
-		(at 123.19 143.51 180)
+		(at 121.92 85.09 180)
 		(fields_autoplaced yes)
 		(effects
@@
 	)
 	(label "LVA31"
-		(at 121.92 207.01 180)
+		(at 121.92 201.93 180)
 		(fields_autoplaced yes)
 		(effects
@@
 	)
 	(label "LVA29"
-		(at 123.19 146.05 180)
+		(at 121.92 194.31 180)
 		(fields_autoplaced yes)
 		(effects
@@
 	)
 	(label "LVA30"
-		(at 121.92 217.17 180)
+		(at 121.92 199.39 180)
 		(fields_autoplaced yes)
 		(effects
@@
 	)
 	(label "LVA2"
-		(at 121.92 191.77 180)
+		(at 121.92 184.15 180)
 		(fields_autoplaced yes)
 		(effects
@@
 	)
 	(label "LVA15"
-		(at 121.92 201.93 180)
+		(at 121.92 92.71 180)
 		(fields_autoplaced yes)
 		(effects
@@
 	)
 	(global_label "LVR_W"
-		(shape input)
+		(shape bidirectional)
 		(at 213.36 114.3 180)
 		(fields_autoplaced yes)
@@
 		)
 		(property "Intersheetrefs" "${INTERSHEET_REFS}"
-			(at 204.5691 114.3 0)
+			(at 203.4578 114.3 0)
 			(effects
 				(font
@@
 		)
 	)
-	(global_label "TICK60"
-		(shape output)
-		(at 213.36 111.76 180)
-		(effects
-			(font
-				(size 1.27 1.27)
-			)
-			(justify right)
-		)
-		(property "Intersheetrefs" "${INTERSHEET_REFS}"
-			(at 204.597 111.633 0)
-			(effects
-				(font
-					(size 1.27 1.27)
-				)
-				(justify right)
-			)
-		)
-	)
 	(global_label "_LVCBE1"
 		(shape output)
@@
 		)
 	)
-	(global_label "TICK50"
-		(shape output)
-		(at 213.36 109.22 180)
+	(global_label "_LVLOCKE"
+		(shape bidirectional)
+		(at 281.94 162.56 0)
+		(fields_autoplaced yes)
 		(effects
 			(font
 				(size 1.27 1.27)
 			)
-			(justify right)
+			(justify left)
 		)
 		(property "Intersheetrefs" "${INTERSHEET_REFS}"
-			(at 204.597 109.22 0)
+			(at 295.1684 162.56 0)
 			(effects
 				(font
 					(size 1.27 1.27)
 				)
-				(justify right)
+				(justify left)
 			)
 		)
@@
 		)
 	)
-	(global_label "_BTNRST"
+	(global_label "_FRST"
 		(shape output)
 		(at 274.32 58.42 0)
@@
 		)
 	)
-	(global_label "_BTNRST"
+	(global_label "_FRST"
 		(shape output)
 		(at 115.57 59.69 0)

Commit message: Main Board Routing 22-MAY-2024
Connections:
- net CLK6: no longer names the net of U110.21 (IO3_14A_GBIN6)
- net _FRST renamed _BTNRST
- no-connect marks 15 -> 16
Changed lines of the file:
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@@
 	(title_block
 		(title "AMIGA PCI")
-		(date "2024-05-18")
+		(date "2024-05-22")
 		(rev "3.0")
 	)
@@
 	)
 	(no_connect
+		(at 281.94 86.36)
+	)
+	(no_connect
 		(at 281.94 167.64)
 	)
@@
 		)
 	)
-	(global_label "_FRST"
+	(global_label "_BTNRST"
 		(shape output)
 		(at 274.32 58.42 0)
@@
 		)
 	)
-	(global_label "_FRST"
+	(global_label "_BTNRST"
 		(shape output)
 		(at 115.57 59.69 0)
@@
 			)
 		)
-	)
-	(global_label "CLK6"
-		(shape input)
-		(at 281.94 86.36 0)
-		(fields_autoplaced yes)
-		(effects
-			(font
-				(size 1.27 1.27)
-			)
-			(justify left)
-		)
-		(property "Intersheetrefs" "${INTERSHEET_REFS}"
-			(at 289.7028 86.36 0)
-			(effects
-				(font
-					(size 1.27 1.27)
-				)
-				(justify left)
-			)
-		)

Commit message: Main Board Routing 22-May-2024a
Connections:
- net _LVLOCKE: now also U110.19 (IO3_13A); no longer U110.7 (IO3_4A)
Changed lines of the file:
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@@
 	)
 	(no_connect
-		(at 281.94 187.96)
+		(at 281.94 162.56)
 	)
 	(no_connect
@@
 	(global_label "_LVLOCKE"
 		(shape bidirectional)
-		(at 281.94 162.56 0)
+		(at 281.94 187.96 0)
 		(fields_autoplaced yes)
 		(effects
@@
 		)
 		(property "Intersheetrefs" "${INTERSHEET_REFS}"
-			(at 295.1684 162.56 0)
+			(at 295.1684 187.96 0)
 			(effects
 				(font
