File: KiCAD/AmigaPCI Mainboard-KiCAD REV 30/power.kicad_sch (KiCad schematic)
At the start: 82 parts, among them CN205 POW SW, CN206 RESET, CN600 Conn_01x03_Pin, CN601 ATX-24, J1 _TA, J10 _RESET, J11 _REGEN, J12 _TBI, J2 CLK7, J210 Case Fan, J5 _TS, J6 _TIP, J7 TT0, J8 TT1, U206 DS1818R-10+T&R, U215 74HCT03, U219 74AHCT04, U220 74LVC08, U222 74HCT4066, U229 74CBT16233, U303 74HCT74, U600 STM8S001J3M, U601 AP2114H-1.2, U818 74AHC1G09

Commit message: Rev 3.0 PCB Updates 29-APR-2024
Parts:
- C110, C111, C112, C113, C114, C115, C116, C117, C118, C119, C120, C121, C133, C134, C601: footprint Capacitor_THT:CP_Radial_D8.0mm_P3.50mm -> Capacitor_THT:CP_Radial_D6.3mm_P2.50mm
Changed lines of the file:
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@@
 			)
 		)
-		(property "Footprint" "Capacitor_THT:CP_Radial_D8.0mm_P3.50mm"
+		(property "Footprint" "Capacitor_THT:CP_Radial_D6.3mm_P2.50mm"
 			(at 125.4252 212.09 0)
 			(effects
@@
 			)
 		)
-		(property "Footprint" "Capacitor_THT:CP_Radial_D8.0mm_P3.50mm"
+		(property "Footprint" "Capacitor_THT:CP_Radial_D6.3mm_P2.50mm"
 			(at 205.4352 212.09 0)
 			(effects
@@
 			)
 		)
-		(property "Footprint" "Capacitor_THT:CP_Radial_D8.0mm_P3.50mm"
+		(property "Footprint" "Capacitor_THT:CP_Radial_D6.3mm_P2.50mm"
 			(at 152.0952 212.09 0)
 			(effects
@@
 			)
 		)
-		(property "Footprint" "Capacitor_THT:CP_Radial_D8.0mm_P3.50mm"
+		(property "Footprint" "Capacitor_THT:CP_Radial_D6.3mm_P2.50mm"
 			(at 178.7652 212.09 0)
 			(effects
@@
 			)
 		)
-		(property "Footprint" "Capacitor_THT:CP_Radial_D8.0mm_P3.50mm"
+		(property "Footprint" "Capacitor_THT:CP_Radial_D6.3mm_P2.50mm"
 			(at 84.7852 212.09 0)
 			(effects
@@
 			)
 		)
-		(property "Footprint" "Capacitor_THT:CP_Radial_D8.0mm_P3.50mm"
+		(property "Footprint" "Capacitor_THT:CP_Radial_D6.3mm_P2.50mm"
 			(at 45.4152 212.09 0)
 			(effects
@@
 			)
 		)
-		(property "Footprint" "Capacitor_THT:CP_Radial_D8.0mm_P3.50mm"
+		(property "Footprint" "Capacitor_THT:CP_Radial_D6.3mm_P2.50mm"
 			(at 164.7952 212.09 0)
 			(effects
@@
 			)
 		)
-		(property "Footprint" "Capacitor_THT:CP_Radial_D8.0mm_P3.50mm"
+		(property "Footprint" "Capacitor_THT:CP_Radial_D6.3mm_P2.50mm"
 			(at 98.7552 212.09 0)
 			(effects
@@
 			)
 		)
-		(property "Footprint" "Capacitor_THT:CP_Radial_D8.0mm_P3.50mm"
+		(property "Footprint" "Capacitor_THT:CP_Radial_D6.3mm_P2.50mm"
 			(at 192.7352 212.09 0)
 			(effects
@@
 			)
 		)
-		(property "Footprint" "Capacitor_THT:CP_Radial_D8.0mm_P3.50mm"
+		(property "Footprint" "Capacitor_THT:CP_Radial_D6.3mm_P2.50mm"
 			(at 26.9748 204.47 0)
 			(effects
@@
 			)
 		)
-		(property "Footprint" "Capacitor_THT:CP_Radial_D8.0mm_P3.50mm"
+		(property "Footprint" "Capacitor_THT:CP_Radial_D6.3mm_P2.50mm"
 			(at 112.7252 212.09 0)
 			(effects
@@
 			)
 		)
-		(property "Footprint" "Capacitor_THT:CP_Radial_D8.0mm_P3.50mm"
+		(property "Footprint" "Capacitor_THT:CP_Radial_D6.3mm_P2.50mm"
 			(at 138.1252 212.09 0)
 			(effects
@@
 			)
 		)
-		(property "Footprint" "Capacitor_THT:CP_Radial_D8.0mm_P3.50mm"
+		(property "Footprint" "Capacitor_THT:CP_Radial_D6.3mm_P2.50mm"
 			(at 58.1152 212.09 0)
 			(effects
@@
 			)
 		)
-		(property "Footprint" "Capacitor_THT:CP_Radial_D8.0mm_P3.50mm"
+		(property "Footprint" "Capacitor_THT:CP_Radial_D6.3mm_P2.50mm"
 			(at 91.7448 43.18 0)
 			(effects
@@
 			)
 		)
-		(property "Footprint" "Capacitor_THT:CP_Radial_D8.0mm_P3.50mm"
+		(property "Footprint" "Capacitor_THT:CP_Radial_D6.3mm_P2.50mm"
 			(at 70.8152 212.09 0)
 			(effects

Commit message: Rev 3.0 PCB Routing 12-MAY-2024
Parts:
- added H11, H12: MountingHole_Pad, MountingHole:MountingHole_2.2mm_M2_DIN965_Pad, symbol Mechanical:MountingHole_Pad
Connections:
- net GND: now also H11.1, H12.1
Other:
- moved on the sheet: H10
Changed lines of the file:
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@@
 	)
 	(junction
+		(at 337.82 177.8)
+		(diameter 0)
+		(color 0 0 0 0)
+	)
+	(junction
 		(at 66.04 176.53)
 		(diameter 0)
@@
 	)
 	(junction
-		(at 347.98 173.99)
-		(diameter 0)
-		(color 0 0 0 0)
-	)
-	(junction
 		(at 140.97 95.25)
 		(diameter 0)
@@
 	)
 	(junction
+		(at 337.82 173.99)
+		(diameter 0)
+		(color 0 0 0 0)
+	)
+	(junction
 		(at 92.71 39.37)
 		(diameter 0)
@@
 	)
 	(junction
+		(at 347.98 173.99)
+		(diameter 0)
+		(color 0 0 0 0)
+	)
+	(junction
 		(at 111.76 55.88)
 		(diameter 0)
@@
 	)
 	(junction
-		(at 86.36 156.21)
+		(at 327.66 173.99)
 		(diameter 0)
 		(color 0 0 0 0)
 	)
 	(junction
-		(at 204.47 204.47)
+		(at 86.36 156.21)
 		(diameter 0)
 		(color 0 0 0 0)
 	)
 	(junction
-		(at 337.82 163.83)
+		(at 204.47 204.47)
 		(diameter 0)
 		(color 0 0 0 0)
 	)
 	(junction
-		(at 337.82 173.99)
+		(at 337.82 163.83)
 		(diameter 0)
 		(color 0 0 0 0)
@@
 	(polyline
 		(pts
-			(xy 322.58 180.34) (xy 359.41 180.34)
+			(xy 322.47 185) (xy 359.3 185)
 		)
 		(stroke
@@
 	(wire
 		(pts
-			(xy 86.36 161.29) (xy 86.36 156.21)
+			(xy 347.98 173.99) (xy 347.98 177.8)
 		)
 		(stroke
@@
 	(wire
 		(pts
-			(xy 337.82 168.91) (xy 337.82 173.99)
+			(xy 86.36 161.29) (xy 86.36 156.21)
 		)
 		(stroke
@@
 	(wire
 		(pts
-			(xy 347.98 173.99) (xy 347.98 168.91)
-		)
-		(stroke
-			(width 0)
-			(type default)
-		)
-	)
-	(wire
-		(pts
 			(xy 83.82 204.47) (xy 97.79 204.47)
 		)
@@
 	(wire
 		(pts
+			(xy 327.66 173.99) (xy 327.66 177.8)
+		)
+		(stroke
+			(width 0)
+			(type default)
+		)
+	)
+	(wire
+		(pts
 			(xy 92.71 50.8) (xy 104.14 50.8)
 		)
@@
 	(polyline
 		(pts
-			(xy 322.58 140.97) (xy 322.58 180.34)
+			(xy 322.47 140.97) (xy 322.47 185)
 		)
 		(stroke
@@
 	(wire
 		(pts
-			(xy 327.66 173.99) (xy 337.82 173.99)
+			(xy 327.66 177.8) (xy 337.82 177.8)
 		)
 		(stroke
@@
 	(wire
 		(pts
+			(xy 337.82 173.99) (xy 337.82 177.8)
+		)
+		(stroke
+			(width 0)
+			(type default)
+		)
+	)
+	(wire
+		(pts
 			(xy 132.08 44.45) (xy 140.97 44.45)
 		)
@@
 	(wire
 		(pts
+			(xy 337.82 168.91) (xy 337.82 173.99)
+		)
+		(stroke
+			(width 0)
+			(type default)
+		)
+	)
+	(wire
+		(pts
 			(xy 31.75 39.37) (xy 34.29 39.37)
 		)
@@
 	(wire
 		(pts
+			(xy 347.98 168.91) (xy 347.98 173.99)
+		)
+		(stroke
+			(width 0)
+			(type default)
+		)
+	)
+	(wire
+		(pts
 			(xy 86.36 161.29) (xy 88.9 161.29)
 		)
@@
 	(polyline
 		(pts
-			(xy 359.41 180.34) (xy 359.41 140.97)
+			(xy 359.3 185) (xy 359.3 140.97)
 		)
 		(stroke
@@
 	(wire
 		(pts
-			(xy 337.82 173.99) (xy 347.98 173.99)
+			(xy 337.82 177.8) (xy 347.98 177.8)
 		)
 		(stroke
@@
 	)
 	(symbol
+		(lib_id "Mechanical:MountingHole_Pad")
+		(at 350.52 173.99 270)
+		(unit 1)
+		(exclude_from_sim no)
+		(in_bom no)
+		(on_board yes)
+		(dnp no)
+		(property "Reference" "H12"
+			(at 354.33 173.99 90)
+			(effects
+				(font
+					(size 1.27 1.27)
+				)
+				(justify left)
+			)
+		)
+		(property "Value" "MountingHole_Pad"
+			(at 354.33 175.133 90)
+			(effects
+				(font
+					(size 1.27 1.27)
+				)
+				(justify left)
+				(hide yes)
+			)
+		)
+		(property "Footprint" "MountingHole:MountingHole_2.2mm_M2_DIN965_Pad"
+			(at 350.52 173.99 0)
+			(effects
+				(font
+					(size 1.27 1.27)
+				)
+				(hide yes)
+			)
+		)
+		(property "Datasheet" "~"
+			(at 350.52 173.99 0)
+			(effects
+				(font
+					(size 1.27 1.27)
+				)
+				(hide yes)
+			)
+		)
+		(property "Description" ""
+			(at 350.52 173.99 0)
+			(effects
+				(font
+					(size 1.27 1.27)
+				)
+				(hide yes)
+			)
+		)
+		(pin "1"
+		)
+		(instances
+			(project "AmigaPCI Mainboard"
+				(path "/72453515-27fe-4336-91f3-e3c8054f7767/4cb777ef-2899-49f4-b38f-a0c07d84fa7d"
+					(reference "H12")
+					(unit 1)
+				)
+			)
+		)
+	)
+	(symbol
 		(lib_id "Device:R_Small")
 		(at 128.27 105.41 90)
@@
 	(symbol
 		(lib_id "power:GND")
-		(at 337.82 173.99 0)
+		(at 337.82 177.8 0)
 		(unit 1)
 		(exclude_from_sim no)
@@
 		(dnp no)
 		(property "Reference" "#PWR0357"
-			(at 337.82 180.34 0)
+			(at 337.82 184.15 0)
 			(effects
 				(font
@@
 		)
 		(property "Value" "GND"
-			(at 337.947 178.3842 0)
+			(at 337.947 182.1942 0)
 			(effects
 				(font
@@
 		)
 		(property "Footprint" ""
-			(at 337.82 173.99 0)
+			(at 337.82 177.8 0)
 			(effects
 				(font
@@
 		)
 		(property "Datasheet" ""
-			(at 337.82 173.99 0)
+			(at 337.82 177.8 0)
 			(effects
 				(font
@@
 		)
 		(property "Description" ""
-			(at 337.82 173.99 0)
+			(at 337.82 177.8 0)
 			(effects
 				(font
@@
 	)
 	(symbol
+		(lib_id "Mechanical:MountingHole_Pad")
+		(at 340.36 173.99 270)
+		(unit 1)
+		(exclude_from_sim no)
+		(in_bom no)
+		(on_board yes)
+		(dnp no)
+		(property "Reference" "H11"
+			(at 344.17 173.99 90)
+			(effects
+				(font
+					(size 1.27 1.27)
+				)
+				(justify left)
+			)
+		)
+		(property "Value" "MountingHole_Pad"
+			(at 344.17 175.133 90)
+			(effects
+				(font
+					(size 1.27 1.27)
+				)
+				(justify left)
+				(hide yes)
+			)
+		)
+		(property "Footprint" "MountingHole:MountingHole_2.2mm_M2_DIN965_Pad"
+			(at 340.36 173.99 0)
+			(effects
+				(font
+					(size 1.27 1.27)
+				)
+				(hide yes)
+			)
+		)
+		(property "Datasheet" "~"
+			(at 340.36 173.99 0)
+			(effects
+				(font
+					(size 1.27 1.27)
+				)
+				(hide yes)
+			)
+		)
+		(property "Description" ""
+			(at 340.36 173.99 0)
+			(effects
+				(font
+					(size 1.27 1.27)
+				)
+				(hide yes)
+			)
+		)
+		(pin "1"
+		)
+		(instances
+			(project "AmigaPCI Mainboard"
+				(path "/72453515-27fe-4336-91f3-e3c8054f7767/4cb777ef-2899-49f4-b38f-a0c07d84fa7d"
+					(reference "H11")
+					(unit 1)
+				)
+			)
+		)
+	)
+	(symbol
 		(lib_id "power:+3V3")
 		(at 121.92 91.44 0)
@@
 	(symbol
 		(lib_id "Mechanical:MountingHole_Pad")
-		(at 350.52 173.99 270)
+		(at 330.2 173.99 270)
 		(unit 1)
 		(exclude_from_sim no)
@@
 		(dnp no)
 		(property "Reference" "H10"
-			(at 354.33 173.99 90)
+			(at 334.01 173.99 90)
 			(effects
 				(font
@@
 		)
 		(property "Value" "MountingHole_Pad"
-			(at 354.33 175.133 90)
+			(at 334.01 175.133 90)
 			(effects
 				(font
@@
 		)
 		(property "Footprint" "MountingHole:MountingHole_4mm_Pad_Via"
-			(at 350.52 173.99 0)
+			(at 330.2 173.99 0)
 			(effects
 				(font
@@
 		)
 		(property "Datasheet" "~"
-			(at 350.52 173.99 0)
+			(at 330.2 173.99 0)
 			(effects
 				(font
@@
 		)
 		(property "Description" ""
-			(at 350.52 173.99 0)
+			(at 330.2 173.99 0)
 			(effects
 				(font

Commit message: Main board routing 14-MAY-2024
Parts:
- H11, H12: footprint MountingHole:MountingHole_2.2mm_M2_DIN965_Pad -> MountingHole:MountingHole_3.5mm_Pad
Changed lines of the file:
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@@
 	(title_block
 		(title "AMIGA PCI")
-		(date "2024-04-30")
+		(date "2024-05-14")
 		(rev "3.0")
 	)
@@
 			)
 		)
-		(property "Footprint" "MountingHole:MountingHole_2.2mm_M2_DIN965_Pad"
+		(property "Footprint" "MountingHole:MountingHole_3.5mm_Pad"
 			(at 350.52 173.99 0)
 			(effects
@@
 			)
 		)
-		(property "Footprint" "MountingHole:MountingHole_2.2mm_M2_DIN965_Pad"
+		(property "Footprint" "MountingHole:MountingHole_3.5mm_Pad"
 			(at 340.36 173.99 0)
 			(effects

Commit message: Main Board Routing 22-MAY-2024
Parts:
- removed C824: 0.1uF, Capacitor_SMD:C_0603_1608Metric, symbol Device:C_Small
- removed R800: 10k, Resistor_SMD:R_0603_1608Metric, symbol Device:R
- removed U206: DS1818R-10+T&R, Package_TO_SOT_SMD:SOT-23, symbol AmigaPCI-Symbols:DS1813
- removed U818: 74AHC1G09, Package_TO_SOT_SMD:SOT-23-5, symbol 74xGxx:74AHC1G08
- added C619: 10uF, Capacitor_THT:CP_Radial_D5.0mm_P2.00mm, symbol AmigaPCI-Symbols:CP_Small-Device
- added U206: MIC1232, Package_SO:SOIC-8_3.9x4.9mm_P1.27mm, symbol AmigaPCI-Symbols:MIC1232
Connections:
- net +1V2: now also C619.1
- net +3V3: no longer C263.2
- net +5V: now also C263.1, U206.8 (VCC)
- net GND: now also C263.2, CN206.1 (Pin_1), C619.2, U206.2 (TD), U206.3 (TOL), U206.4 (GND); no longer C263.1, CN206.2 (Pin_2)
- net RSTBTN: now also CN206.2 (Pin_2), U206.1 (~{PBRST}); no longer CN206.1 (Pin_1)
- net _BTNRST: now also U206.6 (~{RESET})
- new net CLK40: U206.7 (~{ST})
- no-connect marks 24 -> 25
Other:
- moved on the sheet: C263, C610, CN206, D603, R603

Commit message: Routing 24-MAY-2024
Parts:
- removed J1: _TA, Connector_PinHeader_2.54mm:PinHeader_1x01_P2.54mm_Vertical, symbol Connector_Generic:Conn_01x01
- removed J12: _TBI, Connector_PinHeader_2.54mm:PinHeader_1x01_P2.54mm_Vertical, symbol Connector_Generic:Conn_01x01
- removed J5: _TS, Connector_PinHeader_2.54mm:PinHeader_1x01_P2.54mm_Vertical, symbol Connector_Generic:Conn_01x01
- removed J6: _TIP, Connector_PinHeader_2.54mm:PinHeader_1x01_P2.54mm_Vertical, symbol Connector_Generic:Conn_01x01
- removed J7: TT0, Connector_PinHeader_2.54mm:PinHeader_1x01_P2.54mm_Vertical, symbol Connector_Generic:Conn_01x01
- removed J8: TT1, Connector_PinHeader_2.54mm:PinHeader_1x01_P2.54mm_Vertical, symbol Connector_Generic:Conn_01x01

Commit message: Main Board Routing 25-MAY-2024
Parts:
- R601, R603: footprint Resistor_SMD:R_0603_1608Metric -> Resistor_SMD:R_0805_2012Metric
Other:
- note added: "R601, R603 = 1/4 WATT"
Changed lines of the file:
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@@
 		)
 	)
+	(text "R601, R603 = 1/4 WATT"
+		(exclude_from_sim no)
+		(at 156.21 102.616 0)
+		(effects
+			(font
+				(size 1.27 1.27)
+			)
+		)
+	)
 	(text "POWER RAIL INDICATORS"
 		(exclude_from_sim no)
@@
 			)
 		)
-		(property "Footprint" "Resistor_SMD:R_0603_1608Metric"
+		(property "Footprint" "Resistor_SMD:R_0805_2012Metric"
 			(at 128.27 116.84 0)
 			(effects
@@
 			)
 		)
-		(property "Footprint" "Resistor_SMD:R_0603_1608Metric"
+		(property "Footprint" "Resistor_SMD:R_0805_2012Metric"
 			(at 153.67 95.25 0)
 			(effects
