File: KiCAD/AmigaPCI Mainboard-KiCAD REV 30/audio.kicad_sch (KiCad schematic)
At the start: 60 parts, among them CN500 DSP/DVD (RGGL), CN501 AudioJack, Q500 MMBFJ211, Q501 MMBFJ211, Q502 MMBT3906, U220 74LVC08, U500 8364, U501 LF347, U502 LM833

Commit message: Main Board Routing 22-MAY-2024
Connections:
- net _INT2: now also U220.8; no longer U220.11
- net _INT2A: now also U220.9; no longer U220.12
- net _INT2B: now also U220.10; no longer U220.13
Changed lines of the file:
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@@
 	(title_block
 		(title "AMIGA PCI")
-		(date "2024-05-18")
+		(date "2024-05-22")
 		(rev "3.0")
 	)
@@
 	(rectangle
 		(start 267.7668 194.564)
-		(end 320.7512 221.8944)
+		(end 325.7 221.8944)
 		(stroke
 			(width 0)
@@
 		(lib_id "74xx:74LS08")
 		(at 298.3484 213.2584 0)
-		(unit 4)
+		(unit 3)
 		(exclude_from_sim no)
 		(in_bom yes)
@@
 				(path "/72453515-27fe-4336-91f3-e3c8054f7767/71ea5834-c2f1-44b0-9a09-0538600b01fd"
 					(reference "U220")
-					(unit 4)
+					(unit 3)
 				)
 			)

Commit message: Main Board Routing 25-MAY-2024
Parts:
- added R249: 1k, Resistor_SMD:R_0603_1608Metric, symbol Device:R
Connections:
- net +5V: now also R249.1
- net _INT2A: now also R249.2
Changed lines of the file:
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@@
 	)
 	(junction
+		(at 288.29 210.82)
+		(diameter 0)
+		(color 0 0 0 0)
+	)
+	(junction
 		(at 184.023 92.075)
 		(diameter 0)
@@
 	(wire
 		(pts
-			(xy 284.2768 215.7984) (xy 290.7284 215.7984)
+			(xy 284.48 215.9) (xy 290.83 215.9)
 		)
 		(stroke
@@
 	(wire
 		(pts
+			(xy 288.29 210.82) (xy 290.83 210.82)
+		)
+		(stroke
+			(width 0)
+			(type default)
+		)
+	)
+	(wire
+		(pts
 			(xy 232.41 135.509) (xy 251.587 135.509)
 		)
@@
 	(wire
 		(pts
-			(xy 284.2768 210.7184) (xy 290.7284 210.7184)
+			(xy 284.48 210.82) (xy 288.29 210.82)
 		)
 		(stroke
@@
 	(wire
 		(pts
-			(xy 305.9684 213.2584) (xy 312.42 213.2584)
+			(xy 306.07 213.36) (xy 312.42 213.36)
 		)
 		(stroke
@@
 	(text "_INT2"
 		(exclude_from_sim no)
-		(at 284.734 200.7616 0)
+		(at 297.18 200.66 0)
 		(effects
 			(font
@@
 	(global_label "_INT2A"
 		(shape input)
-		(at 284.2768 210.7184 180)
+		(at 284.48 210.82 180)
 		(fields_autoplaced yes)
 		(effects
@@
 		)
 		(property "Intersheetrefs" "${INTERSHEET_REFS}"
-			(at 275.123 210.7184 0)
+			(at 275.3262 210.82 0)
 			(effects
 				(font
@@
 	(global_label "_INT2"
 		(shape output)
-		(at 312.42 213.2584 0)
+		(at 312.42 213.36 0)
 		(fields_autoplaced yes)
 		(effects
@@
 		)
 		(property "Intersheetrefs" "${INTERSHEET_REFS}"
-			(at 320.4852 213.2584 0)
+			(at 320.4852 213.36 0)
 			(effects
 				(font
@@
 	(global_label "_INT2B"
 		(shape input)
-		(at 284.2768 215.7984 180)
+		(at 284.48 215.9 180)
 		(fields_autoplaced yes)
 		(effects
@@
 		)
 		(property "Intersheetrefs" "${INTERSHEET_REFS}"
-			(at 274.9416 215.7984 0)
+			(at 275.1448 215.9 0)
 			(effects
 				(font
@@
 	(symbol
 		(lib_id "74xx:74LS08")
-		(at 298.3484 213.2584 0)
+		(at 298.45 213.36 0)
 		(unit 3)
 		(exclude_from_sim no)
@@
 		(fields_autoplaced yes)
 		(property "Reference" "U220"
-			(at 298.3401 204.6224 0)
+			(at 298.4417 204.724 0)
 			(effects
 				(font
@@
 		)
 		(property "Value" "74LVC08"
-			(at 298.3401 207.1624 0)
+			(at 298.4417 207.264 0)
 			(effects
 				(font
@@
 		)
 		(property "Footprint" "Package_SO:TSSOP-14_4.4x5mm_P0.65mm"
-			(at 298.3484 213.2584 0)
+			(at 298.45 213.36 0)
 			(effects
 				(font
@@
 		)
 		(property "Datasheet" "http://www.ti.com/lit/gpn/sn74LS08"
-			(at 298.3484 213.2584 0)
+			(at 298.45 213.36 0)
 			(effects
 				(font
@@
 		)
 		(property "Description" ""
-			(at 298.3484 213.2584 0)
+			(at 298.45 213.36 0)
 			(effects
 				(font
@@
 	)
 	(symbol
+		(lib_name "+5V_1")
+		(lib_id "power:+5V")
+		(at 288.29 203.2 0)
+		(unit 1)
+		(exclude_from_sim no)
+		(in_bom yes)
+		(on_board yes)
+		(dnp no)
+		(property "Reference" "#PWR0136"
+			(at 288.29 207.01 0)
+			(effects
+				(font
+					(size 1.27 1.27)
+				)
+				(hide yes)
+			)
+		)
+		(property "Value" "+5V"
+			(at 288.29 199.136 0)
+			(effects
+				(font
+					(size 1.27 1.27)
+				)
+			)
+		)
+		(property "Footprint" ""
+			(at 288.29 203.2 0)
+			(effects
+				(font
+					(size 1.27 1.27)
+				)
+				(hide yes)
+			)
+		)
+		(property "Datasheet" ""
+			(at 288.29 203.2 0)
+			(effects
+				(font
+					(size 1.27 1.27)
+				)
+				(hide yes)
+			)
+		)
+		(property "Description" "Power symbol creates a global label with name \"+5V\""
+			(at 288.29 203.2 0)
+			(effects
+				(font
+					(size 1.27 1.27)
+				)
+				(hide yes)
+			)
+		)
+		(pin "1"
+		)
+		(instances
+			(project "AmigaPCI Mainboard"
+				(path "/72453515-27fe-4336-91f3-e3c8054f7767/71ea5834-c2f1-44b0-9a09-0538600b01fd"
+					(reference "#PWR0136")
+					(unit 1)
+				)
+			)
+		)
+	)
+	(symbol
 		(lib_id "Device:R")
 		(at 151.765 123.317 0)
@@
 					(unit 1)
 				)
+			)
+		)
+	)
+	(symbol
+		(lib_id "Device:R")
+		(at 288.29 207.01 0)
+		(unit 1)
+		(exclude_from_sim no)
+		(in_bom yes)
+		(on_board yes)
+		(dnp no)
+		(property "Reference" "R249"
+			(at 286.258 209.55 90)
+			(effects
+				(font
+					(size 1.27 1.27)
+				)
+				(justify left)
+			)
+		)
+		(property "Value" "1k"
+			(at 288.29 208.28 90)
+			(effects
+				(font
+					(size 1.27 1.27)
+				)
+				(justify left)
+			)
+		)
+		(property "Footprint" "Resistor_SMD:R_0603_1608Metric"
+			(at 286.512 207.01 90)
+			(effects
+				(font
+					(size 1.27 1.27)
+				)
+				(hide yes)
+			)
+		)
+		(property "Datasheet" "~"
+			(at 288.29 207.01 0)
+			(effects
+				(font
+					(size 1.27 1.27)
+				)
+				(hide yes)
+			)
+		)
+		(property "Description" ""
+			(at 288.29 207.01 0)
+			(effects
+				(font
+					(size 1.27 1.27)
+				)
+				(hide yes)
+			)
+		)
+		(pin "1"
+		)
+		(pin "2"
+		)
+		(instances
+			(project "AmigaPCI Mainboard"
+				(path "/72453515-27fe-4336-91f3-e3c8054f7767/71ea5834-c2f1-44b0-9a09-0538600b01fd"
+					(reference "R249")
+					(unit 1)
+				)
