File: KiCAD/AmigaPCI Mainboard-KiCAD REV 30/mc68040_level_shift.kicad_sch (KiCad schematic)
At the start: 28 parts, among them U800 74LVC1G17, U801 74LVC1G17, U802 SN74LVC16T245DLR, U803 SN74LVC16T245DLR, U804 SN74LVC16T245DLR, U805 SN74LVC16T245DLR, U806 74LVC245, U807 74LVC245, U808 74LVC245, U809 74LVC245, U810 74LVC245, U811 74LVC245

Commit message: Rev 3.0 PCB Routing 12-MAY-2024
Connections:
- net A0: now also U805.26 (2A8); no longer U805.47 (1A1)
- net A1: now also U805.44 (1A3); no longer U805.40 (1A6)
- net A10: now also U804.35 (2A2); no longer U805.44 (1A3)
- net A11: now also U804.36 (2A1); no longer U805.43 (1A4)
- net A12: now also U804.37 (1A8); no longer U805.46 (1A2)
- net A13: now also U804.38 (1A7); no longer U805.41 (1A5)
- net A14: now also U804.40 (1A6); no longer U805.37 (1A8)
- net A15: now also U804.41 (1A5); no longer U805.33 (2A3)
- net A16: now also U804.43 (1A4); no longer U805.35 (2A2)
- net A17: now also U804.44 (1A3); no longer U805.27 (2A7)
- net A19: now also U804.47 (1A1); no longer U805.29 (2A6)
- net A2: now also U805.46 (1A2); no longer U805.38 (1A7)
- net A20: now also U805.27 (2A7); no longer U804.41 (1A5)
- net A21: now also U805.30 (2A5); no longer U804.37 (1A8)
- net A22: now also U805.41 (1A5); no longer U804.33 (2A3)
- net A23: now also U805.29 (2A6); no longer U804.40 (1A6)
- net A24: now also U805.37 (1A8); no longer U804.26 (2A8)
- net A25: now also U805.32 (2A4); no longer U804.38 (1A7)
- net A26: now also U805.40 (1A6); no longer U804.35 (2A2)
- net A27: now also U805.33 (2A3); no longer U804.30 (2A5)
- net A28: now also U805.43 (1A4); no longer U804.36 (2A1)
- net A29: now also U805.38 (1A7); no longer U804.32 (2A4)
- net A3: now also U805.47 (1A1); no longer U805.36 (2A1)
- net A30: now also U805.36 (2A1); no longer U804.27 (2A7)
- net A31: now also U805.35 (2A2); no longer U805.30 (2A5)
- net A4: now also U804.26 (2A8); no longer U805.32 (2A4)
- net A5: now also U804.27 (2A7); no longer U805.26 (2A8)
- net A6: now also U804.29 (2A6); no longer U804.47 (1A1)
- net A7: now also U804.30 (2A5); no longer U804.43 (1A4)
- net A8: now also U804.32 (2A4); no longer U804.29 (2A6)
- net A9: now also U804.33 (2A3); no longer U804.44 (1A3)
- net D0: now also U802.26 (2A8); no longer U802.46 (1A2)
- net D1: now also U802.27 (2A7); no longer U802.43 (1A4)
- net D10: now also U802.40 (1A6); no longer U802.33 (2A3)
- net D11: now also U802.41 (1A5); no longer U802.32 (2A4)
- net D12: now also U802.43 (1A4); no longer U803.26 (2A8)
- net D13: now also U802.44 (1A3); no longer U803.29 (2A6)
- net D14: now also U802.46 (1A2); no longer U803.30 (2A5)
- net D15: now also U802.47 (1A1); no longer U803.33 (2A3)
- net D16: now also U803.26 (2A8); no longer U803.27 (2A7)
- net D17: now also U803.27 (2A7); no longer U803.35 (2A2)
- net D18: now also U803.29 (2A6); no longer U803.32 (2A4)
- net D19: now also U803.30 (2A5); no longer U803.37 (1A8)
- net D2: now also U802.29 (2A6); no longer U802.47 (1A1)
- net D20: now also U803.32 (2A4); no longer U803.41 (1A5)
- net D21: now also U803.33 (2A3); no longer U803.46 (1A2)
- net D22: now also U803.35 (2A2); no longer U803.40 (1A6)
- net D24: now also U803.37 (1A8); no longer U802.27 (2A7)
- net D26: now also U803.40 (1A6); no longer U802.29 (2A6)
- net D27: now also U803.41 (1A5); no longer U803.43 (1A4)
- net D28: now also U803.43 (1A4); no longer U802.30 (2A5)
- net D3: now also U802.30 (2A5); no longer U802.40 (1A6)
- net D30: now also U803.46 (1A2); no longer U803.47 (1A1)
- net D31: now also U803.47 (1A1); no longer U802.26 (2A8)
- net D4: now also U802.32 (2A4); no longer U802.41 (1A5)
- net D5: now also U802.33 (2A3); no longer U802.38 (1A7)
- net D6: now also U802.35 (2A2); no longer U802.37 (1A8)
- net D8: now also U802.37 (1A8); no longer U802.44 (1A3)
- net D9: now also U802.38 (1A7); no longer U802.35 (2A2)
- net GND: no longer U802.25 (2OE), U802.48 (1OE), U803.25 (2OE), U803.48 (1OE)
- net LVD0: now also U802.23 (2B8); no longer U802.3 (1B2)
- net LVD1: now also U802.22 (2B7); no longer U802.6 (1B4)
- net LVD10: now also U802.9 (1B6); no longer U802.16 (2B3)
- net LVD11: now also U802.8 (1B5); no longer U802.17 (2B4)
- net LVD12: now also U802.6 (1B4); no longer U803.23 (2B8)
- net LVD13: now also U802.5 (1B3); no longer U803.20 (2B6)
- net LVD14: now also U802.3 (1B2); no longer U803.19 (2B5)
- net LVD15: now also U802.2 (1B1); no longer U803.16 (2B3)
- net LVD16: now also U803.23 (2B8); no longer U803.22 (2B7)
- net LVD17: now also U803.22 (2B7); no longer U803.14 (2B2)
- net LVD18: now also U803.20 (2B6); no longer U803.17 (2B4)
- net LVD19: now also U803.19 (2B5); no longer U803.12 (1B8)
- net LVD2: now also U802.20 (2B6); no longer U802.2 (1B1)
- net LVD20: now also U803.17 (2B4); no longer U803.8 (1B5)
- net LVD21: now also U803.16 (2B3); no longer U803.3 (1B2)
- net LVD22: now also U803.14 (2B2); no longer U803.9 (1B6)
- net LVD24: now also U803.12 (1B8); no longer U802.22 (2B7)
- net LVD26: now also U803.9 (1B6); no longer U802.20 (2B6)
- net LVD27: now also U803.8 (1B5); no longer U803.6 (1B4)
- net LVD28: now also U803.6 (1B4); no longer U802.19 (2B5)
- net LVD3: now also U802.19 (2B5); no longer U802.9 (1B6)
- net LVD30: now also U803.3 (1B2); no longer U803.2 (1B1)
- net LVD31: now also U803.2 (1B1); no longer U802.23 (2B8)
- net LVD4: now also U802.17 (2B4); no longer U802.8 (1B5)
- net LVD5: now also U802.16 (2B3); no longer U802.11 (1B7)
- net LVD6: now also U802.14 (2B2); no longer U802.12 (1B8)
- net LVD8: now also U802.12 (1B8); no longer U802.5 (1B3)
- net LVD9: now also U802.11 (1B7); no longer U802.14 (2B2)
- new net _BUFEN: U802.25 (2OE), U802.48 (1OE), U803.25 (2OE), U803.48 (1OE)

Commit message: Main Board Routing 18-MAY-2024
Connections:
- net LVA0: now also U805.23 (2B8); no longer U805.2 (1B1)
- net LVA1: now also U805.5 (1B3); no longer U805.9 (1B6)
- net LVA10: now also U804.14 (2B2); no longer U805.5 (1B3)
- net LVA11: now also U804.13 (2B1); no longer U805.6 (1B4)
- net LVA12: now also U804.12 (1B8); no longer U805.3 (1B2)
- net LVA13: now also U804.11 (1B7); no longer U805.8 (1B5)
- net LVA14: now also U804.9 (1B6); no longer U805.12 (1B8)
- net LVA15: now also U804.8 (1B5); no longer U805.16 (2B3)
- net LVA16: now also U804.6 (1B4); no longer U805.14 (2B2)
- net LVA17: now also U804.5 (1B3); no longer U805.22 (2B7)
- net LVA19: now also U804.2 (1B1); no longer U805.20 (2B6)
- net LVA2: now also U805.3 (1B2); no longer U805.11 (1B7)
- net LVA20: now also U805.22 (2B7); no longer U804.8 (1B5)
- net LVA21: now also U805.19 (2B5); no longer U804.12 (1B8)
- net LVA22: now also U805.8 (1B5); no longer U804.16 (2B3)
- net LVA23: now also U805.20 (2B6); no longer U804.9 (1B6)
- net LVA24: now also U805.12 (1B8); no longer U804.23 (2B8)
- net LVA25: now also U805.17 (2B4); no longer U804.11 (1B7)
- net LVA26: now also U805.9 (1B6); no longer U804.14 (2B2)
- net LVA27: now also U805.16 (2B3); no longer U804.19 (2B5)
- net LVA28: now also U805.6 (1B4); no longer U804.13 (2B1)
- net LVA29: now also U805.11 (1B7); no longer U804.17 (2B4)
- net LVA3: now also U805.2 (1B1); no longer U805.13 (2B1)
- net LVA30: now also U805.13 (2B1); no longer U804.22 (2B7)
- net LVA31: now also U805.14 (2B2); no longer U805.19 (2B5)
- net LVA4: now also U804.23 (2B8); no longer U805.17 (2B4)
- net LVA5: now also U804.22 (2B7); no longer U805.23 (2B8)
- net LVA6: now also U804.20 (2B6); no longer U804.2 (1B1)
- net LVA7: now also U804.19 (2B5); no longer U804.6 (1B4)
- net LVA8: now also U804.17 (2B4); no longer U804.20 (2B6)
- net LVA9: now also U804.16 (2B3); no longer U804.5 (1B3)
Changed lines of the file:
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@@
 	(title_block
 		(title "AMIGA PCI")
-		(date "2024-05-14")
+		(date "2024-05-18")
 		(rev "3.0")
 	)
@@
 	)
 	(label "LVA22"
-		(at 120.65 88.9 0)
+		(at 120.65 142.24 0)
 		(fields_autoplaced yes)
 		(effects
@@
 	)
 	(label "LVA2"
-		(at 120.65 149.86 0)
+		(at 120.65 129.54 0)
 		(fields_autoplaced yes)
 		(effects
@@
 	)
 	(label "LVA31"
-		(at 120.65 170.18 0)
+		(at 120.65 157.48 0)
 		(fields_autoplaced yes)
 		(effects
@@
 	)
 	(label "LVA9"
-		(at 120.65 60.96 0)
+		(at 120.65 88.9 0)
 		(fields_autoplaced yes)
 		(effects
@@
 	)
 	(label "LVA27"
-		(at 120.65 96.52 0)
+		(at 120.65 162.56 0)
 		(fields_autoplaced yes)
 		(effects
@@
 	)
 	(label "LVA11"
-		(at 120.65 137.16 0)
+		(at 120.65 81.28 0)
 		(fields_autoplaced yes)
 		(effects
@@
 	)
 	(label "LVA16"
-		(at 120.65 157.48 0)
+		(at 120.65 63.5 0)
 		(fields_autoplaced yes)
 		(effects
@@
 	)
 	(label "LVA0"
-		(at 120.65 127 0)
+		(at 120.65 180.34 0)
 		(fields_autoplaced yes)
 		(effects
@@
 	)
 	(label "LVA17"
-		(at 120.65 177.8 0)
+		(at 120.65 60.96 0)
 		(fields_autoplaced yes)
 		(effects
@@
 	)
 	(label "LVA20"
-		(at 120.65 68.58 0)
+		(at 120.65 177.8 0)
 		(fields_autoplaced yes)
 		(effects
@@
 	)
 	(label "LVA26"
-		(at 120.65 83.82 0)
+		(at 120.65 144.78 0)
 		(fields_autoplaced yes)
 		(effects
@@
 	)
 	(label "LVA5"
-		(at 120.65 180.34 0)
+		(at 120.65 104.14 0)
 		(fields_autoplaced yes)
 		(effects
@@
 	)
 	(label "LVA24"
-		(at 120.65 106.68 0)
+		(at 120.65 152.4 0)
 		(fields_autoplaced yes)
 		(effects
@@
 	)
 	(label "LVA25"
-		(at 120.65 76.2 0)
+		(at 120.65 165.1 0)
 		(fields_autoplaced yes)
 		(effects
@@
 	)
 	(label "LVA30"
-		(at 120.65 104.14 0)
+		(at 120.65 154.94 0)
 		(fields_autoplaced yes)
 		(effects
@@
 	)
 	(label "LVA4"
-		(at 120.65 165.1 0)
+		(at 120.65 106.68 0)
 		(fields_autoplaced yes)
 		(effects
@@
 	)
 	(label "LVA6"
-		(at 120.65 53.34 0)
+		(at 120.65 99.06 0)
 		(fields_autoplaced yes)
 		(effects
@@
 	)
 	(label "LVA23"
-		(at 120.65 71.12 0)
+		(at 120.65 172.72 0)
 		(fields_autoplaced yes)
 		(effects
@@
 	)
 	(label "LVA1"
-		(at 120.65 144.78 0)
+		(at 120.65 134.62 0)
 		(fields_autoplaced yes)
 		(effects
@@
 	)
 	(label "LVA3"
-		(at 120.65 154.94 0)
+		(at 120.65 127 0)
 		(fields_autoplaced yes)
 		(effects
@@
 	)
 	(label "LVA15"
-		(at 120.65 162.56 0)
+		(at 120.65 68.58 0)
 		(fields_autoplaced yes)
 		(effects
@@
 	)
 	(label "LVA19"
-		(at 120.65 172.72 0)
+		(at 120.65 53.34 0)
 		(fields_autoplaced yes)
 		(effects
@@
 	)
 	(label "LVA7"
-		(at 120.65 63.5 0)
+		(at 120.65 96.52 0)
 		(fields_autoplaced yes)
 		(effects
@@
 	)
 	(label "LVA12"
-		(at 120.65 129.54 0)
+		(at 120.65 78.74 0)
 		(fields_autoplaced yes)
 		(effects
@@
 	)
 	(label "LVA14"
-		(at 120.65 152.4 0)
+		(at 120.65 71.12 0)
 		(fields_autoplaced yes)
 		(effects
@@
 	)
 	(label "LVA29"
-		(at 120.65 91.44 0)
+		(at 120.65 149.86 0)
 		(fields_autoplaced yes)
 		(effects
@@
 	)
 	(label "LVA13"
-		(at 120.65 142.24 0)
+		(at 120.65 76.2 0)
 		(fields_autoplaced yes)
 		(effects
@@
 	)
 	(label "LVA8"
-		(at 120.65 99.06 0)
+		(at 120.65 91.44 0)
 		(fields_autoplaced yes)
 		(effects
@@
 	)
 	(label "LVA10"
-		(at 120.65 134.62 0)
+		(at 120.65 83.82 0)
 		(fields_autoplaced yes)
 		(effects
@@
 	)
 	(label "LVA28"
-		(at 120.65 81.28 0)
+		(at 120.65 137.16 0)
 		(fields_autoplaced yes)
 		(effects
@@
 	)
 	(label "LVA21"
-		(at 120.65 78.74 0)
+		(at 120.65 170.18 0)
 		(fields_autoplaced yes)
 		(effects

Commit message: Main Board Routing 19-MAY-2024
Connections:
- net +3V3: now also U802.31 (VCCA), U802.42 (VCCA), U803.31 (VCCA), U803.42 (VCCA), U804.31 (VCCA), U804.42 (VCCA), U805.31 (VCCA), U805.42 (VCCA); no longer U802.18 (VCCB), U802.7 (VCCB), U803.18 (VCCB), U803.7 (VCCB), U804.18 (VCCB), U804.7 (VCCB), U805.18 (VCCB), U805.7 (VCCB)
- net +5V: now also U802.18 (VCCB), U802.7 (VCCB), U803.18 (VCCB), U803.7 (VCCB), U804.18 (VCCB), U804.7 (VCCB), U805.18 (VCCB), U805.7 (VCCB); no longer U802.31 (VCCA), U802.42 (VCCA), U803.31 (VCCA), U803.42 (VCCA), U804.31 (VCCA), U804.42 (VCCA), U805.31 (VCCA), U805.42 (VCCA)
- net A0: now also U805.2 (1B1); no longer U805.26 (2A8)
- net A1: now also U805.20 (2B6); no longer U805.44 (1A3)
- net A10: now also U804.11 (1B7); no longer U804.35 (2A2)
- net A11: now also U804.12 (1B8); no longer U804.36 (2A1)
- net A12: now also U804.13 (2B1); no longer U804.37 (1A8)
- net A13: now also U804.14 (2B2); no longer U804.38 (1A7)
- net A14: now also U804.16 (2B3); no longer U804.40 (1A6)
- net A15: now also U804.17 (2B4); no longer U804.41 (1A5)
- net A16: now also U804.19 (2B5); no longer U804.43 (1A4)
- net A17: now also U804.20 (2B6); no longer U804.44 (1A3)
- net A18: now also U804.22 (2B7); no longer U804.46 (1A2)
- net A19: now also U804.23 (2B8); no longer U804.47 (1A1)
- net A2: now also U805.22 (2B7); no longer U805.46 (1A2)
- net A20: now also U805.3 (1B2); no longer U805.27 (2A7)
- net A21: now also U805.6 (1B4); no longer U805.30 (2A5)
- net A22: now also U805.17 (2B4); no longer U805.41 (1A5)
- net A23: now also U805.5 (1B3); no longer U805.29 (2A6)
- net A24: now also U805.13 (2B1); no longer U805.37 (1A8)
- net A25: now also U805.8 (1B5); no longer U805.32 (2A4)
- net A26: now also U805.16 (2B3); no longer U805.40 (1A6)
- net A27: now also U805.9 (1B6); no longer U805.33 (2A3)
- net A28: now also U805.19 (2B5); no longer U805.43 (1A4)
- net A29: now also U805.14 (2B2); no longer U805.38 (1A7)
- net A3: now also U805.23 (2B8); no longer U805.47 (1A1)
- net A30: now also U805.12 (1B8); no longer U805.36 (2A1)
- net A31: now also U805.11 (1B7); no longer U805.35 (2A2)
- net A4: now also U804.2 (1B1); no longer U804.26 (2A8)
- net A5: now also U804.3 (1B2); no longer U804.27 (2A7)
- net A6: now also U804.5 (1B3); no longer U804.29 (2A6)
- net A7: now also U804.6 (1B4); no longer U804.30 (2A5)
- net A8: now also U804.8 (1B5); no longer U804.32 (2A4)
- net A9: now also U804.9 (1B6); no longer U804.33 (2A3)
- net D0: now also U802.2 (1B1); no longer U802.26 (2A8)
- net D1: now also U802.3 (1B2); no longer U802.27 (2A7)
- net D10: now also U802.16 (2B3); no longer U802.40 (1A6)
- net D11: now also U802.17 (2B4); no longer U802.41 (1A5)
- net D12: now also U802.19 (2B5); no longer U802.43 (1A4)
- net D13: now also U802.20 (2B6); no longer U802.44 (1A3)
- net D14: now also U802.22 (2B7); no longer U802.46 (1A2)
- net D15: now also U802.23 (2B8); no longer U802.47 (1A1)
- net D16: now also U803.2 (1B1); no longer U803.26 (2A8)
- net D17: now also U803.3 (1B2); no longer U803.27 (2A7)
- net D18: now also U803.5 (1B3); no longer U803.29 (2A6)
- net D19: now also U803.6 (1B4); no longer U803.30 (2A5)
- net D2: now also U802.5 (1B3); no longer U802.29 (2A6)
- net D20: now also U803.8 (1B5); no longer U803.32 (2A4)
- net D21: now also U803.9 (1B6); no longer U803.33 (2A3)
- net D22: now also U803.11 (1B7); no longer U803.35 (2A2)
- net D23: now also U803.12 (1B8); no longer U803.36 (2A1)
- net D24: now also U803.13 (2B1); no longer U803.37 (1A8)
- net D25: now also U803.14 (2B2); no longer U803.38 (1A7)
- net D26: now also U803.16 (2B3); no longer U803.40 (1A6)
- net D27: now also U803.17 (2B4); no longer U803.41 (1A5)
- net D28: now also U803.19 (2B5); no longer U803.43 (1A4)
- net D29: now also U803.20 (2B6); no longer U803.44 (1A3)
- net D3: now also U802.6 (1B4); no longer U802.30 (2A5)
- net D30: now also U803.22 (2B7); no longer U803.46 (1A2)
- net D31: now also U803.23 (2B8); no longer U803.47 (1A1)
- net D4: now also U802.8 (1B5); no longer U802.32 (2A4)
- net D5: now also U802.9 (1B6); no longer U802.33 (2A3)
- net D6: now also U802.11 (1B7); no longer U802.35 (2A2)
- net D7: now also U802.12 (1B8); no longer U802.36 (2A1)
- net D8: now also U802.13 (2B1); no longer U802.37 (1A8)
- net D9: now also U802.14 (2B2); no longer U802.38 (1A7)
- net GND: no longer U809.16 (B2), U809.4 (A2)
- net LVA0: now also U805.47 (1A1); no longer U805.23 (2B8)
- net LVA1: now also U805.29 (2A6); no longer U805.5 (1B3)
- net LVA10: now also U804.38 (1A7); no longer U804.14 (2B2)
- net LVA11: now also U804.37 (1A8); no longer U804.13 (2B1)
- net LVA12: now also U804.36 (2A1); no longer U804.12 (1B8)
- net LVA13: now also U804.35 (2A2); no longer U804.11 (1B7)
- net LVA14: now also U804.33 (2A3); no longer U804.9 (1B6)
- net LVA15: now also U804.32 (2A4); no longer U804.8 (1B5)
- net LVA16: now also U804.30 (2A5); no longer U804.6 (1B4)
- net LVA17: now also U804.29 (2A6); no longer U804.5 (1B3)
- net LVA18: now also U804.27 (2A7); no longer U804.3 (1B2)
- net LVA19: now also U804.26 (2A8); no longer U804.2 (1B1)
- net LVA2: now also U805.27 (2A7); no longer U805.3 (1B2)
- net LVA20: now also U805.46 (1A2); no longer U805.22 (2B7)
- net LVA21: now also U805.43 (1A4); no longer U805.19 (2B5)
- net LVA22: now also U805.32 (2A4); no longer U805.8 (1B5)
- net LVA23: now also U805.44 (1A3); no longer U805.20 (2B6)
- net LVA24: now also U805.36 (2A1); no longer U805.12 (1B8)
- net LVA25: now also U805.41 (1A5); no longer U805.17 (2B4)
- net LVA26: now also U805.33 (2A3); no longer U805.9 (1B6)
- net LVA27: now also U805.40 (1A6); no longer U805.16 (2B3)
- net LVA28: now also U805.30 (2A5); no longer U805.6 (1B4)
- net LVA29: now also U805.35 (2A2); no longer U805.11 (1B7)
- net LVA3: now also U805.26 (2A8); no longer U805.2 (1B1)
- net LVA30: now also U805.37 (1A8); no longer U805.13 (2B1)
- net LVA31: now also U805.38 (1A7); no longer U805.14 (2B2)
- net LVA4: now also U804.47 (1A1); no longer U804.23 (2B8)
- net LVA5: now also U804.46 (1A2); no longer U804.22 (2B7)
- net LVA6: now also U804.44 (1A3); no longer U804.20 (2B6)
- net LVA7: now also U804.43 (1A4); no longer U804.19 (2B5)
- net LVA8: now also U804.41 (1A5); no longer U804.17 (2B4)
- net LVA9: now also U804.40 (1A6); no longer U804.16 (2B3)
- net LVD0: now also U802.47 (1A1); no longer U802.23 (2B8)
- net LVD1: now also U802.46 (1A2); no longer U802.22 (2B7)
- net LVD10: now also U802.33 (2A3); no longer U802.9 (1B6)
- net LVD11: now also U802.32 (2A4); no longer U802.8 (1B5)
- net LVD12: now also U802.30 (2A5); no longer U802.6 (1B4)
- net LVD13: now also U802.29 (2A6); no longer U802.5 (1B3)
- net LVD14: now also U802.27 (2A7); no longer U802.3 (1B2)
- net LVD15: now also U802.26 (2A8); no longer U802.2 (1B1)
- net LVD16: now also U803.47 (1A1); no longer U803.23 (2B8)
- net LVD17: now also U803.46 (1A2); no longer U803.22 (2B7)
- net LVD18: now also U803.44 (1A3); no longer U803.20 (2B6)
- net LVD19: now also U803.43 (1A4); no longer U803.19 (2B5)
- net LVD2: now also U802.44 (1A3); no longer U802.20 (2B6)
- net LVD20: now also U803.41 (1A5); no longer U803.17 (2B4)
- net LVD21: now also U803.40 (1A6); no longer U803.16 (2B3)
- net LVD22: now also U803.38 (1A7); no longer U803.14 (2B2)
- net LVD23: now also U803.37 (1A8); no longer U803.13 (2B1)
- net LVD24: now also U803.36 (2A1); no longer U803.12 (1B8)
- net LVD25: now also U803.35 (2A2); no longer U803.11 (1B7)
- net LVD26: now also U803.33 (2A3); no longer U803.9 (1B6)
- net LVD27: now also U803.32 (2A4); no longer U803.8 (1B5)
- net LVD28: now also U803.30 (2A5); no longer U803.6 (1B4)
- net LVD29: now also U803.29 (2A6); no longer U803.5 (1B3)
- net LVD3: now also U802.43 (1A4); no longer U802.19 (2B5)
- net LVD30: now also U803.27 (2A7); no longer U803.3 (1B2)
- net LVD31: now also U803.26 (2A8); no longer U803.2 (1B1)
- net LVD4: now also U802.41 (1A5); no longer U802.17 (2B4)
- net LVD5: now also U802.40 (1A6); no longer U802.16 (2B3)
- net LVD6: now also U802.38 (1A7); no longer U802.14 (2B2)
- net LVD7: now also U802.37 (1A8); no longer U802.13 (2B1)
- net LVD8: now also U802.36 (2A1); no longer U802.12 (1B8)
- net LVD9: now also U802.35 (2A2); no longer U802.11 (1B7)
- net LVR_W: no longer U802.1 (1DIR), U802.24 (2DIR), U803.1 (1DIR), U803.24 (2DIR), U804.1 (1DIR), U804.24 (2DIR), U805.1 (1DIR), U805.24 (2DIR)
- net R_W: now also U802.1 (1DIR), U802.24 (2DIR), U803.1 (1DIR), U803.24 (2DIR)
- net _BG: now also U804.1 (1DIR), U804.24 (2DIR), U805.1 (1DIR), U805.24 (2DIR)
- new net _LOCKE: U809.16 (B2)
- new net _LVLOCKE: U809.4 (A2)
