File: KiCAD/AmigaPCI Mainboard-KiCAD REV 30/serial.kicad_sch (KiCad schematic)
At the start: 27 parts, among them CN203 DB25_Stack_FemaleAndMale, CN207 POWER LED, Q200 MMBT3904, Q201 MMBT3906, U203 8520, U205 TRS213, U209 74HCT08

Commit message: Main Board Routing 25-MAY-2024
Parts:
- added R248: 1k, Resistor_SMD:R_0603_1608Metric, symbol Device:R
Connections:
- net +5V: now also R248.1
- net _INT6: now also R248.2
Other:
- moved on the sheet: C230, C231, C236, C237, C240, CN203B, CN207, D201, D400, F2, U203B, U205A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
