File: KiCAD/AmigaPCI Mainboard-KiCAD REV 30/chip_memory.kicad_sch (KiCad schematic)
At the start: 25 parts, among them U701 74AHC245, U702 74AHC245, U703 74AHC245, U704 74AHC245, U705 74AHC245, U706 74AHC245, U707 SDRAM(2Mx32)

Commit message: Rev 3.0 PCB Routing 12-MAY-2024
Other:
- note added: "FYI-64MB ONBOARD MEMORY LOCATED AT $0400 0000-$07FF FFFF. DO WE NEED A RAMSEY FOR THIS TO WORK?"
- note added: "Ramsey ID register is at $00DE0043 -04 = $0D -07 = $0F"
Changed lines of the file:
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@@
+		)
+	)
+	(text "Ramsey ID register is at $00DE0043\n-04 = $0D\n-07 = $0F"
+		(exclude_from_sim no)
+		(at 164.211 264.287 0)
+		(effects
+			(font
+				(size 1.27 1.27)
+			)
+			(justify left bottom)
+		)
+	)
+	(text "FYI-64MB ONBOARD MEMORY LOCATED AT $0400 0000-$07FF FFFF.\nDO WE NEED A RAMSEY FOR THIS TO WORK?"
+		(exclude_from_sim no)
+		(at 160.02 256.286 0)
+		(effects
+			(font
+				(size 1.3 1.3)
+			)
+			(justify left bottom)
 		)
 	)

Commit message: Main Board Routing 22-MAY-2024
Parts:
- added J700: RAM CLOCK, Connector_PinHeader_2.54mm:PinHeader_1x03_P2.54mm_Vertical, symbol Jumper:Jumper_3_Open
Connections:
- net RAMCLK: now also J700.2 (C)
- new net CLK40: J700.3 (B)
- new net CLK80: J700.1 (A)
Changed lines of the file:
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@@
 	(title_block
 		(title "AMIGA PCI")
-		(date "2024-05-18")
+		(date "2024-05-22")
 		(rev "3.0")
 	)
@@
 		)
 	)
+	(global_label "CLK80"
+		(shape input)
+		(at 278.13 212.09 180)
+		(fields_autoplaced yes)
+		(effects
+			(font
+				(size 1.27 1.27)
+			)
+			(justify right)
+		)
+		(property "Intersheetrefs" "${INTERSHEET_REFS}"
+			(at 269.1577 212.09 0)
+			(effects
+				(font
+					(size 1.27 1.27)
+				)
+				(justify right)
+			)
+		)
+	)
 	(global_label "_CRCS"
 		(shape input)
@@
 		)
 	)
+	(global_label "CLK40"
+		(shape input)
+		(at 290.83 212.09 0)
+		(fields_autoplaced yes)
+		(effects
+			(font
+				(size 1.27 1.27)
+			)
+			(justify left)
+		)
+		(property "Intersheetrefs" "${INTERSHEET_REFS}"
+			(at 299.8023 212.09 0)
+			(effects
+				(font
+					(size 1.27 1.27)
+				)
+				(justify left)
+			)
+		)
+	)
 	(global_label "_VBEN"
 		(shape input)
@@
 		)
 	)
+	(global_label "RAMCLK"
+		(shape output)
+		(at 284.48 215.9 270)
+		(fields_autoplaced yes)
+		(effects
+			(font
+				(size 1.27 1.27)
+			)
+			(justify right)
+		)
+		(property "Intersheetrefs" "${INTERSHEET_REFS}"
+			(at 284.48 226.2633 90)
+			(effects
+				(font
+					(size 1.27 1.27)
+				)
+				(justify right)
+			)
+		)
+	)
 	(global_label "_CLLBE"
 		(shape input)
@@
 					(unit 1)
 				)
+			)
+		)
+	)
+	(symbol
+		(lib_id "Jumper:Jumper_3_Open")
+		(at 284.48 212.09 0)
+		(unit 1)
+		(exclude_from_sim yes)
+		(in_bom no)
+		(on_board yes)
+		(dnp no)
+		(fields_autoplaced yes)
+		(property "Reference" "J700"
+			(at 284.48 205.74 0)
+			(effects
+				(font
+					(size 1.27 1.27)
+				)
+			)
+		)
+		(property "Value" "RAM CLOCK"
+			(at 284.48 208.28 0)
+			(effects
+				(font
+					(size 1.27 1.27)
+				)
+			)
+		)
+		(property "Footprint" "Connector_PinHeader_2.54mm:PinHeader_1x03_P2.54mm_Vertical"
+			(at 284.48 212.09 0)
+			(effects
+				(font
+					(size 1.27 1.27)
+				)
+				(hide yes)
+			)
+		)
+		(property "Datasheet" "~"
+			(at 284.48 212.09 0)
+			(effects
+				(font
+					(size 1.27 1.27)
+				)
+				(hide yes)
+			)
+		)
+		(property "Description" "Jumper, 3-pole, both open"
+			(at 284.48 212.09 0)
+			(effects
+				(font
+					(size 1.27 1.27)
+				)
+				(hide yes)
+			)
+		)
+		(pin "3"
+		)
+		(pin "1"
+		)
+		(pin "2"
+		)
+		(instances
+			(project "AmigaPCI Mainboard"
+				(path "/72453515-27fe-4336-91f3-e3c8054f7767/f63de3eb-8614-4bac-88f2-650f5bad2338"
+					(reference "J700")
+					(unit 1)
+				)
