File: KiCAD/AmigaPCI 68040 Local Bus Card/CPU.kicad_sch (KiCad schematic)
At the start: 31 parts, among them U101 74LVC245, U102 74LVC245, U103 74LVC245, U104 74LVC245, U105 74LVC245, U106 74LVC245, U107 74LVC245, U108 74LVC245, U200 MC68040

Commit message: Routing 24-MAY-2024
Parts:
- added R100, R101, R102, R103, R104: 2k7, Resistor_SMD:R_0603_1608Metric, symbol Device:R
Connections:
- net +5V: now also R100.1, R101.1, R102.1, R103.1, R104.1
- net SC0: now also R100.2
- net SC1: now also R101.2
- net TDO: now also R104.2
- net _CDIS: now also R102.2
- net _MDIS: now also R103.2
