File: KiCAD/AmigaPCI 68040 Local Bus Card/FastMem.kicad_sch (KiCad schematic)
At the start: 15 parts, among them J400 RAMCLK, U401 SDRAM(16Mx32), U402 SDRAM(16Mx32)

Commit message: Routing 24-MAY-2024
Other:
- note added: "16MB RAMSEY MEMORY LOCATED AT $0700 0000-$07FF FFFF."
- note removed: "64MB ONBOARD MEMORY LOCATED AT $0400 0000-$07FF FFFF. DO WE NEED A RAMSEY FOR THIS TO WORK?"
- note removed: "BANK 0 ONLY 32MB = 8Mx16 64MB = 16Mx16 128MB = 32MX16 BOTH BANKS INSATALLED 64MB = 8Mx16 128MB = 16Mx16 256MB = 32Mx16"
Changed lines of the file:
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@@
 	(title_block
 		(title "AmigaPCI 68040")
-		(date "2024-05-09")
+		(date "2024-05-24")
 		(rev "1.0")
 	)
@@
 		)
 	)
-	(text "BANK 0 ONLY\n32MB = 8Mx16\n64MB = 16Mx16\n128MB = 32MX16\n\nBOTH BANKS INSATALLED\n64MB = 8Mx16\n128MB = 16Mx16\n256MB = 32Mx16"
-		(exclude_from_sim no)
-		(at 250.952 258.064 0)
-		(effects
-			(font
-				(size 3 3)
-			)
-			(justify left bottom)
-		)
-	)
 	(text "RAM CLOCK SPEED"
 		(exclude_from_sim no)
@@
 		)
 	)
-	(text "64MB ONBOARD MEMORY LOCATED AT $0400 0000-$07FF FFFF.\nDO WE NEED A RAMSEY FOR THIS TO WORK?"
+	(text "16MB RAMSEY MEMORY LOCATED AT $0700 0000-$07FF FFFF."
 		(exclude_from_sim no)
-		(at 257.937 202.565 0)
+		(at 237.49 209.042 0)
 		(effects
 			(font
-				(size 1.3 1.3)
+				(size 3 3)
 			)
 			(justify left bottom)
@@
 	(text "Ramsey ID register is at $00DE0043\n-04 = $0D\n-07 = $0F"
 		(exclude_from_sim no)
-		(at 262.128 210.566 0)
+		(at 237.236 224.79 0)
 		(effects
 			(font
-				(size 1.27 1.27)
+				(size 3 3)
 			)
 			(justify left bottom)
