File: KiCAD/DEV/AmigaPCI Mainboard-KiCAD REV 51/clocks.kicad_sch (KiCad schematic)
At the start: 46 parts, among them U108 74AHC04, U210 AT27C4096, U211 AT27C4096, U219 74AHCT04, U230 74LVC157, U812 74LVC245, U813 74LVC245, U814 74LVC245, U815 74LVC08, U816 74LVC245, U817 74LVC245, U818 74LVC245, U819 74LVC245, X1 6MHz, X2 33MHz, X3 28.63636MHz

Commit message: APCI Rev 5.1 Work
Connections:
- net _WEB renamed R_WC
Changed lines of the file:
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@@
 		)
 	)
-	(label "_WEB"
+	(label "R_WC"
 		(at 360.68 143.51 180)
 		(effects
@@
 		)
 	)
-	(label "_WEB"
+	(label "R_WC"
 		(at 381 48.26 0)
 		(effects
@@
 		)
 	)
-	(label "_WEB"
+	(label "R_WC"
 		(at 360.68 66.04 180)
 		(effects
@@
 		)
 	)
-	(label "_WEB"
+	(label "R_WC"
 		(at 360.68 105.41 180)
 		(effects
@@
 		)
 	)
-	(label "_WEB"
+	(label "R_WC"
 		(at 360.68 180.34 180)
 		(effects
@@
 		)
 	)
-	(global_label "_WEB"
+	(global_label "R_WC"
 		(shape input)
 		(at 391.16 48.26 0)
