File: KiCAD/DEV/AmigaPCI Mainboard-KiCAD REV 51/cpu.kicad_sch (KiCad schematic)
At the start: 49 parts, among them CN200 DIN41612_03x40, CN712 SPI, U712 ICE40HX4K-TQ144, U712F1 W25X20CLSN

Commit message: APCI Rev5.1 Work
Parts:
- added R269, R270, R271: 2k7, Resistor_SMD:R_0603_1608Metric, symbol Device:R
Connections:
- net +5V: now also R269.1, R270.1, R271.1
- net _IPL0: now also R269.2
- net _IPL1: now also R270.2
- net _IPL2: now also R271.2

Commit message: Amiga PCI Rev 5.1 Work
Connections:
- net GND: now also CN200.a13 (Pin_a13)
- net TM2: no longer CN200.a13 (Pin_a13)
- net _BLS: now reaches U712.113 (IO0_170)
- no-connect marks 5 -> 4
Changed lines of the file:
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@@
 	(title_block
 		(title "AMIGA PCI")
-		(date "2025-03-31")
+		(date "2025-04-01")
 		(rev "5.1")
 	)
@@
 	)
 	(junction
+		(at 222.25 140.97)
+		(diameter 0)
+		(color 0 0 0 0)
+	)
+	(junction
 		(at 68.58 213.36)
 		(diameter 0)
@@
 	)
 	(no_connect
-		(at 134.62 172.72)
-	)
-	(no_connect
 		(at 125.73 83.82)
 	)
@@
 	(wire
 		(pts
-			(xy 222.25 123.19) (xy 222.25 176.53)
+			(xy 222.25 123.19) (xy 222.25 140.97)
 		)
 		(stroke
@@
 	(wire
 		(pts
-			(xy 208.28 140.97) (xy 229.87 140.97)
-		)
-		(stroke
-			(width 0)
-			(type default)
-		)
-	)
-	(wire
-		(pts
 			(xy 224.79 69.85) (xy 229.87 69.85)
 		)
@@
 	(wire
 		(pts
-			(xy 134.62 172.72) (xy 125.73 172.72)
+			(xy 125.73 172.72) (xy 144.78 172.72)
 		)
 		(stroke
@@
 	(wire
 		(pts
+			(xy 222.25 140.97) (xy 222.25 176.53)
+		)
+		(stroke
+			(width 0)
+			(type default)
+		)
+	)
+	(wire
+		(pts
 			(xy 68.58 210.82) (xy 74.93 210.82)
 		)
@@
 	(wire
 		(pts
+			(xy 222.25 140.97) (xy 229.87 140.97)
+		)
+		(stroke
+			(width 0)
+			(type default)
+		)
+	)
+	(wire
+		(pts
 			(xy 163.83 76.2) (xy 163.83 83.82)
 		)
@@
 		)
 	)
-	(global_label "TM2"
+	(global_label "_BLS"
 		(shape output)
-		(at 208.28 140.97 180)
-		(fields_autoplaced yes)
+		(at 144.78 172.72 0)
 		(effects
 			(font
 				(size 1.27 1.27)
 			)
-			(justify right)
+			(justify left)
 		)
 		(property "Intersheetrefs" "${INTERSHEET_REFS}"
-			(at 201.6663 140.97 0)
+			(at 152.4 172.72 0)
 			(effects
 				(font
 					(size 1.27 1.27)
 				)
-				(justify right)
+				(justify left)
 			)
 		)

Commit message: APCI Rev 5.1 Work
Connections:
- net _WEA renamed R_WB
Changed lines of the file:
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@@
 		)
 	)
-	(global_label "_WEA"
+	(global_label "R_WB"
 		(shape input)
 		(at 134.62 228.6 0)

Commit message: APCI Rev 5.1 Work
Parts:
- added R163: 2k7, Resistor_SMD:R_0603_1608Metric, symbol Device:R_Small
- added R276: 2k7, Resistor_SMD:R_0603_1608Metric, symbol Device:R
- added U814, U816, U817: 74LVC245, Package_SO:TSSOP-20_4.4x6.5mm_P0.65mm, symbol AmigaPCI-Symbols:74LVC245
Connections:
- net +3V3: now also R221.1, R242.1, R163.2, R276.1, U814.1 (A->B)
- net +5V: no longer R221.1, R242.1
- net GND: now also U814.19 (CE), U816.11 (B7), U816.12 (B6), U816.13 (B5), U816.14 (B4), U816.15 (B3), U816.16 (B2), U816.19 (CE), U816.4 (A2), U816.5 (A3), U816.6 (A4), U816.7 (A5), U816.8 (A6), U816.9 (A7), U817.19 (CE)
- net LVC1: now also U814.12 (B6)
- net LVC3: now also U814.13 (B5)
- net _TCI: now also R276.2
- new net BUSDIR: U817.1 (A->B)
- new net C1: U814.8 (A6)
- new net C3: U814.7 (A5)
- new net LVOVL: U814.11 (B7)
- new net LVPARITY: U816.3 (A1)
- new net OVL: U814.9 (A7)
- new net PAR: U816.17 (B1)
- new net PCIDIR: U816.1 (A->B)
- new net _BUSREQ0: U814.18 (B0)
- new net _BUSREQ1: U814.16 (B2)
- new net _BUSREQ2: U814.17 (B1)
- new net _BUSREQ3: U814.14 (B4)
- new net _BUSREQ4: U814.15 (B3)
- new net _CBE0: U817.2 (A0)
- new net _CBE1: U817.3 (A1)
- new net _CBE2: U817.5 (A3)
- new net _CBE3: U817.6 (A4)
- new net _DEVSEL: U817.16 (B2)
- new net _FRAME: U817.7 (A5)
- new net _IRDY: U817.8 (A6)
- new net _LVCBE0: U817.18 (B0)
- new net _LVCBE1: U817.17 (B1)
- new net _LVCBE2: U817.15 (B3)
- new net _LVCBE3: U817.14 (B4)
- new net _LVDEVSEL: R163.1, U817.4 (A2)
- new net _LVFRAME: U817.13 (B5)
- new net _LVIRDY: U817.12 (B6)
- new net _LVPERR: U816.18 (B0)
- new net _LVTRDY: U817.9 (A7)
- new net _PERR: U816.2 (A0)
- new net _REQ0: U814.2 (A0)
- new net _REQ1: U814.4 (A2)
- new net _REQ2: U814.3 (A1)
- new net _REQ3: U814.6 (A4)
- new net _REQ4: U814.5 (A3)
- new net _TRDY: U817.11 (B7)
Other:
- note added: "ADDRESS PHASE DATA PHASE ------------- ------------- PAR _PERR PAR _PERR --------------------------------------- CPU WR BRIDGE PCI BRIDGE PCI CPU RD BRIDGE PCI PCI BRIDGE DMA WR PCI BRIDGE PCI BRIDGE DMA RD PCI BRIDGE BRIDGE PCI"
- note added: "PCI BUFFERS"
- moved on the sheet: R221, R227, R228, R234, R235, R236, R238, R239, R240, R242, R243, R244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

Commit message: APCI Rev 5.1 Work
Parts:
- removed R227, R228: 2k7, Resistor_SMD:R_0603_1608Metric, symbol Device:R
Connections:
- net UPA0 is gone; now on net GND: CN200.c33 (Pin_c33)
- net UPA1 is gone; now on net GND: CN200.b34 (Pin_b34)
- net GND: no longer CN200.a13 (Pin_a13)
- net TM2: now also CN200.a13 (Pin_a13)
