File: KiCAD/DEV/AmigaPCI Mainboard-KiCAD REV 51/floppy.kicad_sch (KiCad schematic)
At the start: 25 parts, among them CN203 DB25_Stack_FemaleAndMale, CN204 INTERNAL FLOPPY, J200 SHORT FOR DF1, J201 1-2 AMIGA DRIVES/2-3 PC DRIVES, J202 1-2 AMIGA DRIVES/2-3 PC DRIVES, J207 TICK, J208 TBASE, U204 8520, U209 74HCT08, U212 74HCT74, U213 74HCT00, U215 74HCT03, U219 74AHCT04, U305 74HCT08

Commit message: APCI Rev5.1 Work
Parts:
- added D206, D207, D208, D209: ESDS452, Package_TO_SOT_SMD:SOT-23, symbol AmigaPCI-Symbols:ESDS452
Connections:
- net GND: now also D206.3 (GND), D207.3 (GND), D208.3 (GND), D209.3 (GND)
- net PPD0: now also D206.2 (IO2)
- net PPD1: now also D206.1 (IO1)
- net PPD2: now also D207.2 (IO2)
- net PPD3: now also D207.1 (IO1)
- net PPD4: now also D208.2 (IO2)
- net PPD5: now also D208.1 (IO1)
- net PPD6: now also D209.2 (IO2)
- net PPD7: now also D209.1 (IO1)
Other:
- moved on the sheet: U219D, U219F

Commit message: APCI Rev 5.1 Work
Parts:
- added D210, D212: ESDS452, AmigaPCI:SOT-23, symbol AmigaPCI-Symbols:ESDS452
- D206, D207, D208, D209: footprint Package_TO_SOT_SMD:SOT-23 -> AmigaPCI:SOT-23
Connections:
- net GND: now also D210.3 (GND), D212.3 (GND)
- net PBUSY: now also D210.1 (IO1)
- net PPD0: now also D206.1 (IO1); no longer D206.2 (IO2)
- net PPD1: now also D206.2 (IO2); no longer D206.1 (IO1)
- net PPD2: now also D207.1 (IO1); no longer D207.2 (IO2)
- net PPD3: now also D207.2 (IO2); no longer D207.1 (IO1)
- net PPD4: now also D208.1 (IO1); no longer D208.2 (IO2)
- net PPD5: now also D208.2 (IO2); no longer D208.1 (IO1)
- net PPD6: now also D209.1 (IO1); no longer D209.2 (IO2)
- net PPD7: now also D209.2 (IO2); no longer D209.1 (IO1)
- net PPOUT: now also D210.2 (IO2)
- net _FIR0: now also D212.2 (IO2)
- net _FIR1: now also D212.1 (IO1)
Other:
- moved on the sheet: D206, D207, D208, D209, U219D, U219F
