File: KiCAD/DEV/AmigaPCI Mainboard-KiCAD REV 51/pcibus.kicad_sch (KiCad schematic)
At the start: 67 parts, among them CN100 PCI32-5V, CN101 PCI32-5V, CN102 PCI32-5V, CN103 PCI32-5V, CN104 PCI32-5V, U814 74LVC245, U815 74LVC08, U816 74LVC245, U817 74LVC245

Commit message: APCI Rev 5.1 Work
Connections:
- net +3V3: now also C100.1, C101.1, C102.1, C103.1, C104.1, C105.1, C106.1, C107.1, C108.1, C109.1, R101.2, R102.2, R105.1, R106.1, R107.1, R108.2, R109.2, R110.2, R113.1, R114.1, R115.1, R116.2, R117.2, R118.2, R121.1, R122.1, R123.1, R124.2, R125.2, R126.2, R129.1, R130.1, R131.1, R132.2, R133.2, R134.2, R137.1, R138.1, R139.1, R146.1, R147.1, R148.1, R149.1, R150.1, R162.2, RN100.1 (common)
- net +5V: no longer C100.1, C101.1, C102.1, C103.1, C104.1, C105.1, C106.1, C107.1, C108.1, C109.1, R101.2, R102.2, R105.1, R106.1, R107.1, R108.2, R109.2, R110.2, R113.1, R114.1, R115.1, R116.2, R117.2, R118.2, R121.1, R122.1, R123.1, R124.2, R125.2, R126.2, R129.1, R130.1, R131.1, R132.2, R133.2, R134.2, R137.1, R138.1, R139.1, R146.1, R147.1, R148.1, R149.1, R150.1, R162.2, RN100.1 (common)

Commit message: APCI Rev 5.1 Work
Parts:
- removed R163: 2k7, Resistor_SMD:R_0603_1608Metric, symbol Device:R_Small
- removed U814, U816, U817: 74LVC245, Package_SO:TSSOP-20_4.4x6.5mm_P0.65mm, symbol AmigaPCI-Symbols:74LVC245
Connections:
- net +3V3: no longer R108.2, R116.2, R124.2, R132.2, R162.2, RN100.1 (common), RN101.1 (common)
- net +5V: now also R108.2, R116.2, R124.2, R132.2, R162.2, RN100.1 (common), RN101.1 (common)
Other:
- note removed: "ADDRESS PHASE DATA PHASE ------------- ------------- PAR _PERR PAR _PERR --------------------------------------- CPU WR BRIDGE PCI BRIDGE PCI CPU RD BRIDGE PCI PCI BRIDGE DMA WR PCI BRIDGE PCI BRIDGE DMA RD PCI BRIDGE BRIDGE PCI"
- note removed: "PULL ME!"
- moved on the sheet: R108, R116, R124, R132, R162
