File: KiCAD/DEV/AmigaPCI 68040 Local Bus Card Rev 42/CardConnector.kicad_sch (KiCad schematic)
At the start: 43 parts, among them CN100 DIN41612_03x40, CN111 SPI, U111 ICE40HX4K-TQ144, U409F2 W25X20CLSN, X100 40MHz

Commit message: Local Bus Card Rev 4.2 work.
Connections:
- net UPA0 is gone; now on net GND: CN100.c33 (Pin_c33)
- net UPA1 is gone; now on net GND: CN100.b34 (Pin_b34)
- net GND: no longer CN100.a13 (Pin_a13)
- new net TM2: CN100.a13 (Pin_a13)
Changed lines of the file:
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@@
 	(title_block
 		(title "AmigaPCI 68040 Local Bus Card")
-		(date "2025-04-03")
+		(date "2025-04-10")
 		(rev "4.2")
 	)
@@
 	)
 	(junction
+		(at 87.63 146.05)
+		(diameter 0)
+		(color 0 0 0 0)
+	)
+	(junction
 		(at 194.31 59.69)
 		(diameter 0)
@@
 	)
 	(junction
+		(at 87.63 140.97)
+		(diameter 0)
+		(color 0 0 0 0)
+	)
+	(junction
 		(at 360.68 161.29)
 		(diameter 0)
@@
 	)
 	(junction
-		(at 59.69 135.89)
-		(diameter 0)
-		(color 0 0 0 0)
-	)
-	(junction
 		(at 302.26 59.69)
 		(diameter 0)
@@
 	(wire
 		(pts
-			(xy 59.69 135.89) (xy 59.69 171.45)
+			(xy 59.69 118.11) (xy 59.69 171.45)
 		)
 		(stroke
@@
 	(wire
 		(pts
+			(xy 80.01 140.97) (xy 87.63 140.97)
+		)
+		(stroke
+			(width 0)
+			(type default)
+		)
+	)
+	(wire
+		(pts
 			(xy 191.77 38.1) (xy 191.77 24.13)
 		)
@@
 	(wire
 		(pts
-			(xy 59.69 118.11) (xy 59.69 135.89)
-		)
-		(stroke
-			(width 0)
-			(type default)
-		)
-	)
-	(wire
-		(pts
 			(xy 179.07 48.26) (xy 179.07 54.61)
 		)
@@
 	(wire
 		(pts
-			(xy 80.01 140.97) (xy 101.6 140.97)
-		)
-		(stroke
-			(width 0)
-			(type default)
-		)
-	)
-	(wire
-		(pts
 			(xy 118.11 116.84) (xy 123.19 116.84)
 		)
@@
 	(wire
 		(pts
-			(xy 59.69 135.89) (xy 67.31 135.89)
-		)
-		(stroke
-			(width 0)
-			(type default)
-		)
-	)
-	(wire
-		(pts
 			(xy 57.15 163.83) (xy 67.31 163.83)
 		)
@@
 	(wire
 		(pts
+			(xy 87.63 146.05) (xy 87.63 166.37)
+		)
+		(stroke
+			(width 0)
+			(type default)
+		)
+	)
+	(wire
+		(pts
 			(xy 273.05 171.45) (xy 264.16 171.45)
 		)
@@
 	(wire
 		(pts
-			(xy 87.63 113.03) (xy 87.63 166.37)
+			(xy 87.63 113.03) (xy 87.63 140.97)
 		)
 		(stroke
@@
 		)
 	)
+	(wire
+		(pts
+			(xy 45.72 135.89) (xy 67.31 135.89)
+		)
+		(stroke
+			(width 0)
+			(type default)
+		)
+	)
 	(bus
 		(pts
@@
 	(wire
 		(pts
-			(xy 80.01 146.05) (xy 101.6 146.05)
-		)
-		(stroke
-			(width 0)
-			(type default)
-		)
-	)
-	(wire
-		(pts
 			(xy 118.11 91.44) (xy 123.19 91.44)
 		)
@@
 	(wire
 		(pts
+			(xy 80.01 146.05) (xy 87.63 146.05)
+		)
+		(stroke
+			(width 0)
+			(type default)
+		)
+	)
+	(wire
+		(pts
 			(xy 80.01 100.33) (xy 101.6 100.33)
 		)
@@
 	(wire
 		(pts
+			(xy 87.63 140.97) (xy 87.63 146.05)
+		)
+		(stroke
+			(width 0)
+			(type default)
+		)
+	)
+	(wire
+		(pts
 			(xy 332.74 50.8) (xy 342.9 50.8)
 		)
@@
 		)
 	)
+	(global_label "TM2"
+		(shape input)
+		(at 45.72 135.89 180)
+		(fields_autoplaced yes)
+		(effects
+			(font
+				(size 1.27 1.27)
+			)
+			(justify right)
+		)
+		(property "Intersheetrefs" "${INTERSHEET_REFS}"
+			(at 39.1063 135.89 0)
+			(effects
+				(font
+					(size 1.27 1.27)
+				)
+				(justify right)
+			)
+		)
+	)
 	(global_label "_BR"
 		(shape input)
@@
 		)
 	)
-	(global_label "UPA0"
-		(shape input)
-		(at 101.6 140.97 0)
-		(fields_autoplaced yes)
-		(effects
-			(font
-				(size 1.27 1.27)
-			)
-			(justify left)
-		)
-		(property "Intersheetrefs" "${INTERSHEET_REFS}"
-			(at 109.4838 140.97 0)
-			(effects
-				(font
-					(size 1.27 1.27)
-				)
-				(justify left)
-			)
-		)
-	)
 	(global_label "BCLKB"
 		(shape output)
@@
 			(effects
 				(font
-					(size 1.27 1.27)
-				)
-				(justify left)
-			)
-		)
-	)
-	(global_label "UPA1"
-		(shape input)
-		(at 101.6 146.05 0)
-		(fields_autoplaced yes)
-		(effects
-			(font
-				(size 1.27 1.27)
-			)
-			(justify left)
-		)
-		(property "Intersheetrefs" "${INTERSHEET_REFS}"
-			(at 109.4838 146.05 0)
-			(effects
-				(font
